Commit message: custom moveit config. adapted launch file.

File: mopa_description/robots/panda_hand_realsense.urdf.xacro (robot description, xacro)
@@ -4,5 +4,6 @@
   <xacro:include filename="$(find franka_description)/robots/hand.xacro"/>
   <xacro:include filename="$(find mopa_description)/robots/realsense.xacro"/>
-  <xacro:panda_arm xyz="0 0 0" />
+  <link name="panda_base"/>
+  <xacro:panda_arm xyz="0 0 0" connected_to="panda_base"/>
   <xacro:hand ns="panda" rpy="0 0 ${-pi/4}" connected_to="panda_link8" />
   <xacro:realsense ns="panda" rpy="3.14 -1.55 0.0" xyz="0.04 0.0 0.04" connected_to="panda_hand"/>

Commit message: Added camera model to the URDF

File: mopa_description/robots/panda_hand_realsense.urdf.xacro (robot description, xacro)
@@ -7,4 +7,7 @@
   <xacro:panda_arm xyz="0 0 0" connected_to="panda_base"/>
   <xacro:hand ns="panda" rpy="0 0 ${-pi/4}" connected_to="panda_link8" />
-  <xacro:realsense ns="panda" rpy="3.14 -1.55 0.0" xyz="0.04 0.0 0.04" connected_to="panda_hand"/>
+  <!-- Hand-eye calibration -->
+  <xacro:property name="xyz_panda_link7_camera_link" value="0.06308534561732076 -0.08993980659751674 0.1481860837701407"/>
+  <xacro:property name="rpy_panda_link7_camera_link" value="-2.68850999 -1.56973844 -1.20267232"/>
+  <xacro:realsense ns="panda" rpy="${rpy_panda_link7_camera_link}" xyz="${xyz_panda_link7_camera_link}" connected_to="panda_link7"/>
 </robot>

File: mopa_description/robots/realsense.xacro (robot description, xacro)
@@ -5,5 +5,5 @@
       <joint name="${ns}_realsense_joint" type="fixed">
         <parent link="${connected_to}"/>
-        <child link="${ns}_realsense_link"/>
+        <child link="camera_link"/>
         <origin xyz="${xyz}" rpy="${rpy}"/>
       </joint>
@@ -14,5 +14,17 @@
       <xacro:include filename="$(find mopa_description)/robots/realsense.gazebo.xacro"/>
     </xacro:if>
-    <link name="${ns}_realsense_link">
+    <!-- The following values model the aluminum peripherial case for the
+  	D435 camera, with the camera joint represented by the actual
+  	peripherial camera tripod mount -->
+    <xacro:property name="d435_cam_width" value="0.090"/>
+    <xacro:property name="d435_cam_height" value="0.025"/>
+    <xacro:property name="d435_cam_depth" value="0.02505"/>
+    <xacro:property name="d435_cam_mount_from_center_offset" value="0.0149"/>
+    <!-- The following offset is relative the the physical D435 camera peripherial
+  	camera tripod mount -->
+    <xacro:property name="d435_cam_depth_px" value="${d435_cam_mount_from_center_offset}"/>
+    <xacro:property name="d435_cam_depth_py" value="0.0175"/>
+    <xacro:property name="d435_cam_depth_pz" value="${d435_cam_height/2}"/>
+    <link name="camera_link">
       <inertial>
         <mass value="0.05" />
@@ -20,14 +32,13 @@
       </inertial>
       <visual>
+        <origin xyz="${d435_cam_mount_from_center_offset} ${-d435_cam_depth_py} 0" rpy="${pi/2} 0 ${pi/2}"/>
         <geometry>
-          <mesh filename="package://mopa_description/meshes/realsense_r200.dae"/>
+          <mesh filename="package://realsense2_description/meshes/d435.dae" />
         </geometry>
-        <material name="blueish">
-          <color rgb="0.01 0.73 0.99 1.0"/>
-        </material>
+        <material name="aluminum"/>
       </visual>
       <collision>
         <geometry>
-          <box size="0.008 0.13 0.02"/>
+          <box size="${d435_cam_depth} ${d435_cam_width} ${d435_cam_height}"/>
         </geometry>
       </collision>

Commit message: Add EE to URDF

File: mopa_description/robots/panda_hand_realsense.urdf.xacro (robot description, xacro)
@@ -11,3 +11,10 @@
   <xacro:property name="rpy_panda_link7_camera_link" value="-2.68850999 -1.56973844 -1.20267232"/>
   <xacro:realsense ns="panda" rpy="${rpy_panda_link7_camera_link}" xyz="${xyz_panda_link7_camera_link}" connected_to="panda_link7"/>
+  <!-- Add EE frame -->
+  <link name="panda_default_EE"/>
+  <joint name="joint_link8_default_ee" type="fixed">
+        <parent link="panda_link8"/>
+        <child link="panda_default_EE"/>
+        <origin rpy="0.000 0.000 -0.785" xyz="0.000 0.000 0.103"/>
+  </joint>
 </robot>
