Commit message: Created panda mount and cleaning up xacros

File: moma_description/urdf/mobmi.urdf.xacro (robot description, xacro)
@@ -5,23 +5,12 @@
   <xacro:ridgeback/>
   <!-- YuMi mount -->
-  <link name="ridgeback_yumi_mount_link">
-    <visual>
-      <geometry>
-        <mesh filename="package://moma_description/meshes/ridgeback_yumi_mount.dae"/>
-      </geometry>
-    </visual>
-    <collision>
-      <geometry>
-        <mesh filename="package://moma_description/meshes/ridgeback_yumi_mount.dae"/>
-      </geometry>
-    </collision>
-  </link>
-  <joint name="ridgeback_yumi_mount_joint" type="fixed">
-    <origin xyz="0 0 0" rpy="0 0 1.571" />
-    <parent link="mid_mount" />
-    <child link="ridgeback_yumi_mount_link" />
-  </joint>
+  <xacro:include
+    filename="$(find moma_description)/urdf/mounts/yumi_mount.urdf.xacro"/>
+  <xacro:yumi_mount connected_to="mid_mount" />
   <!-- YuMi -->
+  <xacro:property name="mid_mount_to_yumi_xyz" value="0.285 0 0.248" />
+  <xacro:property name="mid_mount_to_yumi_rpy" value="0 0 0" />
   <xacro:include filename="$(find moma_description)/urdf/yumi.xacro"/>
-  <xacro:yumi connected_to="ridgeback_yumi_mount_link" rpy="0 0 -${pi/2}"  xyz="0 -0.285 0.248"/>
+  <xacro:yumi connected_to="mid_mount"
+    rpy="${mid_mount_to_yumi_rpy}" xyz="${mid_mount_to_yumi_xyz}"/>
 </robot>

File: moma_description/urdf/mopa.urdf.xacro (robot description, xacro)
@@ -1,7 +1,16 @@
 <?xml version="1.0" encoding="utf-8"?>
 <robot xmlns:xacro="http://www.ros.org/wiki/xacro" name="mopa">
+  <!-- Ridgeback -->
   <xacro:include filename="$(find moma_description)/urdf/ridgeback.xacro"/>
+  <xacro:ridgeback/>
+  <!-- Panda mount -->
+  <xacro:include
+    filename="$(find moma_description)/urdf/mounts/panda_mount.urdf.xacro"/>
+  <xacro:panda_mount connected_to="mid_mount" />
+  <!-- Panda -->
+  <xacro:property name="mid_mount_to_panda_xyz" value="0.317 0 0.44" />
+  <xacro:property name="mid_mount_to_panda_rpy" value="0 0 0" />
   <xacro:include filename="$(find moma_description)/urdf/panda.xacro"/>
-  <xacro:ridgeback/>
-  <xacro:panda connected_to="top_link" xyz="0.2 0 0.3" />
+  <xacro:panda connected_to="mid_mount"
+    rpy="${mid_mount_to_panda_rpy}" xyz="${mid_mount_to_panda_xyz}"/>
 </robot>

Commit message: Added calibration comments.

File: moma_description/urdf/mobmi.urdf.xacro (robot description, xacro)
@@ -9,4 +9,5 @@
   <xacro:yumi_mount connected_to="mid_mount" />
   <!-- YuMi -->
+  <!-- State of calibration: Never (insert dd.mm.yyyy as soon as calibrated) -->
   <xacro:property name="mid_mount_to_yumi_xyz" value="0.285 0 0.248" />
   <xacro:property name="mid_mount_to_yumi_rpy" value="0 0 0" />

File: moma_description/urdf/mopa.urdf.xacro (robot description, xacro)
@@ -9,5 +9,6 @@
   <xacro:panda_mount connected_to="mid_mount" />
   <!-- Panda -->
-  <xacro:property name="mid_mount_to_panda_xyz" value="0.317 0 0.44" />
+  <!-- State of calibration: Never (insert dd.mm.yyyy as soon as calibrated) -->
+  <xacro:property name="mid_mount_to_panda_xyz" value="0.317 0 0.443" />
   <xacro:property name="mid_mount_to_panda_rpy" value="0 0 0" />
   <xacro:include filename="$(find moma_description)/urdf/panda.xacro"/>
