Commit message: Added hardware interface selection for panda and mopa

File: moma_description/urdf/mopa.urdf.xacro (robot description, xacro)
@@ -13,5 +13,8 @@
   <xacro:property name="mid_mount_to_panda_rpy" value="0 0 0" />
   <xacro:include filename="$(find moma_description)/urdf/panda.xacro"/>
+  <xacro:arg name="gazebo_panda_hardware_interface"
+    default="PositionJointInterface"/>
   <xacro:panda connected_to="mid_mount"
-    rpy="${mid_mount_to_panda_rpy}" xyz="${mid_mount_to_panda_xyz}"/>
+    rpy="${mid_mount_to_panda_rpy}" xyz="${mid_mount_to_panda_xyz}"
+    hardware_interface="$(arg gazebo_panda_hardware_interface)"/>
 </robot>

File: moma_description/urdf/panda.urdf.xacro (robot description, xacro)
@@ -2,6 +2,8 @@
 <robot xmlns:xacro="http://www.ros.org/wiki/xacro" name="panda">
   <link name="world" />
+  <xacro:arg name="gazebo_panda_hardware_interface"
+    default="PositionJointInterface"/>
   <xacro:include filename="$(find moma_description)/urdf/panda.xacro"/>
-  <xacro:panda connected_to="world"/>
+  <xacro:panda connected_to="world" hardware_interface="$(arg gazebo_panda_hardware_interface)"/>
   <gazebo>
     <plugin name="gazebo_ros_control" filename="libgazebo_ros_control.so">

File: moma_description/urdf/panda.xacro (robot description, xacro)
@@ -1,8 +1,10 @@
 <?xml version="1.0" encoding="utf-8"?>
 <robot xmlns:xacro="http://www.ros.org/wiki/xacro" name="panda">
-  <xacro:macro name="panda" params="connected_to:='' rpy:='0 0 0' xyz:='0 0 0'">
+  <xacro:macro name="panda" params="connected_to:='' rpy:='0 0 0' xyz:='0 0 0'
+    hardware_interface:='PositionJointInterface'">
     <!-- Panda arm  -->
     <xacro:include filename="$(find franka_description)/robots/panda_arm.xacro"/>
-    <xacro:panda_arm connected_to="${connected_to}" rpy="${rpy}" xyz="${xyz}"/>
+    <xacro:panda_arm connected_to="${connected_to}" rpy="${rpy}" xyz="${xyz}"
+      hardware_interface="${hardware_interface}"/>
     <!-- Panda hand -->
     <xacro:include filename="$(find franka_description)/robots/hand.xacro"/>
