Commit message: Added table to Yumi's URDF

File: moma_description/urdf/yumi.urdf.xacro (robot description, xacro)
@@ -4,3 +4,29 @@
   <xacro:include filename="$(find moma_description)/urdf/yumi.xacro"/>
   <xacro:yumi connected_to="base_link"/>
+  <!-- Add a table to avoid collisions with it -->
+  <link name="table_link">
+    <inertial>
+      <origin xyz="0 0 0.5" rpy="0 0 0"/>
+      <mass value="1"/>
+      <inertia ixx="100"  ixy="0"  ixz="0" iyy="100" iyz="0" izz="100" />
+    </inertial>
+    <visual>
+      <geometry>
+        <box size="0.6 0.6 0.04" />
+      </geometry>
+      <material name="magic">
+        <color rgba="0 0.625 0.625 0.625"/>
+      </material>
+    </visual>
+    <collision>
+      <geometry>
+        <box size="0.6 0.6 0.04" />
+      </geometry>
+    </collision>
+ </link>
+ <joint name="table_joint" type="fixed">
+    <parent link="base_link"/>
+    <child link="table_link"/>
+    <origin rpy="0.0 0.0 0.0" xyz="0.5 0.0 0.0"/>
+  </joint>
 </robot>

Commit message: Added EE to yumi_l

File: moma_description/urdf/yumi.urdf.xacro (robot description, xacro)
@@ -4,29 +4,3 @@
   <xacro:include filename="$(find moma_description)/urdf/yumi.xacro"/>
   <xacro:yumi connected_to="base_link"/>
-  <!-- Add a table to avoid collisions with it -->
-  <link name="table_link">
-    <inertial>
-      <origin xyz="0 0 0.5" rpy="0 0 0"/>
-      <mass value="1"/>
-      <inertia ixx="100"  ixy="0"  ixz="0" iyy="100" iyz="0" izz="100" />
-    </inertial>
-    <visual>
-      <geometry>
-        <box size="0.6 0.6 0.04" />
-      </geometry>
-      <material name="magic">
-        <color rgba="0 0.625 0.625 0.625"/>
-      </material>
-    </visual>
-    <collision>
-      <geometry>
-        <box size="0.6 0.6 0.04" />
-      </geometry>
-    </collision>
- </link>
- <joint name="table_joint" type="fixed">
-    <parent link="base_link"/>
-    <child link="table_link"/>
-    <origin rpy="0.0 0.0 0.0" xyz="0.5 0.0 0.0"/>
-  </joint>
 </robot>

File: moma_description/urdf/yumi.xacro (robot description, xacro)
@@ -24,4 +24,11 @@
       <origin xyz="0 0 0.007" rpy="0 0 ${pi}"/>
     </xacro:yumi_servo_gripper>
+    <!-- Add end effector frame for MoveIt -->
+    <link name="yumi_l_default_ee"/>
+    <joint name="joint_link_7_l_default_ee" type="fixed">
+      <parent link="yumi_link_7_l"/>
+      <child link="yumi_l_default_ee"/>
+      <origin rpy="0.0 0.0 1.571" xyz="0.0 0.0 0.1407"/>
+    </joint>
     <!-- Mount realsense -->
     <joint name="realsense_mount_joint" type="fixed">
@@ -33,5 +40,4 @@
       <visual>
         <geometry>
-          <!-- TODO(mbreyer) use CAD model for nicer looks -->
           <box size="0.14 0.05 0.04"/>
         </geometry>
@@ -47,4 +53,30 @@
     <xacro:include filename="$(find moma_description)/urdf/realsense.xacro"/>
     <xacro:realsense ns="yumi" connected_to="yumi_link_7_r" rpy="${rpy_yumi_link7_camera_link}" xyz="${xyz_yumi_link7_camera_link}"/>
+    <!-- Add a table to avoid collisions with it -->
+    <link name="table_link">
+      <inertial>
+        <origin xyz="0 0 0.5" rpy="0 0 0"/>
+        <mass value="1"/>
+        <inertia ixx="100"  ixy="0"  ixz="0" iyy="100" iyz="0" izz="100" />
+      </inertial>
+      <visual>
+        <geometry>
+          <box size="0.6 0.6 0.04" />
+        </geometry>
+        <material name="magic">
+          <color rgba="0 0.625 0.625 0.625"/>
+        </material>
+      </visual>
+      <collision>
+        <geometry>
+          <box size="0.6 0.6 0.04" />
+        </geometry>
+      </collision>
+  </link>
+  <joint name="table_joint" type="fixed">
+      <parent link="yumi_body"/>
+      <child link="table_link"/>
+      <origin rpy="0.0 0.0 0.0" xyz="0.5 0.0 0.0"/>
+    </joint>
   </xacro:macro>
 </robot>
