Commit message: Added pico flexx and chameleon to the URDF

File: moma_description/urdf/yumi.xacro (robot description, xacro)
@@ -7,5 +7,5 @@
     <xacro:include filename="$(find yumi_description)/urdf/yumi.xacro"/>
     <xacro:yumi name="yumi" hardware_interface="PositionJointInterface" parent="yumi_mount_link">
-      <origin/>  <!-- this has no effect -->
+      <origin/>
     </xacro:yumi>
     <xacro:unless value="${not connected_to}">
@@ -24,5 +24,10 @@
       <origin xyz="0 0 0.007" rpy="0 0 ${pi}"/>
     </xacro:yumi_servo_gripper>
-    <!-- TODO(mbreyer) mount pico flexx and chameleon -->
+    <!-- Mount pico flexx -->
+    <xacro:include filename="$(find moma_description)/urdf/pico_flexx.xacro"/>
+    <xacro:pico_flexx ns="yumi_r" connected_to="yumi_link_7_r" rpy="-0.22930307 -0.01920052 -0.00072021" xyz="-0.00152 -0.0601 0.0475"/>
+    <!-- Mount chameleon -->
+    <xacro:include filename="$(find moma_description)/urdf/chameleon.xacro"/>
+    <xacro:chameleon ns="yumi_r" connected_to="yumi_link_7_r" rpy="0.2542769 -0.00998312 -3.13862441" xyz="0.00114 -0.0911 0.0690"/>
   </xacro:macro>
 </robot>

Commit message: Realsense-wrist transform

File: moma_description/urdf/yumi.xacro (robot description, xacro)
@@ -25,9 +25,8 @@
     </xacro:yumi_servo_gripper>
     <!-- Mount pico flexx -->
-    <xacro:include filename="$(find moma_description)/urdf/pico_flexx.xacro"/>
-    <xacro:pico_flexx ns="yumi_r" connected_to="yumi_link_7_r" rpy="-0.22930307 -0.01920052 -0.00072021" xyz="-0.00152 -0.0601 0.0475"/>
-    <!-- Mount chameleon -->
-    <xacro:include filename="$(find moma_description)/urdf/chameleon.xacro"/>
-    <xacro:chameleon ns="yumi_r" connected_to="yumi_link_7_r" rpy="0.2542769 -0.00998312 -3.13862441" xyz="0.00114 -0.0911 0.0690"/>
+    <xacro:property name="xyz_yumi_link7_camera_link" value="-0.021534365646869183 -0.098057755914108952 0.069194569224013028"/>
+    <xacro:property name="rpy_yumi_link7_camera_link" value="-2.97446 -1.46168 -1.7345"/>
+    <xacro:include filename="$(find moma_description)/urdf/realsense.xacro"/>
+    <xacro:realsense ns="yumi" connected_to="yumi_link_7_r" rpy="${rpy_yumi_link7_camera_link}" xyz="${xyz_yumi_link7_camera_link}"/>
   </xacro:macro>
 </robot>

Commit message: Adapt collision matrix. Add collision box for realsense mount.

File: moma_description/urdf/yumi.xacro (robot description, xacro)
@@ -25,4 +25,22 @@
     </xacro:yumi_servo_gripper>
     <!-- Mount realsense -->
+    <joint name="realsense_mount_joint" type="fixed">
+        <parent link="yumi_link_7_r"/>
+        <child link="realsense_mount"/>
+        <origin rpy="0 0 0" xyz="0 -0.06 0.05"/>
+    </joint>
+    <link name="realsense_mount">
+      <visual>
+        <geometry>
+          <!-- TODO(mbreyer) use CAD model for nicer looks -->
+          <box size="0.14 0.05 0.04"/>
+        </geometry>
+      </visual>
+      <collision>
+        <geometry>
+          <box size="0.14 0.05 0.04"/>
+        </geometry>
+      </collision>
+    </link>
     <xacro:property name="xyz_yumi_link7_camera_link" value="-0.021534365646869183 -0.098057755914108952 0.069194569224013028"/>
     <xacro:property name="rpy_yumi_link7_camera_link" value="-2.97446 -1.46168 -1.7345"/>

Commit message: Fixed grasping sequence

File: moma_description/urdf/yumi.xacro (robot description, xacro)
@@ -56,9 +56,10 @@
     <link name="table_link">
       <inertial>
-        <origin xyz="0 0 0.5" rpy="0 0 0"/>
+        <origin xyz="0 0 0" rpy="0 0 0"/>
         <mass value="1"/>
         <inertia ixx="100"  ixy="0"  ixz="0" iyy="100" iyz="0" izz="100" />
       </inertial>
       <visual>
+        <origin xyz="0 0 0.22" rpy="0 0 0" />
         <geometry>
           <box size="0.6 0.6 0.04" />
@@ -69,4 +70,5 @@
       </visual>
       <collision>
+        <origin xyz="0 0 0.22" rpy="0 0 0" />
         <geometry>
           <box size="0.6 0.6 0.04" />
