Commit message: Add base to panda offset and visualization of base

File: moma_description/urdf/superpanda.urdf.xacro (robot description, xacro)
@@ -28,6 +28,19 @@
         <limit effort="0" velocity="0"/>
     </joint>
-    <link name="base_theta" />
+    <link name="base_theta">
+        <visual>
+          <origin xyz="0 0 0.1"/>
+          <geometry>
+            <box size="0.5 0.3 0.2"/>
+          </geometry>
+        </visual>
+    </link>
+    <joint name="base_to_panda" type="fixed">
+        <parent link="base_theta" />
+        <child link="arm_root" />
+        <origin xyz="0 0 0.2" rpy="0 0 0"/>
+    </joint>
+    <link name="arm_root" />
     <xacro:include filename="$(find moma_description)/urdf/panda.xacro"/>
-    <xacro:panda connected_to="base_theta" tool="$(arg tool)"/>
+    <xacro:panda connected_to="arm_root" tool="$(arg tool)"/>
 </robot>

Commit message: wip

File: moma_description/urdf/superpanda.urdf.xacro (robot description, xacro)
@@ -1,17 +1,17 @@
 <?xml version="1.0" encoding="utf-8"?>
-<robot xmlns:xacro="http://www.ros.org/wiki/xacro" name="royalpanda">
+<robot xmlns:xacro="http://www.ros.org/wiki/xacro" name="superpanda">
   <!-- SMB Arguments -->
   <xacro:arg name="wheel_joint_type"          default="continuous"/>
   <xacro:arg name="simulation"                default="true"/>
-  <xacro:arg name="use_ros_skid_steer"        default="false"/> <!-- Specify one! -->
+  <xacro:arg name="use_ros_skid_steer"        default="false"/>  <!-- Specify one! -->
   <xacro:arg name="use_ros_control"           default="true"/>
   <xacro:arg name="lidar"                     default="true"/>
   <xacro:arg name="robot_namespace"           default=""/>
   <xacro:arg name="description_name_xacro"    default="robot_description"/>
-  <xacro:arg name="publish_tf"                default="false"/>
+  <xacro:arg name="publish_tf"                default="true"/>
   <xacro:arg name="tracking_camera"           default="true"/>
   <xacro:property name="lidar" value="$(arg lidar)"/>
   <!-- SMB Includes -->
-  <xacro:include filename="$(find smb_description)/urdf/smb_big_properties.urdf.xacro" />
+  <xacro:include filename="$(find smb_description)/urdf/smb_piloting_properties.urdf.xacro" />
   <xacro:if value="$(arg simulation)">
     <xacro:include filename="$(find smb_description)/urdf/smb_gazebo_addins.urdf.xacro"/>
@@ -23,9 +23,9 @@
   <xacro:smb wheel_joint_type="$(arg wheel_joint_type)" simulation="$(arg simulation)" tracking_camera="$(arg tracking_camera)"/>
   <!-- Rigid fix between SMB and Panda -->
-  <link name="franka_mount_link" />
+  <link name="arm_mount_link"/>
   <joint name="arm_mount_joint" type="fixed">
       <parent link="base_link" />
-      <child link="franka_mount_link" />
-      <origin xyz="0.21 0.0 0.3" rpy="0 0 0"/>
+      <child link="arm_mount_link" />
+      <origin xyz="0.115 0.0 ${0.228+chassisHeight/2.0}" rpy="0 0 0"/>
   </joint>
   <!-- Panda Arguments -->
@@ -34,4 +34,4 @@
   <xacro:arg name="control_mode" default='Position'/>
   <xacro:include filename="$(find moma_description)/urdf/panda.xacro"/>
-  <xacro:panda connected_to="base_link" use_fixed_realsense="$(arg use_fixed_realsense)" control_mode="$(arg control_mode)" tool="$(arg tool)"/>
+  <xacro:panda connected_to="arm_mount_link" use_fixed_realsense="$(arg use_fixed_realsense)" control_mode="$(arg control_mode)" tool="$(arg tool) include_gazebo_control:=false"/>
 </robot>

Commit message: Add prototype MPC for Superpanda in simulation

File: moma_description/urdf/superpanda.urdf.xacro (robot description, xacro)
@@ -1,4 +1,39 @@
 <?xml version="1.0" encoding="utf-8"?>
 <robot xmlns:xacro="http://www.ros.org/wiki/xacro" name="superpanda">
+  <!-- MPC Arguments -->
+  <xacro:arg name="mpc_model" default="false"/>
+  <xacro:if value="$(arg mpc_model)">
+    <link name="world" />
+    <joint name="base_prismatic_x" type="prismatic">
+      <parent link="world" />
+      <child link="base_x" />
+      <origin xyz="0 0 0" rpy="0 0 0"/>
+      <axis xyz="1 0 0"/>
+      <limit effort="0" velocity="0"/>
+    </joint>
+    <link name="base_x" />
+    <joint name="base_prismatic_y" type="prismatic">
+      <parent link="base_x" />
+      <child link="base_y" />
+      <origin xyz="0 0 0" rpy="0 0 0"/>
+      <axis xyz="0 1 0"/>
+      <limit effort="0" velocity="0"/>
+    </joint>
+    <link name="base_y" />
+    <joint name="base_revolute_theta" type="revolute">
+      <parent link="base_y" />
+      <child link="base_theta" />
+      <origin xyz="0 0 0" rpy="0 0 0"/>
+      <axis xyz="0 0 1"/>
+      <limit effort="0" velocity="0"/>
+    </joint>
+    <link name="base_theta" />
+    <joint name="base_to_panda" type="fixed">
+      <parent link="base_theta" />
+      <child link="base_link" />
+      <origin xyz="0 0 0.2" rpy="0 0 0"/>
+    </joint>
+    <link name="base_link" />
+  </xacro:if>
   <!-- SMB Arguments -->
   <xacro:arg name="wheel_joint_type"          default="continuous"/>
@@ -17,15 +52,17 @@
     <xacro:include filename="$(find smb_description)/urdf/smb_gazebo_addins.urdf.xacro"/>
   </xacro:if>
-  <!-- SMB -->
-  <xacro:include filename="$(find smb_description)/urdf/smb.urdf.xacro">
-    <xacro:arg name="lidar" default="$(arg lidar)"/>
-  </xacro:include>
-  <xacro:smb wheel_joint_type="$(arg wheel_joint_type)" simulation="$(arg simulation)" tracking_camera="$(arg tracking_camera)"/>
+  <xacro:unless value="$(arg mpc_model)">
+    <!-- SMB -->
+    <xacro:include filename="$(find smb_description)/urdf/smb.urdf.xacro">
+      <xacro:arg name="lidar" default="$(arg lidar)"/>
+    </xacro:include>
+    <xacro:smb wheel_joint_type="$(arg wheel_joint_type)" simulation="$(arg simulation)" tracking_camera="$(arg tracking_camera)"/>
+  </xacro:unless>
   <!-- Rigid fix between SMB and Panda -->
   <link name="arm_mount_link"/>
   <joint name="arm_mount_joint" type="fixed">
-      <parent link="base_link" />
-      <child link="arm_mount_link" />
-      <origin xyz="0.115 0.0 ${0.228+chassisHeight/2.0}" rpy="0 0 0"/>
+    <parent link="base_link" />
+    <child link="arm_mount_link" />
+    <origin xyz="0.115 0.0 ${0.228+chassisHeight/2.0}" rpy="0 0 0"/>
   </joint>
   <!-- Panda Arguments -->

Commit message: Fix offset

File: moma_description/urdf/superpanda.urdf.xacro (robot description, xacro)
@@ -29,8 +29,8 @@
     </joint>
     <link name="base_theta" />
-    <joint name="base_to_panda" type="fixed">
+    <joint name="base_to_link" type="fixed">
       <parent link="base_theta" />
       <child link="base_link" />
-      <origin xyz="0 0 0.2" rpy="0 0 0"/>
+      <origin xyz="0 0 0" rpy="0 0 0"/>
     </joint>
     <link name="base_link" />
