Commit message: Mimic panda finger joint

File: moma_description/urdf/panda.xacro (robot description, xacro)
@@ -15,4 +15,11 @@
       <origin rpy="0.0 0.0 -0.785" xyz="0.0 0.0 0.103"/>
     </joint>
+    <!-- mimic joints for gazebo simulation -->
+    <gazebo>
+      <plugin name="panda_hand_mimic_joint_plugin" filename="libroboticsgroup_gazebo_mimic_joint_plugin.so">
+        <joint>panda_finger_joint1</joint>
+        <mimicJoint>panda_finger_joint2</mimicJoint>
+      </plugin>
+    </gazebo>
     <!-- Mount Realsense -->
     <xacro:property name="xyz_panda_link7_camera_link" value="0.06308534561732076 -0.08993980659751674 0.1481860837701407"/>

Commit message: Use realsense nominal extrinsics in simulation

File: moma_description/urdf/panda.xacro (robot description, xacro)
@@ -2,11 +2,11 @@
 <robot xmlns:xacro="http://www.ros.org/wiki/xacro" name="panda">
   <xacro:macro name="panda" params="connected_to:='' rpy:='0 0 0' xyz:='0 0 0'">
-    <!-- Panda arm  -->
+    <!-- panda arm  -->
     <xacro:include filename="$(find franka_description)/robots/panda_arm.xacro"/>
     <xacro:panda_arm connected_to="${connected_to}" rpy="${rpy}" xyz="${xyz}"/>
-    <!-- Panda hand -->
+    <!-- panda hand -->
     <xacro:include filename="$(find franka_description)/robots/hand.xacro"/>
     <xacro:hand ns="panda" rpy="0 0 ${-pi/4}" connected_to="panda_link8"/>
-    <!-- Add end effector frame for MoveIt -->
+    <!-- end effector frame for MoveIt -->
     <link name="panda_default_ee"/>
     <joint name="joint_link8_default_ee" type="fixed">
@@ -15,5 +15,5 @@
       <origin rpy="0.0 0.0 -0.785" xyz="0.0 0.0 0.103"/>
     </joint>
-    <!-- mimic joints for gazebo simulation -->
+    <!-- gazebo plugin to mimic finger joints -->
     <gazebo>
       <plugin name="panda_hand_mimic_joint_plugin" filename="libroboticsgroup_gazebo_mimic_joint_plugin.so">
@@ -22,9 +22,11 @@
       </plugin>
     </gazebo>
-    <!-- Mount Realsense -->
-    <xacro:property name="xyz_panda_link7_camera_link" value="0.06308534561732076 -0.08993980659751674 0.1481860837701407"/>
-    <xacro:property name="rpy_panda_link7_camera_link" value="-2.68850999 -1.56973844 -1.20267232"/>
-    <xacro:include filename="$(find moma_description)/urdf/realsense.xacro"/>
-    <xacro:realsense ns="panda" connected_to="panda_link7" rpy="${rpy_panda_link7_camera_link}" xyz="${xyz_panda_link7_camera_link}"/>
+    <!-- realsense -->
+    <xacro:include filename="$(find realsense2_description)/urdf/_d435.urdf.xacro" />
+    <xacro:property name="panda_link7_camera_bottom_screw_frame_rpy" value="-2.68850999 -1.56973844 -1.20267232" />
+    <xacro:property name="panda_link7_camera_bottom_screw_frame_xyz" value="0.06585917 -0.06861364 0.14820608" />
+    <xacro:sensor_d435 parent="panda_link7">
+      <origin rpy="${panda_link7_camera_bottom_screw_frame_rpy}" xyz="${panda_link7_camera_bottom_screw_frame_xyz}" />
+    </xacro:sensor_d435>
   </xacro:macro>
 </robot>

Commit message: Royal panda moveit config

File: moma_description/urdf/panda.xacro (robot description, xacro)
@@ -1,5 +1,5 @@
 <?xml version="1.0" encoding="utf-8"?>
 <robot xmlns:xacro="http://www.ros.org/wiki/xacro" name="panda">
-  <xacro:macro name="panda" params="connected_to:='' rpy:='0 0 0' xyz:='0 0 0' use_fixed_realsense:=false">
+  <xacro:macro name="panda" params="connected_to:='' rpy:='0 0 0' xyz:='0 0 0' use_fixed_realsense:=false include_gazebo_control:=true">
     <!-- panda arm  -->
     <xacro:include filename="$(find franka_description)/robots/panda_arm.xacro"/>
@@ -17,5 +17,5 @@
     <!-- Gazebo tags -->
     <xacro:include filename="$(find franka_description)/robots/panda_arm.gazebo.xacro"/>
-    <xacro:panda_gazebo arm_id="panda"/>
+    <xacro:panda_gazebo arm_id="panda" include_gazebo_control="${include_gazebo_control}"/>
     <!-- wrist realsense -->
     <xacro:include filename="$(find realsense2_description)/urdf/_d435.urdf.xacro" />

File: moma_description/urdf/royalpanda.urdf.xacro (robot description, xacro)
@@ -10,4 +10,4 @@
     <link name="franka_mount_link" />
     <xacro:include filename="$(find moma_description)/urdf/panda.xacro"/>
-    <xacro:panda connected_to="franka_mount_link"/>
+    <xacro:panda connected_to="franka_mount_link" include_gazebo_control="false"/>
 </robot>

Commit message: test admittance controller

File: moma_description/urdf/panda.xacro (robot description, xacro)
@@ -12,4 +12,13 @@
       <xacro:panda_hand_gazebo arm_id="panda"/>
     </xacro:if>
+    <xacro:unless value="${tool == 'panda_hand'}">
+      <!-- Add panda hand link if not added by previous block for consistency -->
+      <joint name="panda_hand_joint" type="fixed">
+        <parent link="panda_link8"/>
+        <child link="panda_hand"/>
+        <origin rpy="0 0 -0.785398163397" xyz="0 0 0"/>
+      </joint>
+      <link name="panda_hand"/>
+    </xacro:unless>
     <!-- robotiq 2f-85 -->
     <xacro:if value="${tool == 'robotiq_2f_85'}">

Commit message: Add fallback for tool frame

File: moma_description/urdf/panda.xacro (robot description, xacro)
@@ -5,4 +5,12 @@
     <xacro:include filename="$(find franka_description)/robots/panda_arm.xacro"/>
     <xacro:panda_arm connected_to="${connected_to}" rpy="${rpy}" xyz="${xyz}"/>
+    <!-- no tool frame -->
+    <xacro:if value="${tool == 'none' or tool == 'panda_hand'}">
+      <link name="tool_frame"/>
+      <joint name="tool_frame_joint" type="fixed">
+        <parent link="panda_link8"/>
+        <child link="tool_frame"/>
+      </joint>
+    </xacro:if>
     <!-- panda hand -->
     <xacro:if value="${tool == 'panda_hand'}">

Commit message: adding detection logic to piloting demo [wip]

File: moma_description/urdf/panda.xacro (robot description, xacro)
@@ -11,4 +11,5 @@
         <parent link="panda_link8"/>
         <child link="tool_frame"/>
+        <origin rpy="0 0 -0.785398163397" xyz="0 0 0.12"/>
       </joint>
     </xacro:if>

Commit message: camera info and topics also published in sim

File: moma_description/urdf/panda.xacro (robot description, xacro)
@@ -1,5 +1,6 @@
 <?xml version="1.0" encoding="utf-8"?>
 <robot xmlns:xacro="http://www.ros.org/wiki/xacro" name="panda">
-  <xacro:macro name="panda" params="connected_to:='' rpy:='0 0 0' xyz:='0 0 0' use_fixed_realsense:=false include_gazebo_control:=true tool:='panda_hand' control_mode:='Position' robot_namespace:='' control_namespace:=''">
+  <xacro:macro name="panda" params="connected_to:='' rpy:='0 0 0' xyz:='0 0 0' use_fixed_realsense:=false include_gazebo_control:=true
+    tool:='panda_hand' control_mode:='Position' robot_namespace:='' control_namespace:='' wrist_camera_name:='wrist_camera'">
     <!-- panda arm  -->
     <xacro:include filename="$(find franka_description)/robots/panda_arm.xacro"/>
@@ -58,8 +59,8 @@
     <xacro:include filename="$(find realsense2_description)/urdf/_d435.urdf.xacro" />
     <xacro:include filename="$(find moma_description)/urdf/realsense.gazebo.xacro" />
-    <xacro:realsense_gazebo_plugin camera_name="wrist_camera"/>
+    <xacro:realsense_gazebo_plugin camera_name="${wrist_camera_name}"/>
     <xacro:property name="panda_link7_camera_bottom_screw_frame_rpy" value="-2.68850999 -1.56973844 -1.20267232" />
     <xacro:property name="panda_link7_camera_bottom_screw_frame_xyz" value="0.06585917 -0.06861364 0.14820608" />
-    <xacro:sensor_d435 parent="panda_link7" name="wrist_camera">
+    <xacro:sensor_d435 parent="panda_link7" name="${wrist_camera_name}" use_nominal_extrinsics="true">
       <origin rpy="${panda_link7_camera_bottom_screw_frame_rpy}" xyz="${panda_link7_camera_bottom_screw_frame_xyz}" />
     </xacro:sensor_d435>

File: moma_description/urdf/superpanda.urdf.xacro (robot description, xacro)
@@ -71,4 +71,6 @@
   <xacro:arg name="control_mode" default='Position'/>
   <xacro:include filename="$(find moma_description)/urdf/panda.xacro"/>
-  <xacro:panda connected_to="arm_mount_link" use_fixed_realsense="$(arg use_fixed_realsense)" control_mode="$(arg control_mode)" tool="$(arg tool)" include_gazebo_control="true" robot_namespace="" control_namespace="control"/>
+  <xacro:panda connected_to="arm_mount_link" use_fixed_realsense="$(arg use_fixed_realsense)"
+    control_mode="$(arg control_mode)" tool="$(arg tool)" include_gazebo_control="true" robot_namespace=""
+    control_namespace="control" wrist_camera_name="hand_eye"/>
 </robot>

Commit message: Update camera calibration

File: moma_description/urdf/panda.xacro (robot description, xacro)
@@ -15,6 +15,6 @@
     <xacro:include filename="$(find moma_description)/urdf/realsense.gazebo.xacro" />
     <xacro:realsense_gazebo_plugin camera_name="wrist_camera"/>
-    <xacro:property name="panda_link7_camera_bottom_screw_frame_rpy" value="-2.68850999 -1.56973844 -1.20267232" />
-    <xacro:property name="panda_link7_camera_bottom_screw_frame_xyz" value="0.06585917 -0.06861364 0.14820608" />
+    <xacro:property name="panda_link7_camera_bottom_screw_frame_rpy" value="-0.5033 -1.566 2.865" />
+    <xacro:property name="panda_link7_camera_bottom_screw_frame_xyz" value="0.0256 -0.0246 0.1522" />
     <xacro:sensor_d435 parent="panda_link7" name="wrist_camera">
       <origin rpy="${panda_link7_camera_bottom_screw_frame_rpy}" xyz="${panda_link7_camera_bottom_screw_frame_xyz}" />

Commit message: bugs fixes

File: moma_description/urdf/panda.xacro (robot description, xacro)
@@ -1,5 +1,5 @@
 <?xml version="1.0" encoding="utf-8"?>
 <robot xmlns:xacro="http://www.ros.org/wiki/xacro" name="panda">
-  <xacro:macro name="panda" params="connected_to:='' rpy:='0 0 0' xyz:='0 0 0' use_fixed_realsense:=false tool:='panda_hand'">
+  <xacro:macro name="panda" params="connected_to:='' rpy:='0 0 0' xyz:='0 0 0' wrist_camera_name:='wrist_camera' use_fixed_realsense:=false tool:='panda_hand'">
     <!-- panda arm  -->
     <xacro:include filename="$(find franka_description)/robots/panda_arm.xacro"/>

Commit message: Updated descriptions

File: moma_description/urdf/panda.xacro (robot description, xacro)
@@ -1,7 +1,7 @@
 <?xml version="1.0" encoding="utf-8"?>
 <robot xmlns:xacro="http://www.ros.org/wiki/xacro" name="panda">
-  <xacro:macro name="moma_panda" params="use_fixed_realsense:=false use_nominal_extrinsics:=false">
+  <xacro:macro name="moma_panda" params="use_fixed_realsense:=false use_nominal_extrinsics:=false ">
     <!-- panda arm  -->
-    <xacro:include filename="$(find franka_description)/robots/panda_arm.urdf.xacro"/>
+    <xacro:include filename="$(find franka_description)/robots/panda_arm.urdf.xacro" />
     <!-- end effector frame for MoveIt -->
     <link name="panda_default_ee"/>

File: moma_description/urdf/realsense.gazebo.xacro (robot description, xacro)
@@ -3,5 +3,5 @@
   <xacro:macro name="realsense_gazebo_plugin" params="camera_name:=camera">
     <gazebo reference="${camera_name}_link">
-      <sensor type="depth" name="${camera_name}">
+      <sensor type="depth" name="depth">
         <always_on>true</always_on>
         <update_rate>30</update_rate>
@@ -18,5 +18,5 @@
           </clip>
         </camera>
-        <plugin filename="libgazebo_ros_openni_kinect.so" name="camera_plugin">
+        <plugin filename="libgazebo_ros_openni_kinect.so" name="depth_camera_plugin">
           <alwaysOn>true</alwaysOn>
           <!-- <baseline>0.2</baseline> -->

File: moma_description/urdf/royalpanda.urdf.xacro (robot description, xacro)
@@ -9,5 +9,4 @@
     </joint>
     <link name="franka_mount_link" />
-    <xacro:include filename="$(find moma_description)/urdf/panda.xacro"/>
-    <xacro:panda connected_to="franka_mount_link" include_gazebo_control="false"/>
+    <xacro:include filename="$(find moma_description)/urdf/panda.urdf.xacro"/>
 </robot>

Commit message: correct impedance controller params and panda_EE frame for real to sim transfer

File: moma_description/urdf/panda.xacro (robot description, xacro)
@@ -52,4 +52,11 @@
       <origin rpy="0.0 0.0 -0.785" xyz="0.0 0.0 0.103"/>
     </joint>
+    <!-- end effector as for the real hardware -->
+    <link name="panda_EE"/>
+    <joint name="joint_link8_panda_EE" type="fixed">
+      <parent link="panda_link8"/>
+      <child link="panda_EE"/>
+      <origin rpy="0.0 0.0 -0.785" xyz="0.0 0.0 0.103"/>
+    </joint>
     <!-- wrist realsense -->
     <xacro:include filename="$(find realsense2_description)/urdf/_d435.urdf.xacro" />

Commit message: Migrate from old franka_ros dependency to official one
The MPC pid gains need more tuning in sim

File: moma_description/urdf/panda.xacro (robot description, xacro)
@@ -1,8 +1,13 @@
 <?xml version="1.0" encoding="utf-8"?>
 <robot xmlns:xacro="http://www.ros.org/wiki/xacro" name="panda">
-  <xacro:macro name="panda" params="connected_to:='' rpy:='0 0 0' xyz:='0 0 0' use_fixed_realsense:=false
+  <xacro:macro name="panda" params="connected_to:='' rpy:='0 0 0' xyz:='0 0 0' sim:=false use_fixed_realsense:=false
     tool:='panda_hand' wrist_camera_name:='wrist_camera'">
     <!-- panda arm  -->
-    <xacro:include filename="$(find franka_description)/robots/panda_arm.xacro"/>
+    <xacro:if value="${sim}">
+        <xacro:include filename="$(find franka_description)/robots/panda_gazebo.xacro"/>
+    </xacro:if>
+    <xacro:unless value="${sim}">
+        <xacro:include filename="$(find franka_description)/robots/panda_arm.xacro"/>
+    </xacro:unless>
     <xacro:panda_arm connected_to="${connected_to}" rpy="${rpy}" xyz="${xyz}"/>
     <!-- no tool frame -->

File: moma_description/urdf/superpanda.urdf.xacro (robot description, xacro)
@@ -2,4 +2,5 @@
 <robot xmlns:xacro="http://www.ros.org/wiki/xacro" name="superpanda">
   <!-- Panda Arguments -->
+  <xacro:arg name="sim" default="false"/>
   <xacro:arg name="use_fixed_realsense" default="false"/>
   <xacro:arg name="tool" default="panda_hand"/>
@@ -62,4 +63,5 @@
   <xacro:panda
     connected_to="arm_mount_link"
+    sim="$(arg sim)"
     use_fixed_realsense="$(arg use_fixed_realsense)"
     wrist_camera_name="$(arg wrist_camera_name)"
