Commit message: b4 master changes update

File: moma_description/urdf/giraffe.gazebo.xacro (robot description, xacro)
@@ -8,5 +8,5 @@
     <link name="base_footprint" />
     <joint name="base_joint" type="fixed">
-        <origin rpy="0 0 0" xyz="0 0 0.0" />
+        <origin rpy="0 0 0" xyz="0 0 0" />
         <parent link="base_link" />
         <child link="body_link" />

File: moma_description/urdf/giraffe.urdf.xacro (robot description, xacro)
@@ -22,4 +22,5 @@
                       use_fixed_camera="$(arg use_fixed_camera)"
                       use_wrist_camera="$(arg use_wrist_camera)"
+                      use_bota="$(arg use_bota)"
                       include_control_plugin="true"/>
 </robot>

File: moma_description/urdf/panda_arm.xacro (robot description, xacro)
@@ -1,4 +1,4 @@
 <?xml version='1.0' encoding='utf-8'?>
-<robot xmlns:xacro="http://www.ros.org/wiki/xacro">
+<robot xmlns:xacro="http://www.ros.org/wiki/xacro" name="panda">
   <!-- Adapted from franka_description/robots/common/franka_robot.xacro -->
   <xacro:macro name="moma_panda"
@@ -24,5 +24,4 @@
     <xacro:include filename="$(find franka_description)/robots/common/utils.xacro" />
     <xacro:include filename="$(find franka_description)/robots/common/franka_arm.xacro" />
-    <index xyz="1 2 3" rpy="1 2 3"/>
     <!-- Put in a basic arm. -->
     <xacro:franka_arm arm_id="${arm_id}" safety_distance="0.03" gazebo="${gazebo}"
