Commit message: moveit assistant for giraffe

File: moma_description/urdf/giraffe.urdf.xacro (robot description, xacro)
@@ -1,17 +1,25 @@
 <?xml version="1.0" encoding="utf-8"?>
 <robot xmlns:xacro="http://www.ros.org/wiki/xacro" name="giraffe">
-    <!-- <xacro:include filename="$(find gmp_robot)/config/urdf/gmp.urdf"/> -->
+    <xacro:arg name="use_fixed_camera" default="false" />
+    <xacro:arg name="use_wrist_camera" default="true" />
+    <xacro:arg name="use_bota" default="false" />
+    <xacro:arg name="load_gripper" default="true" />
+    <xacro:arg name="gazebo" default="true" />
+    <xacro:arg name="arm_id" default="panda" />
+    <xacro:include filename="$(find gmp_robot)/config/urdf/gmp.urdf"/>
     <!-- add link in z-link -->
     <link name="franka_mount_link"/>
-    <!-- <joint name="arm_mount_joint" type="fixed"> -->
-        <!-- <parent link="z_axis_link"/> -->
-        <!-- <child link="franka_mount_link"/> -->
-        <!-- <origin xyz="0.0 0.3 0.3345" rpy="0 0 0" /> -->
-    <!-- </joint> -->
+    <joint name="arm_mount_joint" type="fixed">
+        <parent link="z_axis_link"/>
+        <child link="franka_mount_link"/>
+        <origin xyz="-0.285 0.0 0.0325" rpy="0 0 3.141" />
+    </joint>
     <xacro:include filename="$(find moma_description)/urdf/panda_arm.xacro"/>
-    <xacro:moma_panda gazebo="true"
-                      fixed_to_world="false"
+    <xacro:moma_panda gazebo="$(arg gazebo)"
                       parent="franka_mount_link"
-                      use_wrist_camera="true"
+                      hand="$(arg load_gripper)"
+                      arm_id="$(arg arm_id)"
+                      use_fixed_camera="$(arg use_fixed_camera)"
+                      use_wrist_camera="$(arg use_wrist_camera)"
                       include_control_plugin="true"/>
 </robot>

File: moma_description/urdf/panda_arm.xacro (robot description, xacro)
@@ -3,5 +3,6 @@
   <!-- Adapted from franka_description/robots/common/franka_robot.xacro -->
   <xacro:macro name="moma_panda"
-    params="arm_id:='panda'
+    params="
+        arm_id:='panda'
         parent:='world'
         xyz:='0 0 0'
@@ -11,8 +12,6 @@
         hand:=true
         gazebo:=false
-        fixed_to_world:=false
         use_wrist_camera:=false
         wrist_calibration_rpy:='-1.117916 -1.5611535 -2.8045692'
-        wrist_calibration_xyz:='0.03062033586096833 -0.025020246008959142 0.10095534939725603'
         wrist_camera_parent_link:='panda_link8'
         use_fixed_camera:=false
@@ -25,18 +24,16 @@
     <xacro:include filename="$(find franka_description)/robots/common/utils.xacro" />
     <xacro:include filename="$(find franka_description)/robots/common/franka_arm.xacro" />
+    <index xyz="1 2 3" rpy="1 2 3"/>
     <!-- Put in a basic arm. -->
-    <xacro:franka_arm arm_id="${arm_id}"
-        connected_to="${parent}"
-        xyz="${xyz}"
-        rpy="${rpy}"
-        safety_distance="0.03"
-        gazebo="${gazebo}"
-        joint_limits="${xacro.load_yaml('$(find franka_description)/robots/panda/joint_limits.yaml')}" />
-    <!-- Offset the hand if we have a bota sensor. -->
+    <xacro:franka_arm arm_id="${arm_id}" safety_distance="0.03" gazebo="${gazebo}"
+      joint_limits="${xacro.load_yaml('$(find franka_description)/robots/panda/joint_limits.yaml')}" />
+    <!-- Offset the hand if we have a bota sensor. Make sure to change this if you calibrate the wrist camera! -->
     <xacro:if value="${use_bota}">
       <xacro:property name="hand_xyz" value="0 0 0.035"/>
+      <xacro:property name="wrist_calibration_xyz" value='0.03062033586096833 -0.025020246008959142 0.10095534939725603'/>
     </xacro:if>
     <xacro:unless value="${use_bota}">
       <xacro:property name="hand_xyz" value="0 0 0"/>
+      <xacro:property name="wrist_calibration_xyz" value='0.03062033586096833 -0.025020246008959142 0.04595534939725603'/>
     </xacro:unless>
     <!-- Put in a basic hand. -->

Commit message: giraffe moveit config, works in sim

File: moma_description/urdf/giraffe.urdf.xacro (robot description, xacro)
@@ -1,26 +1,27 @@
 <?xml version="1.0" encoding="utf-8"?>
 <robot xmlns:xacro="http://www.ros.org/wiki/xacro" name="giraffe">
-    <xacro:arg name="use_fixed_camera" default="false" />
-    <xacro:arg name="use_wrist_camera" default="true" />
-    <xacro:arg name="use_bota" default="false" />
-    <xacro:arg name="load_gripper" default="true" />
-    <xacro:arg name="gazebo" default="true" />
-    <xacro:arg name="arm_id" default="panda" />
-    <xacro:include filename="$(find gmp_robot)/config/urdf/gmp.urdf"/>
-    <!-- add link in z-link -->
-    <link name="franka_mount_link"/>
-    <joint name="arm_mount_joint" type="fixed">
-        <parent link="z_axis_link"/>
-        <child link="franka_mount_link"/>
-        <origin xyz="-0.285 0.0 0.0325" rpy="0 0 3.141" />
-    </joint>
-    <xacro:include filename="$(find moma_description)/urdf/panda_arm.xacro"/>
-    <xacro:moma_panda gazebo="$(arg gazebo)"
-                      parent="franka_mount_link"
-                      hand="$(arg load_gripper)"
-                      arm_id="$(arg arm_id)"
-                      use_fixed_camera="$(arg use_fixed_camera)"
-                      use_wrist_camera="$(arg use_wrist_camera)"
-                      use_bota="$(arg use_bota)"
-                      include_control_plugin="true"/>
+  <xacro:arg name="use_fixed_camera" default="false" />
+  <xacro:arg name="use_wrist_camera" default="true" />
+  <xacro:arg name="use_bota" default="false" />
+  <xacro:arg name="load_gripper" default="true" />
+  <xacro:arg name="gazebo" default="true" />
+  <xacro:arg name="arm_id" default="panda" />
+  <!-- <xacro:arg name="use_nominal_extrinsics" default="false"/> -->
+  <xacro:include filename="$(find gmp_robot)/config/urdf/gmp.xacro"/>
+  <xacro:gmp include_control_plugin="true" multiple_robots="true"/>
+  <link name="franka_mount_link"/>
+  <joint name="arm_mount_joint" type="fixed">
+    <parent link="z_axis_link"/>
+    <child link="franka_mount_link"/>
+    <origin xyz="-0.285 0.0 0.03" rpy="0 0 3.141"/>
+  </joint>
+  <xacro:include filename="$(find moma_description)/urdf/panda_arm.xacro"/>
+  <xacro:moma_panda gazebo="$(arg gazebo)"
+    parent="franka_mount_link"
+    hand="$(arg load_gripper)"
+    arm_id="$(arg arm_id)"
+    use_fixed_camera="$(arg use_fixed_camera)"
+    use_wrist_camera="$(arg use_wrist_camera)"
+    use_bota="$(arg use_bota)"
+    include_control_plugin="true"/>
 </robot>

File: moma_description/urdf/panda_arm.xacro (robot description, xacro)
@@ -4,23 +4,23 @@
   <xacro:macro name="moma_panda"
     params="
-        arm_id:='panda'
-        parent:='world'
-        xyz:='0 0 0'
-        rpy:='0 0 0'
-        tcp_xyz:='0 0 0.1034'
-        tcp_rpy='0 0 0'
-        hand:=true
-        gazebo:=false
-        use_wrist_camera:=false
-        wrist_calibration_rpy:='-0.0109077 -1.5469874 2.3727493'
-        wrist_calibration_xyz:='0.02144228129647578 -0.028987519327164604 0.04877543953719046'
-        wrist_camera_parent_link:='panda_link8'
-        use_fixed_camera:=false
-        fixed_calibration_rpy:='-0.1566281 1.3870703 2.9725147'
-        fixed_calibration_xyz:='0.890 -0.162 1.293'
-        fixed_camera_parent_link:='panda_link0'
-        use_bota:=false
-        include_control_plugin:=true,
-        publish_realsense_extrinsics:=true">
+    arm_id:='panda'
+    parent:='world'
+    xyz:='0 0 0'
+    rpy:='0 0 0'
+    tcp_xyz:='0 0 0.1034'
+    tcp_rpy='0 0 0'
+    hand:=true
+    gazebo:=false
+    use_wrist_camera:=false
+    wrist_calibration_rpy:='-0.0109077 -1.5469874 2.3727493'
+    wrist_calibration_xyz:='0.02144228129647578 -0.028987519327164604 0.04877543953719046'
+    wrist_camera_parent_link:='panda_link8'
+    use_fixed_camera:=false
+    fixed_calibration_rpy:='-0.1566281 1.3870703 2.9725147'
+    fixed_calibration_xyz:='0.890 -0.162 1.293'
+    fixed_camera_parent_link:='panda_link0'
+    use_bota:=false
+    include_control_plugin:=true,
+    publish_realsense_extrinsics:=true">
     <xacro:include filename="$(find franka_description)/robots/common/utils.xacro" />
     <xacro:include filename="$(find franka_description)/robots/common/franka_arm.xacro" />
@@ -46,6 +46,5 @@
         connected_to="${arm_id}_link8"
         safety_distance="0.03"
-        gazebo="${gazebo}"
-      />
+        gazebo="${gazebo}" />
     </xacro:if>
     <!-- wrist realsense -->
@@ -128,6 +127,5 @@
       <xacro:transmission-franka-model arm_id="${arm_id}"
         root="${arm_id}_joint1"
-        tip="${arm_id}_joint8"
-      />
+        tip="${arm_id}_joint8" />
       <xacro:if value="${hand}">
         <xacro:gazebo-joint joint="${arm_id}_finger_joint1"
@@ -135,5 +133,5 @@
         <xacro:gazebo-joint joint="${arm_id}_finger_joint2"
           transmission="hardware_interface/EffortJointInterface" />
-        <!-- Friction specific material for Rubber/Rubber contact -->
+          <!-- Friction specific material for Rubber/Rubber contact -->
         <xacro:gazebo-friction link="${arm_id}_leftfinger" mu="1.13" />
         <xacro:gazebo-friction link="${arm_id}_rightfinger" mu="1.13" />
@@ -144,4 +142,7 @@
             <controlPeriod>0.001</controlPeriod>
             <robotSimType>franka_gazebo/FrankaHWSim</robotSimType>
+            <robotNamespace>/panda</robotNamespace>
+            <robotParam>robot_description_arm</robotParam>
+            <robotDescription>robot_description_arm</robotDescription>
           </plugin>
           <self_collide>true</self_collide>
@@ -149,4 +150,11 @@
       </xacro:if>
     </xacro:if>
+    <!-- end effector frame for MoveIt -->
+    <link name="${arm_id}_default_ee"/>
+    <joint name="joint_link8_default_ee" type="fixed">
+      <parent link="${arm_id}_link8"/>
+      <child link="${arm_id}_default_ee"/>
+      <origin rpy="0.0 0.0 -0.785" xyz="0.0 0.0 0.103"/>
+    </joint>
   </xacro:macro>
 </robot>
