Commit message: added table to URDF to avoid collisions with it

File: moma_description/urdf/panda.urdf.xacro (robot description, xacro)
@@ -4,3 +4,29 @@
   <xacro:include filename="$(find moma_description)/urdf/panda.xacro"/>
   <xacro:panda connected_to="base_link"/>
+  <!-- Add a table to avoid collisions with it -->
+  <link name="table_link">
+    <inertial>
+      <origin xyz="0 0 0.5" rpy="0 0 0"/>
+      <mass value="1"/>
+      <inertia ixx="100"  ixy="0"  ixz="0" iyy="100" iyz="0" izz="100" />
+    </inertial>
+    <visual>
+      <geometry>
+        <box size="1.0 0.8 0.3" />
+      </geometry>
+      <material name="magic">
+        <color rgba="0 0.625 0.625 0.625"/>
+      </material>
+    </visual>
+    <collision>
+      <geometry>
+        <box size="1.0 0.8 0.3" />
+      </geometry>
+    </collision>
+ </link>
+ <joint name="table_joint" type="fixed">
+    <parent link="base_link"/>
+    <child link="table_link"/>
+    <origin rpy="0.0 0.0 0.0" xyz="0.65 0.0 0.0"/>
+  </joint>
 </robot>

Commit message: Unified launch file for gazebo.

File: moma_description/urdf/panda.urdf.xacro (robot description, xacro)
@@ -1,32 +1,6 @@
 <?xml version="1.0" encoding="utf-8"?>
 <robot xmlns:xacro="http://www.ros.org/wiki/xacro" name="panda">
-  <link name="base_link"/>
+  <link name="world" />
   <xacro:include filename="$(find moma_description)/urdf/panda.xacro"/>
-  <xacro:panda connected_to="base_link"/>
-  <!-- Add a table to avoid collisions with it -->
-  <link name="table_link">
-    <inertial>
-      <origin xyz="0 0 0.5" rpy="0 0 0"/>
-      <mass value="1"/>
-      <inertia ixx="100"  ixy="0"  ixz="0" iyy="100" iyz="0" izz="100" />
-    </inertial>
-    <visual>
-      <geometry>
-        <box size="1.0 0.8 0.3" />
-      </geometry>
-      <material name="magic">
-        <color rgba="0 0.625 0.625 0.625"/>
-      </material>
-    </visual>
-    <collision>
-      <geometry>
-        <box size="1.0 0.8 0.3" />
-      </geometry>
-    </collision>
- </link>
- <joint name="table_joint" type="fixed">
-    <parent link="base_link"/>
-    <child link="table_link"/>
-    <origin rpy="0.0 0.0 0.0" xyz="0.65 0.0 0.0"/>
-  </joint>
+  <xacro:panda connected_to="world"/>
 </robot>

Commit message: Fixed panda.

File: moma_description/urdf/panda.urdf.xacro (robot description, xacro)
@@ -4,3 +4,35 @@
   <xacro:include filename="$(find moma_description)/urdf/panda.xacro"/>
   <xacro:panda connected_to="world"/>
+  <gazebo>
+    <plugin name="gazebo_ros_control" filename="libgazebo_ros_control.so">
+      <robotNamespace>/</robotNamespace>
+    </plugin>
+  </gazebo>
+  <!-- NOTE from Julien: Recommending to spawn a table separately, not here -->
+  <!-- Add a table to avoid collisions with it -->
+  <!-- <link name="table_link">
+    <inertial>
+      <origin xyz="0 0 0.5" rpy="0 0 0"/>
+      <mass value="1"/>
+      <inertia ixx="100"  ixy="0"  ixz="0" iyy="100" iyz="0" izz="100" />
+    </inertial>
+    <visual>
+      <geometry>
+        <box size="1.0 0.8 0.3" />
+      </geometry>
+      <material name="magic">
+        <color rgba="0 0.625 0.625 0.625"/>
+      </material>
+    </visual>
+    <collision>
+      <geometry>
+        <box size="1.0 0.8 0.3" />
+      </geometry>
+    </collision>
+ </link>
+ <joint name="table_joint" type="fixed">
+    <parent link="world"/>
+    <child link="table_link"/>
+    <origin rpy="0.0 0.0 0.0" xyz="0.65 0.0 0.0"/>
+  </joint> -->
 </robot>

File: moma_description/urdf/yumi.urdf.xacro (robot description, xacro)
@@ -4,3 +4,11 @@
   <xacro:include filename="$(find moma_description)/urdf/yumi.xacro"/>
   <xacro:yumi connected_to="base_link"/>
+  <!-- NOTE: franka_ros did not include gazebo tag for roscontrol plugin, it might be that
+  including this tag is necessary for yumi as well (in case that the arm just drop
+  even if the controllers were spawned with the controller manager).
+  <gazebo>
+    <plugin name="gazebo_ros_control" filename="libgazebo_ros_control.so">
+      <robotNamespace>/</robotNamespace>
+    </plugin>
+  </gazebo> -->
 </robot>

Commit message: Minor

File: moma_description/urdf/panda.urdf.xacro (robot description, xacro)
@@ -7,5 +7,5 @@
   <link name="table_link">
     <inertial>
-      <origin xyz="0 0 0.5" rpy="0 0 0"/>
+      <origin xyz="0 0 0" rpy="0 0 0"/>
       <mass value="1"/>
       <inertia ixx="100"  ixy="0"  ixz="0" iyy="100" iyz="0" izz="100" />
@@ -13,5 +13,5 @@
     <visual>
       <geometry>
-        <box size="1.0 0.8 0.3" />
+        <box size="1.0 0.8 0.07" />
       </geometry>
       <material name="magic">
@@ -21,5 +21,5 @@
     <collision>
       <geometry>
-        <box size="1.0 0.8 0.3" />
+        <box size="1.0 0.8 0.07" />
       </geometry>
     </collision>

Commit message: Removed table from panda xacro

File: moma_description/urdf/panda.urdf.xacro (robot description, xacro)
@@ -4,29 +4,3 @@
   <xacro:include filename="$(find moma_description)/urdf/panda.xacro"/>
   <xacro:panda connected_to="base_link"/>
-  <!-- Add a table to avoid collisions with it -->
-  <link name="table_link">
-    <inertial>
-      <origin xyz="0 0 0" rpy="0 0 0"/>
-      <mass value="1"/>
-      <inertia ixx="100"  ixy="0"  ixz="0" iyy="100" iyz="0" izz="100" />
-    </inertial>
-    <visual>
-      <geometry>
-        <box size="1.0 0.8 0.07" />
-      </geometry>
-      <material name="magic">
-        <color rgba="0 0.625 0.625 0.625"/>
-      </material>
-    </visual>
-    <collision>
-      <geometry>
-        <box size="1.0 0.8 0.07" />
-      </geometry>
-    </collision>
- </link>
- <joint name="table_joint" type="fixed">
-    <parent link="base_link"/>
-    <child link="table_link"/>
-    <origin rpy="0.0 0.0 0.0" xyz="0.65 0.0 0.0"/>
-  </joint>
 </robot>

Commit message: Gazebo simulation of joint position controlled panda

File: moma_description/urdf/panda.urdf.xacro (robot description, xacro)
@@ -1,6 +1,11 @@
 <?xml version="1.0" encoding="utf-8"?>
 <robot xmlns:xacro="http://www.ros.org/wiki/xacro" name="panda">
-  <link name="base_link"/>
   <xacro:include filename="$(find moma_description)/urdf/panda.xacro"/>
-  <xacro:panda connected_to="base_link"/>
+  <link name="world"/>
+  <xacro:panda connected_to="world"/>
+  <gazebo>
+    <plugin name="gazebo_ros_control" filename="libgazebo_ros_control.so">
+      <robotNamespace>/</robotNamespace>
+    </plugin>
+  </gazebo>
 </robot>

Commit message: Missing base_link added
Otherwise point cloud would not show up in rviz

File: moma_description/urdf/panda.urdf.xacro (robot description, xacro)
@@ -3,5 +3,11 @@
   <xacro:include filename="$(find moma_description)/urdf/panda.xacro"/>
   <link name="world"/>
-  <xacro:panda connected_to="world"/>
+  <link name="base_link"/>
+  <joint name="base_link_joint" type="fixed">
+    <parent link="world"/>
+    <child link="base_link"/>
+    <origin rpy="0 0 0" xyz="0 0 0"/>
+  </joint>
+  <xacro:panda connected_to="base_link"/>
   <gazebo>
     <plugin name="gazebo_ros_control" filename="libgazebo_ros_control.so">

Commit message: flag that can be used to spawn an external camera

File: moma_description/urdf/panda.urdf.xacro (robot description, xacro)
@@ -1,4 +1,5 @@
 <?xml version="1.0" encoding="utf-8"?>
 <robot xmlns:xacro="http://www.ros.org/wiki/xacro" name="panda">
+  <xacro:arg name="use_fixed_realsense" default="false"/>
   <xacro:include filename="$(find moma_description)/urdf/panda.xacro"/>
   <link name="world"/>
@@ -9,5 +10,5 @@
     <origin rpy="0 0 0" xyz="0 0 0"/>
   </joint>
-  <xacro:panda connected_to="base_link"/>
+  <xacro:panda connected_to="base_link" use_fixed_realsense="$(arg use_fixed_realsense)"/>
   <gazebo>
     <plugin name="gazebo_ros_control" filename="libgazebo_ros_control.so">

File: moma_description/urdf/panda.xacro (robot description, xacro)
@@ -1,5 +1,5 @@
 <?xml version="1.0" encoding="utf-8"?>
 <robot xmlns:xacro="http://www.ros.org/wiki/xacro" name="panda">
-  <xacro:macro name="panda" params="connected_to:='' rpy:='0 0 0' xyz:='0 0 0'">
+  <xacro:macro name="panda" params="connected_to:='' rpy:='0 0 0' xyz:='0 0 0' use_fixed_realsense:=false">
     <!-- panda arm  -->
     <xacro:include filename="$(find franka_description)/robots/panda_arm.xacro"/>
@@ -24,5 +24,5 @@
       </plugin>
     </gazebo>
-    <!-- realsense -->
+    <!-- wrist realsense -->
     <xacro:include filename="$(find realsense2_description)/urdf/_d435.urdf.xacro" />
     <xacro:include filename="$(find moma_description)/urdf/realsense.gazebo.xacro" />
@@ -33,4 +33,13 @@
       <origin rpy="${panda_link7_camera_bottom_screw_frame_rpy}" xyz="${panda_link7_camera_bottom_screw_frame_xyz}" />
     </xacro:sensor_d435>
+    <!-- fixed realsense -->
+    <xacro:if value="${use_fixed_realsense}">
+      <xacro:realsense_gazebo_plugin camera_name="fixed_camera"/>
+      <xacro:property name="base_link_camera_bottom_screw_frame_rpy" value="0 0.79 -0.79" />
+      <xacro:property name="base_link_camera_bottom_screw_frame_xyz" value="0.1 0.75 0.9" />
+      <xacro:sensor_d435 parent="base_link" name="fixed_camera">
+        <origin rpy="${base_link_camera_bottom_screw_frame_rpy}" xyz="${base_link_camera_bottom_screw_frame_xyz}" />
+      </xacro:sensor_d435>
+    </xacro:if>
   </xacro:macro>
 </robot>

Commit message: sync with tree: grasp-demo-gazebo for dual camera

File: moma_description/urdf/panda.urdf.xacro (robot description, xacro)
@@ -1,4 +1,5 @@
 <?xml version="1.0" encoding="utf-8"?>
 <robot xmlns:xacro="http://www.ros.org/wiki/xacro" name="panda">
+  <xacro:arg name="use_fixed_realsense" default="false"/>
   <xacro:include filename="$(find moma_description)/urdf/panda.xacro"/>
   <link name="world"/>
@@ -9,5 +10,5 @@
     <origin rpy="0 0 0" xyz="0 0 0"/>
   </joint>
-  <xacro:panda connected_to="base_link"/>
+   <xacro:panda connected_to="base_link" use_fixed_realsense="$(arg use_fixed_realsense)"/>
   <gazebo>
     <plugin name="gazebo_ros_control" filename="libgazebo_ros_control.so">

File: moma_description/urdf/panda.xacro (robot description, xacro)
@@ -1,5 +1,5 @@
 <?xml version="1.0" encoding="utf-8"?>
 <robot xmlns:xacro="http://www.ros.org/wiki/xacro" name="panda">
-  <xacro:macro name="panda" params="connected_to:='' rpy:='0 0 0' xyz:='0 0 0'">
+   <xacro:macro name="panda" params="connected_to:='' rpy:='0 0 0' xyz:='0 0 0' use_fixed_realsense:=false">
     <!-- panda arm  -->
     <xacro:include filename="$(find franka_description)/robots/panda_arm.xacro"/>
@@ -24,12 +24,22 @@
       </plugin>
     </gazebo>
-    <!-- realsense -->
+     <!-- wrist realsense -->
     <xacro:include filename="$(find realsense2_description)/urdf/_d435.urdf.xacro" />
     <xacro:include filename="$(find moma_description)/urdf/realsense.gazebo.xacro" />
+    <xacro:realsense_gazebo_plugin camera_name="wrist_camera"/>
     <xacro:property name="panda_link7_camera_bottom_screw_frame_rpy" value="-2.68850999 -1.56973844 -1.20267232" />
     <xacro:property name="panda_link7_camera_bottom_screw_frame_xyz" value="0.06585917 -0.06861364 0.14820608" />
-    <xacro:sensor_d435 parent="panda_link7">
+     <xacro:sensor_d435 parent="panda_link7" name="wrist_camera">
       <origin rpy="${panda_link7_camera_bottom_screw_frame_rpy}" xyz="${panda_link7_camera_bottom_screw_frame_xyz}" />
     </xacro:sensor_d435>
+    <!-- fixed realsense -->
+    <xacro:if value="${use_fixed_realsense}">
+      <xacro:realsense_gazebo_plugin camera_name="fixed_camera"/>
+      <xacro:property name="base_link_camera_bottom_screw_frame_rpy" value="0 0.79 -0.79" />
+      <xacro:property name="base_link_camera_bottom_screw_frame_xyz" value="0.1 0.75 0.9" />
+      <xacro:sensor_d435 parent="base_link" name="fixed_camera">
+        <origin rpy="${base_link_camera_bottom_screw_frame_rpy}" xyz="${base_link_camera_bottom_screw_frame_xyz}" />
+      </xacro:sensor_d435>
+    </xacro:if>
   </xacro:macro>
 </robot>

File: moma_description/urdf/realsense.gazebo.xacro (robot description, xacro)
@@ -1,40 +1,42 @@
 <?xml version='1.0' encoding='utf-8'?>
 <robot xmlns:xacro="http://www.ros.org/wiki/xacro" name="realsense">
-  <gazebo reference="camera_link">
-    <sensor type="depth" name="camera">
-      <always_on>true</always_on>
-      <update_rate>30</update_rate>
-      <camera>
-        <horizontal_fov>0.976899239</horizontal_fov>
-        <image>
-          <format>R8G8B8</format>
-          <width>640</width>
-          <height>480</height>
-        </image>
-        <clip>
-          <near>0.1</near>
-          <far>10</far>
-        </clip>
-      </camera>
-      <plugin filename="libgazebo_ros_openni_kinect.so" name="camera_plugin">
-        <alwaysOn>true</alwaysOn>
-        <!-- <baseline>0.2</baseline> -->
-        <updateRate>0.0</updateRate>
-        <cameraName>camera</cameraName>
-        <imageTopicName>/camera/color/image_raw</imageTopicName>
-        <cameraInfoTopicName>/camera/color/camera_info</cameraInfoTopicName>
-        <depthImageTopicName>/camera/depth/image_rect_raw</depthImageTopicName>
-        <depthImageCameraInfoTopicName>/camera/depth/camera_info</depthImageCameraInfoTopicName>
-        <pointCloudTopicName>/camera/depth/color/points</pointCloudTopicName>
-        <frameName>camera_depth_optical_frame</frameName>
-        <pointCloudCutoff>0.1</pointCloudCutoff>
-        <pointCloudCutoffMax>10</pointCloudCutoffMax>
-        <distortionK1>0</distortionK1>
-        <distortionK2>0</distortionK2>
-        <distortionK3>0</distortionK3>
-        <distortionT1>0</distortionT1>
-        <distortionT2>0</distortionT2>
-      </plugin>
-    </sensor>
-  </gazebo>
+ <xacro:macro name="realsense_gazebo_plugin" params="camera_name:=camera">
+    <gazebo reference="${camera_name}_link">
+      <sensor type="depth" name="${camera_name}">
+        <always_on>true</always_on>
+        <update_rate>30</update_rate>
+        <camera>
+          <horizontal_fov>0.976899239</horizontal_fov>
+          <image>
+            <format>R8G8B8</format>
+            <width>640</width>
+            <height>480</height>
+          </image>
+          <clip>
+            <near>0.1</near>
+            <far>10</far>
+          </clip>
+        </camera>
+        <plugin filename="libgazebo_ros_openni_kinect.so" name="camera_plugin">
+          <alwaysOn>true</alwaysOn>
+          <!-- <baseline>0.2</baseline> -->
+          <updateRate>0.0</updateRate>
+          <cameraName>${camera_name}</cameraName>
+          <imageTopicName>/${camera_name}/color/image_raw</imageTopicName>
+          <cameraInfoTopicName>/${camera_name}/color/camera_info</cameraInfoTopicName>
+          <depthImageTopicName>/${camera_name}/depth/image_rect_raw</depthImageTopicName>
+          <depthImageCameraInfoTopicName>/${camera_name}/depth/camera_info</depthImageCameraInfoTopicName>
+          <pointCloudTopicName>/${camera_name}/depth/color/points</pointCloudTopicName>
+          <frameName>${camera_name}_depth_optical_frame</frameName>
+          <pointCloudCutoff>0.1</pointCloudCutoff>
+          <pointCloudCutoffMax>10</pointCloudCutoffMax>
+          <distortionK1>0</distortionK1>
+          <distortionK2>0</distortionK2>
+          <distortionK3>0</distortionK3>
+          <distortionT1>0</distortionT1>
+          <distortionT2>0</distortionT2>
+        </plugin>
+      </sensor>
+    </gazebo>
+  </xacro:macro>
 </robot>

Commit message: panda example in gazebo now working

File: moma_description/urdf/panda.urdf.xacro (robot description, xacro)
@@ -11,8 +11,3 @@
   </joint>
   <xacro:panda connected_to="base_link" use_fixed_realsense="$(arg use_fixed_realsense)"/>
-  <gazebo>
-    <plugin name="gazebo_ros_control" filename="libgazebo_ros_control.so">
-      <robotNamespace>/</robotNamespace>
-    </plugin>
-  </gazebo>
 </robot>

File: moma_description/urdf/panda.xacro (robot description, xacro)
@@ -15,13 +15,7 @@
       <origin rpy="0.0 0.0 -0.785" xyz="0.0 0.0 0.103"/>
     </joint>
-    <!-- gazebo plugin to mimic finger joints -->
-    <gazebo>
-      <plugin name="panda_hand_mimic_joint_plugin" filename="libroboticsgroup_gazebo_mimic_joint_plugin.so">
-        <joint>panda_finger_joint1</joint>
-        <mimicJoint>panda_finger_joint2</mimicJoint>
-        <hasPID></hasPID>
-        <multiplier>2.0</multiplier>
-      </plugin>
-    </gazebo>
+    <!-- Gazebo Tags -->
+    <xacro:include filename="$(find franka_description)/robots/panda_arm.gazebo.xacro"/>
+    <xacro:panda_gazebo arm_id="panda"/>
     <!-- wrist realsense -->
     <xacro:include filename="$(find realsense2_description)/urdf/_d435.urdf.xacro" />

Commit message: Updated franka ros

File: moma_description/urdf/panda.urdf.xacro (robot description, xacro)
@@ -11,8 +11,3 @@
   </joint>
   <xacro:panda connected_to="base_link" use_fixed_realsense="$(arg use_fixed_realsense)"/>
-  <gazebo>
-    <plugin name="gazebo_ros_control" filename="libgazebo_ros_control.so">
-      <robotNamespace>/</robotNamespace>
-    </plugin>
-  </gazebo>
 </robot>

File: moma_description/urdf/panda.xacro (robot description, xacro)
@@ -15,13 +15,7 @@
       <origin rpy="0.0 0.0 -0.785" xyz="0.0 0.0 0.103"/>
     </joint>
-    <!-- gazebo plugin to mimic finger joints -->
-    <gazebo>
-      <plugin name="panda_hand_mimic_joint_plugin" filename="libroboticsgroup_gazebo_mimic_joint_plugin.so">
-        <joint>panda_finger_joint1</joint>
-        <mimicJoint>panda_finger_joint2</mimicJoint>
-        <hasPID></hasPID>
-        <multiplier>2.0</multiplier>
-      </plugin>
-    </gazebo>
+    <!-- Gazebo tags -->
+    <xacro:include filename="$(find franka_description)/robots/panda_arm.gazebo.xacro"/>
+    <xacro:panda_gazebo arm_id="panda"/>
     <!-- wrist realsense -->
     <xacro:include filename="$(find realsense2_description)/urdf/_d435.urdf.xacro" />

Commit message: flexible control interface

File: moma_description/urdf/panda.urdf.xacro (robot description, xacro)
@@ -2,4 +2,5 @@
 <robot xmlns:xacro="http://www.ros.org/wiki/xacro" name="panda">
   <xacro:arg name="use_fixed_realsense" default="false"/>
+  <xacro:arg name="control_mode" default='Position'/>
   <xacro:include filename="$(find moma_description)/urdf/panda.xacro"/>
   <link name="world"/>
@@ -10,4 +11,4 @@
     <origin rpy="0 0 0" xyz="0 0 0"/>
   </joint>
-  <xacro:panda connected_to="base_link" use_fixed_realsense="$(arg use_fixed_realsense)"/>
+  <xacro:panda connected_to="base_link" use_fixed_realsense="$(arg use_fixed_realsense)" control_mode="$(arg control_mode)"/>
 </robot>

File: moma_description/urdf/panda.xacro (robot description, xacro)
@@ -1,5 +1,5 @@
 <?xml version="1.0" encoding="utf-8"?>
 <robot xmlns:xacro="http://www.ros.org/wiki/xacro" name="panda">
-  <xacro:macro name="panda" params="connected_to:='' rpy:='0 0 0' xyz:='0 0 0' use_fixed_realsense:=false include_gazebo_control:=true">
+  <xacro:macro name="panda" params="connected_to:='' rpy:='0 0 0' xyz:='0 0 0' use_fixed_realsense:=false include_gazebo_control:=true control_mode:='Position'">
     <!-- panda arm  -->
     <xacro:include filename="$(find franka_description)/robots/panda_arm.xacro"/>
@@ -17,5 +17,5 @@
     <!-- Gazebo tags -->
     <xacro:include filename="$(find moma_description)/urdf/panda_arm.gazebo.xacro"/>
-    <xacro:panda_gazebo arm_id="panda" include_gazebo_control="${include_gazebo_control}"/>
+    <xacro:panda_gazebo arm_id="panda" include_gazebo_control="${include_gazebo_control}" control_mode="${control_mode}"/>
     <!-- wrist realsense -->
     <xacro:include filename="$(find realsense2_description)/urdf/_d435.urdf.xacro" />

File: moma_description/urdf/panda_arm.gazebo.xacro (robot description, xacro)
@@ -1,5 +1,5 @@
 <?xml version='1.0' encoding='utf-8'?>
 <robot xmlns:xacro="http://www.ros.org/wiki/xacro" name="panda">
-  <xacro:macro name="panda_gazebo" params="arm_id include_gazebo_control:=true">
+  <xacro:macro name="panda_gazebo" params="arm_id include_gazebo_control:=true control_mode:='Position'">
     <gazebo reference="${arm_id}_link0"/>
     <gazebo reference="${arm_id}_link1"/>
@@ -18,8 +18,7 @@
         <type>transmission_interface/SimpleTransmission</type>
         <joint name="${arm_id}_joint${joint_num}">
-          <hardwareInterface>hardware_interface/PositionJointInterface</hardwareInterface>
+          <hardwareInterface>hardware_interface/${control_mode}JointInterface</hardwareInterface>
         </joint>
         <actuator name="${arm_id}_joint${joint_num}_motor">
-          <hardwareInterface>hardware_interface/PositionJointInterface</hardwareInterface>
           <mechanicalReduction>1</mechanicalReduction>
         </actuator>
