Commit message: possibility to swap grippers for panda

File: moma_description/urdf/panda.urdf.xacro (robot description, xacro)
@@ -2,4 +2,5 @@
 <robot xmlns:xacro="http://www.ros.org/wiki/xacro" name="panda">
   <xacro:arg name="use_fixed_realsense" default="false"/>
+  <xacro:arg name="tool" default="panda_hand"/>
   <xacro:arg name="control_mode" default='Position'/>
   <xacro:include filename="$(find moma_description)/urdf/panda.xacro"/>
@@ -11,4 +12,4 @@
     <origin rpy="0 0 0" xyz="0 0 0"/>
   </joint>
-  <xacro:panda connected_to="base_link" use_fixed_realsense="$(arg use_fixed_realsense)" control_mode="$(arg control_mode)"/>
+  <xacro:panda connected_to="base_link" use_fixed_realsense="$(arg use_fixed_realsense)" control_mode="$(arg control_mode)" tool="$(arg tool)"/>
 </robot>

File: moma_description/urdf/panda.xacro (robot description, xacro)
@@ -1,11 +1,22 @@
 <?xml version="1.0" encoding="utf-8"?>
 <robot xmlns:xacro="http://www.ros.org/wiki/xacro" name="panda">
-  <xacro:macro name="panda" params="connected_to:='' rpy:='0 0 0' xyz:='0 0 0' use_fixed_realsense:=false include_gazebo_control:=true control_mode:='Position'">
+  <xacro:macro name="panda" params="connected_to:='' rpy:='0 0 0' xyz:='0 0 0' use_fixed_realsense:=false include_gazebo_control:=true tool:='panda_hand' control_mode:='Position'">
     <!-- panda arm  -->
     <xacro:include filename="$(find franka_description)/robots/panda_arm.xacro"/>
     <xacro:panda_arm connected_to="${connected_to}" rpy="${rpy}" xyz="${xyz}"/>
     <!-- panda hand -->
-    <xacro:include filename="$(find franka_description)/robots/hand.xacro"/>
-    <xacro:hand ns="panda" rpy="0 0 ${-pi/4}" connected_to="panda_link8"/>
+    <xacro:if value="${tool == 'panda_hand'}">
+      <xacro:include filename="$(find franka_description)/robots/hand.xacro"/>
+      <xacro:include filename="$(find moma_description)/grippers/panda_hand/panda_hand.gazebo.xacro"/>
+      <xacro:hand ns="panda" rpy="0 0 ${-pi/4}" connected_to="panda_link8"/>
+      <xacro:panda_hand_gazebo arm_id="panda"/>
+    </xacro:if>
+    <!-- robotiq 2f-85 -->
+    <xacro:if value="${tool == 'robotiq_2f_85'}">
+      <xacro:include filename="$(find moma_description)/grippers/robotiq_2f_85/urdf/robotiq_2f_85.xacro"/>
+      <xacro:robotiq_arg2f_85 parent="panda_link8" prefix="">
+        <origin xyz="0 0 0" rpy="0 0 0"/>
+      </xacro:robotiq_arg2f_85>
+    </xacro:if>
     <!-- end effector frame for MoveIt -->
     <link name="panda_default_ee"/>

File: moma_description/urdf/panda_arm.gazebo.xacro (robot description, xacro)
@@ -11,7 +11,4 @@
     <gazebo reference="${arm_id}_link7"/>
     <gazebo reference="${arm_id}_link8"/>
-    <gazebo reference="${arm_id}_hand"/>
-    <gazebo reference="${arm_id}_leftfinger"/>
-    <gazebo reference="${arm_id}_rightfinger"/>
     <xacro:macro name="arm_control" params="joint_num">
       <transmission name="${arm_id}_joint${joint_num}_trans">
@@ -32,23 +29,4 @@
     <xacro:arm_control joint_num="6"/>
     <xacro:arm_control joint_num="7"/>
-    <transmission name="${arm_id}_finger_joint1_trans">
-      <type>transmission_interface/SimpleTransmission</type>
-      <joint name="${arm_id}_finger_joint1">
-        <hardwareInterface>hardware_interface/PositionJointInterface</hardwareInterface>
-      </joint>
-      <actuator name="${arm_id}_finger_joint1_motor">
-        <mechanicalReduction>1</mechanicalReduction>
-      </actuator>
-    </transmission>
-    <!-- Don't need this since the second joint is to be mimicked -->
-    <!-- <transmission name="${arm_id}_finger_joint2_trans">
-      <type>transmission_interface/SimpleTransmission</type>
-      <joint name="${arm_id}_finger_joint2">
-        <hardwareInterface>hardware_interface/PositionJointInterface</hardwareInterface>
-      </joint>
-      <actuator name="${arm_id}_finger_joint2_motor">
-        <mechanicalReduction>1</mechanicalReduction>
-      </actuator>
-    </transmission> -->
     <xacro:if value="${include_gazebo_control}">
       <gazebo>
@@ -58,13 +36,4 @@
       </gazebo>
     </xacro:if>
-    <!-- gazebo plugin to mimic finger joints -->
-    <gazebo>
-      <plugin name="panda_hand_mimic_joint_plugin" filename="libroboticsgroup_gazebo_mimic_joint_plugin.so">
-        <joint>panda_finger_joint1</joint>
-        <mimicJoint>panda_finger_joint2</mimicJoint>
-        <hasPID></hasPID>
-        <multiplier>2.0</multiplier>
-      </plugin>
-    </gazebo>
   </xacro:macro>
 </robot>

Commit message: Fixed panda in gazebo

File: moma_description/urdf/panda.urdf.xacro (robot description, xacro)
@@ -3,11 +3,4 @@
   <xacro:arg name="use_fixed_realsense" default="false"/>
   <xacro:include filename="$(find moma_description)/urdf/panda.xacro"/>
-  <link name="world"/>
-  <link name="base_link"/>
-  <joint name="base_link_joint" type="fixed">
-    <parent link="world"/>
-    <child link="base_link"/>
-    <origin rpy="0 0 0" xyz="0 0 0"/>
-  </joint>
-  <xacro:panda connected_to="base_link" use_fixed_realsense="$(arg use_fixed_realsense)"/>
+  <xacro:moma_panda use_fixed_realsense="$(arg use_fixed_realsense)"/>
 </robot>

File: moma_description/urdf/panda.xacro (robot description, xacro)
@@ -1,11 +1,7 @@
 <?xml version="1.0" encoding="utf-8"?>
 <robot xmlns:xacro="http://www.ros.org/wiki/xacro" name="panda">
-  <xacro:macro name="panda" params="connected_to:='' rpy:='0 0 0' xyz:='0 0 0' use_fixed_realsense:=false include_gazebo_control:=true">
+  <xacro:macro name="moma_panda" params="use_fixed_realsense:=false">
     <!-- panda arm  -->
-    <xacro:include filename="$(find franka_description)/robots/panda_arm.xacro"/>
-    <xacro:panda_arm connected_to="${connected_to}" rpy="${rpy}" xyz="${xyz}"/>
-    <!-- panda hand -->
-    <xacro:include filename="$(find franka_description)/robots/hand.xacro"/>
-    <xacro:hand ns="panda" rpy="0 0 ${-pi/4}" connected_to="panda_link8"/>
+    <xacro:include filename="$(find franka_description)/robots/panda_arm.urdf.xacro"/>
     <!-- end effector frame for MoveIt -->
     <link name="panda_default_ee"/>

Commit message: seems to work

File: moma_description/urdf/panda.urdf.xacro (robot description, xacro)
@@ -4,4 +4,5 @@
   <xacro:arg name="tool" default="panda_hand"/>
   <xacro:arg name="control_mode" default='Position'/>
+  <xacro:arg name="inclde_gazebo_control" default="true"/>
   <xacro:include filename="$(find moma_description)/urdf/panda.xacro"/>
   <link name="world"/>
@@ -12,4 +13,4 @@
     <origin rpy="0 0 0" xyz="0 0 0"/>
   </joint>
-  <xacro:panda connected_to="base_link" use_fixed_realsense="$(arg use_fixed_realsense)" control_mode="$(arg control_mode)" tool="$(arg tool)"/>
+  <xacro:panda connected_to="base_link" use_fixed_realsense="$(arg use_fixed_realsense)" control_mode="$(arg control_mode)" tool="$(arg tool) inclde_gazebo_control=$(inclde_gazebo_control)"/>
 </robot>

File: moma_description/urdf/panda.xacro (robot description, xacro)
@@ -1,5 +1,5 @@
 <?xml version="1.0" encoding="utf-8"?>
 <robot xmlns:xacro="http://www.ros.org/wiki/xacro" name="panda">
-  <xacro:macro name="panda" params="connected_to:='' rpy:='0 0 0' xyz:='0 0 0' use_fixed_realsense:=false include_gazebo_control:=true tool:='panda_hand' control_mode:='Position'">
+  <xacro:macro name="panda" params="connected_to:='' rpy:='0 0 0' xyz:='0 0 0' use_fixed_realsense:=false include_gazebo_control:=true tool:='panda_hand' control_mode:='Position' robot_namespace:='' control_namespace:=''">
     <!-- panda arm  -->
     <xacro:include filename="$(find franka_description)/robots/panda_arm.xacro"/>
@@ -44,5 +44,6 @@
     <!-- Gazebo tags -->
     <xacro:include filename="$(find moma_description)/urdf/panda_arm.gazebo.xacro"/>
-    <xacro:panda_gazebo arm_id="panda" include_gazebo_control="${include_gazebo_control}" control_mode="${control_mode}"/>
+    <xacro:panda_gazebo arm_id="panda" include_gazebo_control="${include_gazebo_control}" control_mode="${control_mode}"
+      robot_namespace="${robot_namespace}" control_namespace="${control_namespace}"/>
     <!-- wrist realsense -->
     <xacro:include filename="$(find realsense2_description)/urdf/_d435.urdf.xacro" />

File: moma_description/urdf/panda_arm.gazebo.xacro (robot description, xacro)
@@ -1,5 +1,6 @@
 <?xml version='1.0' encoding='utf-8'?>
 <robot xmlns:xacro="http://www.ros.org/wiki/xacro" name="panda">
-  <xacro:macro name="panda_gazebo" params="arm_id include_gazebo_control:=true control_mode:='Position'">
+  <xacro:macro name="panda_gazebo" params="arm_id include_gazebo_control:=true control_mode:='Position'
+    robot_namespace:='' control_namespace:=''">
     <gazebo reference="${arm_id}_link0"/>
     <gazebo reference="${arm_id}_link1"/>
@@ -32,5 +33,7 @@
       <gazebo>
         <plugin name="gazebo_ros_control" filename="libgazebo_ros_control.so">
-          <robotNamespace>/</robotNamespace>
+          <robotNamespace>${robot_namespace}/${control_namespace}</robotNamespace>
+          <robotDescription>robot_description</robotDescription>
+          <robotSimType>gazebo_ros_control/DefaultRobotHWSim</robotSimType>
         </plugin>
       </gazebo>

File: moma_description/urdf/superpanda.urdf.xacro (robot description, xacro)
@@ -4,6 +4,6 @@
   <xacro:arg name="wheel_joint_type"          default="continuous"/>
   <xacro:arg name="simulation"                default="true"/>
-  <xacro:arg name="use_ros_skid_steer"        default="false"/>  <!-- Specify one! -->
-  <xacro:arg name="use_ros_control"           default="true"/>
+  <xacro:arg name="use_ros_skid_steer"        default="false"/>  <!-- This does not work nicely -->
+  <xacro:arg name="use_ros_control"           default="false"/>  <!-- Set to faulse as we import already a plugin for the arm-->
   <xacro:arg name="lidar"                     default="true"/>
   <xacro:arg name="robot_namespace"           default=""/>
@@ -34,4 +34,4 @@
   <xacro:arg name="control_mode" default='Position'/>
   <xacro:include filename="$(find moma_description)/urdf/panda.xacro"/>
-  <xacro:panda connected_to="arm_mount_link" use_fixed_realsense="$(arg use_fixed_realsense)" control_mode="$(arg control_mode)" tool="$(arg tool) include_gazebo_control:=false"/>
+  <xacro:panda connected_to="arm_mount_link" use_fixed_realsense="$(arg use_fixed_realsense)" control_mode="$(arg control_mode)" tool="$(arg tool)" include_gazebo_control="true" robot_namespace="" control_namespace="control"/>
 </robot>

Commit message: splitting smb and panda namespaces

File: moma_description/urdf/panda.urdf.xacro (robot description, xacro)
@@ -6,4 +6,5 @@
   <xacro:arg name="include_gazebo_control" default="true"/>
   <xacro:include filename="$(find moma_description)/urdf/panda.xacro"/>
+  <xacro:include filename="$(find moma_description)/urdf/panda_arm.gazebo.xacro"/>
   <link name="world"/>
   <link name="base_link"/>
@@ -13,4 +14,5 @@
     <origin rpy="0 0 0" xyz="0 0 0"/>
   </joint>
-  <xacro:panda connected_to="base_link" use_fixed_realsense="$(arg use_fixed_realsense)" control_mode="$(arg control_mode)" tool="$(arg tool)" include_gazebo_control="$(arg include_gazebo_control)"/>
+  <xacro:panda connected_to="base_link" use_fixed_realsense="$(arg use_fixed_realsense)" tool="$(arg tool)"/>
+  <xacro:panda_gazebo arm_id="panda" include_gazebo_control="false" control_mode="$(arg control_mode)"/>
 </robot>

File: moma_description/urdf/panda.xacro (robot description, xacro)
@@ -1,5 +1,5 @@
 <?xml version="1.0" encoding="utf-8"?>
 <robot xmlns:xacro="http://www.ros.org/wiki/xacro" name="panda">
-  <xacro:macro name="panda" params="connected_to:='' rpy:='0 0 0' xyz:='0 0 0' use_fixed_realsense:=false include_gazebo_control:=true tool:='panda_hand' control_mode:='Position' robot_namespace:='' control_namespace:=''">
+  <xacro:macro name="panda" params="connected_to:='' rpy:='0 0 0' xyz:='0 0 0' use_fixed_realsense:=false tool:='panda_hand'">
     <!-- panda arm  -->
     <xacro:include filename="$(find franka_description)/robots/panda_arm.xacro"/>
@@ -50,8 +50,4 @@
       <origin rpy="0.0 0.0 -0.785" xyz="0.0 0.0 0.103"/>
     </joint>
-    <!-- Gazebo tags -->
-    <xacro:include filename="$(find moma_description)/urdf/panda_arm.gazebo.xacro"/>
-    <xacro:panda_gazebo arm_id="panda" include_gazebo_control="${include_gazebo_control}" control_mode="${control_mode}"
-      robot_namespace="${robot_namespace}" control_namespace="${control_namespace}"/>
     <!-- wrist realsense -->
     <xacro:include filename="$(find realsense2_description)/urdf/_d435.urdf.xacro" />

File: moma_description/urdf/panda_arm.gazebo.xacro (robot description, xacro)
@@ -1,6 +1,6 @@
 <?xml version='1.0' encoding='utf-8'?>
 <robot xmlns:xacro="http://www.ros.org/wiki/xacro" name="panda">
-  <xacro:macro name="panda_gazebo" params="arm_id include_gazebo_control:=true control_mode:='Position'
-    robot_namespace:='' control_namespace:=''">
+  <xacro:macro name="panda_gazebo" params="arm_id control_mode:='Position'
+    robot_namespace:='' control_namespace:='' description_name:='robot_description' include_gazebo_control:=true">
     <gazebo reference="${arm_id}_link0"/>
     <gazebo reference="${arm_id}_link1"/>
@@ -34,5 +34,6 @@
         <plugin name="gazebo_ros_control" filename="libgazebo_ros_control.so">
           <robotNamespace>${robot_namespace}/${control_namespace}</robotNamespace>
-          <robotDescription>robot_description</robotDescription>
+          <robotDescription>${description_name}</robotDescription>
+          <robotParam>${description_name}</robotParam>
           <robotSimType>gazebo_ros_control/DefaultRobotHWSim</robotSimType>
         </plugin>

File: moma_description/urdf/superpanda.urdf.xacro (robot description, xacro)
@@ -1,6 +1,21 @@
 <?xml version="1.0" encoding="utf-8"?>
 <robot xmlns:xacro="http://www.ros.org/wiki/xacro" name="superpanda">
+  <!-- Panda Arguments -->
+  <xacro:arg name="use_fixed_realsense" default="false"/>
+  <xacro:arg name="tool" default="panda_hand"/>
+  <xacro:arg name="control_mode" default='Position'/>
   <!-- MPC Arguments -->
   <xacro:arg name="mpc_model" default="false"/>
+  <!-- SMB Arguments -->
+  <xacro:arg name="wheel_joint_type"          default="continuous"/>
+  <xacro:arg name="simulation"                default="true"/>
+  <xacro:arg name="lidar"                     default="true"/>
+  <xacro:arg name="robot_namespace"           default=""/>
+  <xacro:arg name="description_name_xacro"    default="robot_description"/>
+  <xacro:arg name="publish_tf"                default="true"/>
+  <xacro:arg name="tracking_camera"           default="true"/>
+  <xacro:property name="lidar" value="$(arg lidar)"/>
+  <xacro:include filename="$(find smb_description)/urdf/smb_piloting_properties.urdf.xacro" />
+  <!-- Optionally load a kinematic chain for MPC or the full smb model -->
   <xacro:if value="$(arg mpc_model)">
     <link name="world" />
@@ -36,22 +51,5 @@
     <link name="base_link" />
   </xacro:if>
-  <!-- SMB Arguments -->
-  <xacro:arg name="wheel_joint_type"          default="continuous"/>
-  <xacro:arg name="simulation"                default="true"/>
-  <xacro:arg name="use_ros_skid_steer"        default="false"/>  <!-- This does not work nicely -->
-  <xacro:arg name="use_ros_control"           default="false"/>  <!-- Set to faulse as we import already a plugin for the arm-->
-  <xacro:arg name="lidar"                     default="true"/>
-  <xacro:arg name="robot_namespace"           default=""/>
-  <xacro:arg name="description_name_xacro"    default="robot_description"/>
-  <xacro:arg name="publish_tf"                default="true"/>
-  <xacro:arg name="tracking_camera"           default="true"/>
-  <xacro:property name="lidar" value="$(arg lidar)"/>
-  <!-- SMB Includes -->
-  <xacro:include filename="$(find smb_description)/urdf/smb_piloting_properties.urdf.xacro" />
   <xacro:unless value="$(arg mpc_model)">
-    <xacro:if value="$(arg simulation)">
-      <xacro:include filename="$(find smb_description)/urdf/smb_gazebo_addins.urdf.xacro"/>
-    </xacro:if>
-    <!-- SMB -->
     <xacro:include filename="$(find smb_description)/urdf/smb.urdf.xacro">
       <xacro:arg name="lidar" default="$(arg lidar)"/>
@@ -59,4 +57,10 @@
     <xacro:smb wheel_joint_type="$(arg wheel_joint_type)" simulation="$(arg simulation)" tracking_camera="$(arg tracking_camera)"/>
   </xacro:unless>
+  <!-- Load Panda -->
+  <xacro:include filename="$(find moma_description)/urdf/panda.xacro"/>
+  <xacro:panda
+    connected_to="arm_mount_link"
+    use_fixed_realsense="$(arg use_fixed_realsense)"
+    tool="$(arg tool)"/>
   <!-- Rigid fix between SMB and Panda -->
   <link name="arm_mount_link"/>
@@ -66,9 +70,19 @@
     <origin xyz="0.115 0.0 ${0.228+chassisHeight/2.0}" rpy="0 0 0"/>
   </joint>
-  <!-- Panda Arguments -->
-  <xacro:arg name="use_fixed_realsense" default="false"/>
-  <xacro:arg name="tool" default="panda_hand"/>
-  <xacro:arg name="control_mode" default='Position'/>
-  <xacro:include filename="$(find moma_description)/urdf/panda.xacro"/>
-  <xacro:panda connected_to="arm_mount_link" use_fixed_realsense="$(arg use_fixed_realsense)" control_mode="$(arg control_mode)" tool="$(arg tool)" include_gazebo_control="true" robot_namespace="" control_namespace="control"/>
+  <!-- Gazebo plugins for control -->
+  <xacro:if value="$(arg simulation)">
+      <xacro:include filename="$(find moma_description)/urdf/panda_arm.gazebo.xacro"/>
+      <xacro:include filename="$(find smb_description)/urdf/smb_ros_control.gazebo.xacro"/>
+      <xacro:smb_ros_control_plugin
+        description_name="smb_description"
+        broadcast_tf="false"
+        robot_namespace=""
+        control_namespace="smb"/>
+      <xacro:panda_gazebo
+        arm_id="panda"
+        control_mode="$(arg control_mode)"
+        description_name="arm_description"
+        robot_namespace=""
+        control_namespace="panda"/>
+  </xacro:if>
 </robot>

Commit message: Added flag to use nominal realsense extrinsics

File: moma_description/urdf/panda.urdf.xacro (robot description, xacro)
@@ -2,5 +2,6 @@
 <robot xmlns:xacro="http://www.ros.org/wiki/xacro" name="panda">
   <xacro:arg name="use_fixed_realsense" default="false"/>
+  <xacro:arg name="use_nominal_extrinsics" default="false"/>
   <xacro:include filename="$(find moma_description)/urdf/panda.xacro"/>
-  <xacro:moma_panda use_fixed_realsense="$(arg use_fixed_realsense)"/>
+  <xacro:moma_panda use_fixed_realsense="$(arg use_fixed_realsense)" use_nominal_extrinsics="$(arg use_nominal_extrinsics)"/>
 </robot>

File: moma_description/urdf/panda.xacro (robot description, xacro)
@@ -1,5 +1,5 @@
 <?xml version="1.0" encoding="utf-8"?>
 <robot xmlns:xacro="http://www.ros.org/wiki/xacro" name="panda">
-  <xacro:macro name="moma_panda" params="use_fixed_realsense:=false">
+  <xacro:macro name="moma_panda" params="use_fixed_realsense:=false use_nominal_extrinsics:=false">
     <!-- panda arm  -->
     <xacro:include filename="$(find franka_description)/robots/panda_arm.urdf.xacro"/>
@@ -17,5 +17,5 @@
     <xacro:property name="panda_link7_camera_bottom_screw_frame_rpy" value="-2.68850999 -1.56973844 -1.20267232" />
     <xacro:property name="panda_link7_camera_bottom_screw_frame_xyz" value="0.06585917 -0.06861364 0.14820608" />
-    <xacro:sensor_d435 parent="panda_link7" name="wrist_camera">
+    <xacro:sensor_d435 parent="panda_link7" name="wrist_camera" use_nominal_extrinsics="${use_nominal_extrinsics}">
       <origin rpy="${panda_link7_camera_bottom_screw_frame_rpy}" xyz="${panda_link7_camera_bottom_screw_frame_xyz}" />
     </xacro:sensor_d435>
