Commit message: On the way of combining panda and ridgeback

File: moma_description/urdf/panda.urdf.xacro (robot description, xacro)
@@ -10,4 +10,5 @@
   <xacro:arg name="use_fixed_realsense" default="false"/>
   <xacro:arg name="use_nominal_extrinsics" default="false"/>
+  <xacro:arg name="include_control_plugin" default="false"/>
   <xacro:include filename="$(find moma_description)/urdf/panda_arm.xacro"/>
   <xacro:moma_panda arm_id="$(arg arm_id)"
@@ -19,4 +20,5 @@
                     rpy="$(arg rpy)"
                     use_fixed_realsense="$(arg use_fixed_realsense)"
-                    use_nominal_extrinsics="$(arg use_nominal_extrinsics)"/>
+                    use_nominal_extrinsics="$(arg use_nominal_extrinsics)"
+                    include_control_plugin="$(arg include_control_plugin)"/>
 </robot>

File: moma_description/urdf/panda_arm.xacro (robot description, xacro)
@@ -10,5 +10,6 @@
                                        rpy:='0 0 0'
                                        use_fixed_realsense:=false
-                                       use_nominal_extrinsics:=false">
+                                       use_nominal_extrinsics:=false
+                                       include_control_plugin:=false">
   <xacro:unless value="${gazebo}">
     <!-- Create a URDF for a real hardware -->
@@ -72,11 +73,16 @@
        tip="${arm_id}_joint8"
      />
-    <gazebo>
-      <plugin name="gazebo_ros_control" filename="libgazebo_ros_control.so">
-        <controlPeriod>0.001</controlPeriod>
-        <robotSimType>franka_gazebo/FrankaHWSim</robotSimType>
-      </plugin>
-      <self_collide>true</self_collide>
-    </gazebo>
+    <xacro:if value="${include_control_plugin}">
+      <gazebo>
+        <plugin name="gazebo_ros_control" filename="libgazebo_ros_control.so">
+          <controlPeriod>0.001</controlPeriod>
+          <robotSimType>franka_gazebo/FrankaHWSim</robotSimType>
+          <robotNamespace>/panda</robotNamespace>
+          <robotParam>robot_description_arm</robotParam>
+          <robotDescription>robot_description_arm</robotDescription>
+        </plugin>
+        <self_collide>true</self_collide>
+      </gazebo>
+    </xacro:if>
   </xacro:if>
   <!-- end effector frame for MoveIt -->

File: moma_description/urdf/ridgeback.xacro (robot description, xacro)
@@ -1,7 +1,10 @@
 <?xml version="1.0" encoding="utf-8"?>
 <robot xmlns:xacro="http://www.ros.org/wiki/xacro" name="ridgeback">
-  <xacro:macro name="ridgeback">
+  <xacro:macro name="ridgeback" params="include_control_plugin:=false">
     <!-- Ridgeback -->
-    <xacro:include filename="$(find ridgeback_description)/urdf/ridgeback.urdf.xacro"/>
+    <xacro:include filename="$(find moma_description)/urdf/ridgeback_nocontrol.xacro"/>
+    <xacro:if value="${include_control_plugin}">
+      <xacro:include filename="$(find moma_description)/urdf/ridgeback.gazebo.xacro"/>
+    </xacro:if>
     <!-- Sensor mount -->
     <link name="ridgeback_sensor_mount_link">

File: moma_description/urdf/royalpanda.urdf.xacro (robot description, xacro)
@@ -4,14 +4,22 @@
     <xacro:include filename="$(find moma_description)/urdf/ridgeback.xacro"/>
     <xacro:ridgeback/>
+    <!-- <link name="world"/>
+    <link name="mid_mount"/>
+    <joint name="world_joint" type="fixed">
+        <parent link="world"/>
+        <child link="mid_mount"/>
+        <origin xyz="0 0 0" rpy="0 0 0"/>
+    </joint> -->
+    <link name="franka_mount_link"/>
     <joint name="arm_mount_joint" type="fixed">
-        <parent link="mid_mount" />
-        <child link="franka_mount_link" />
+        <parent link="mid_mount"/>
+        <child link="franka_mount_link"/>
         <origin xyz="$(optenv RIDGEBACK_FRANKA_XYZ 0.21 0.0 0.2)" rpy="$(optenv RIDGEBACK_FRANKA_RPY 0 0 0)"/>
     </joint>
-    <link name="franka_mount_link" />
     <xacro:include filename="$(find moma_description)/urdf/panda_arm.xacro"/>
     <xacro:moma_panda gazebo="true"
                       fixed_to_world="false"
                       connected_to="franka_mount_link"
-                      use_nominal_extrinsics="$(arg use_nominal_extrinsics)"/>
+                      use_nominal_extrinsics="$(arg use_nominal_extrinsics)"
+                      include_control_plugin="true"/>
 </robot>

Commit message: Update arm xacros.

File: moma_description/urdf/panda.urdf.xacro (robot description, xacro)
@@ -4,21 +4,19 @@
   <xacro:arg name="hand" default="true"/>
   <xacro:arg name="gazebo" default="false"/>
-  <xacro:arg name="fixed_to_world" default="false"/>
-  <xacro:arg name="connected_to" default=""/>
   <xacro:arg name="xyz" default="0 0 0"/>
   <xacro:arg name="rpy" default="0 0 0"/>
-  <xacro:arg name="use_fixed_realsense" default="false"/>
-  <xacro:arg name="use_nominal_extrinsics" default="false"/>
+  <xacro:arg name="use_fixed_camera" default="true"/>
+  <xacro:arg name="use_wrist_camera" default="true"/>
   <xacro:arg name="include_control_plugin" default="false"/>
+  <xacro:arg name="parent" default="world"/>
   <xacro:include filename="$(find moma_description)/urdf/panda_arm.xacro"/>
   <xacro:moma_panda arm_id="$(arg arm_id)"
                     hand="$(arg hand)"
                     gazebo="$(arg gazebo)"
-                    fixed_to_world="$(arg fixed_to_world)"
-                    connected_to="$(arg connected_to)"
+                    parent="$(arg parent)"
                     xyz="$(arg xyz)"
                     rpy="$(arg rpy)"
-                    use_fixed_realsense="$(arg use_fixed_realsense)"
-                    use_nominal_extrinsics="$(arg use_nominal_extrinsics)"
+                    use_fixed_camera="$(arg use_fixed_camera)"
+                    use_wrist_camera="$(arg use_wrist_camera)"
                     include_control_plugin="$(arg include_control_plugin)"/>
 </robot>

File: moma_description/urdf/panda_arm.xacro (robot description, xacro)
@@ -1,122 +1,145 @@
 <?xml version='1.0' encoding='utf-8'?>
-<robot xmlns:xacro="http://www.ros.org/wiki/xacro" name="panda">
-<!-- Adapted from franka_description/robots/common/franka_robot.xacro -->
-<xacro:macro name="moma_panda" params="arm_id:='panda'
-                                       hand:=true
-                                       gazebo:=false
-                                       fixed_to_world:=false
-                                       connected_to:=''
-                                       xyz:='0 0 0'
-                                       rpy:='0 0 0'
-                                       use_fixed_realsense:=false
-                                       use_nominal_extrinsics:=false
-                                       include_control_plugin:=false">
-  <xacro:include filename="$(find franka_description)/robots/common/utils.xacro" />
-  <xacro:include filename="$(find franka_description)/robots/common/franka_arm.xacro" />
-  <!-- Positional offset between $(arm_id)_hand -> $(arm_id)_hand_tcp [m]. Only used when hand:=true -->
-  <xacro:arg name="tcp_xyz" default="0 0 0.1034" />
-  <!-- Rotational offset between $(arm_id)_hand -> $(arm_id)_hand_tcp [rad]. Only used when hand:=true -->
-  <xacro:arg name="tcp_rpy" default="0 0 0" />
-  <xacro:franka_arm
-      arm_id="${arm_id}"
-      connected_to="${connected_to}"
-      xyz="${xyz}"
-      rpy="${rpy}"
-      safety_distance="0.03"
-      gazebo="${gazebo}"
-      joint_limits="${xacro.load_yaml('$(find franka_description)/robots/panda/joint_limits.yaml')}"/>
-  <xacro:if value="${hand}">
-    <xacro:include filename="$(find franka_description)/robots/common/franka_hand.xacro"/>
-    <xacro:franka_hand
+<robot xmlns:xacro="http://www.ros.org/wiki/xacro">
+  <!-- Adapted from franka_description/robots/common/franka_robot.xacro -->
+  <xacro:macro name="moma_panda"
+    params="
+        arm_id:='panda'
+        parent:='world'
+        xyz:='0 0 0'
+        rpy:='0 0 0'
+        tcp_xyz:='0 0 0.1034'
+        tcp_rpy='0 0 0'
+        hand:=true
+        gazebo:=false
+        use_wrist_camera:=false
+        wrist_calibration_rpy:='-0.891 -1.562 -3.040'
+        wrist_calibration_xyz:='0.0306 -0.0267  0.1604'
+        wrist_camera_parent_link:='panda_link7'
+        use_fixed_camera:=false
+        fixed_calibration_rpy:='0 1.57 0'
+        fixed_calibration_xyz:='1 0 1'
+        fixed_camera_parent_link:='panda_link0'
+        include_control_plugin:=false">
+    <xacro:include filename="$(find franka_description)/robots/common/utils.xacro" />
+    <xacro:include filename="$(find franka_description)/robots/common/franka_arm.xacro" />
+    <!-- Put in a basic arm. -->
+    <xacro:franka_arm arm_id="${arm_id}" safety_distance="0.03" gazebo="${gazebo}"
+      joint_limits="${xacro.load_yaml('$(find franka_description)/robots/panda/joint_limits.yaml')}" />
+    <!-- Put in a basic hand. -->
+    <xacro:if value="${hand}">
+      <xacro:include filename="$(find franka_description)/robots/common/franka_hand.xacro" />
+      <xacro:franka_hand
         arm_id="${arm_id}"
         rpy="0 0 ${-pi/4}"
-        tcp_xyz="$(arg tcp_xyz)"
-        tcp_rpy="$(arg tcp_rpy)"
+        tcp_xyz="${tcp_xyz}"
+        tcp_rpy="${tcp_rpy}"
         connected_to="${arm_id}_link8"
         safety_distance="0.03"
         gazebo="${gazebo}"
-     />
-  </xacro:if>
-  <xacro:if value="${gazebo}">
-    <!-- Gazebo requires a joint to a link called "world" for statically mounted robots -->
-    <xacro:if value="${fixed_to_world}">
-      <link name="world" />
-      <joint name="world_joint" type="fixed">
-        <origin xyz="${xyz}" rpy="${rpy}" />
-        <parent link="world" />
-        <child  link="${arm_id}_link0" />
-      </joint>
+      />
     </xacro:if>
-    <xacro:gazebo-joint joint="${arm_id}_joint1" transmission="hardware_interface/PositionJointInterface" />
-    <xacro:gazebo-joint joint="${arm_id}_joint2" transmission="hardware_interface/PositionJointInterface" />
-    <xacro:gazebo-joint joint="${arm_id}_joint3" transmission="hardware_interface/PositionJointInterface" />
-    <xacro:gazebo-joint joint="${arm_id}_joint4" transmission="hardware_interface/PositionJointInterface" />
-    <xacro:gazebo-joint joint="${arm_id}_joint5" transmission="hardware_interface/PositionJointInterface" />
-    <xacro:gazebo-joint joint="${arm_id}_joint6" transmission="hardware_interface/PositionJointInterface" />
-    <xacro:gazebo-joint joint="${arm_id}_joint7" transmission="hardware_interface/PositionJointInterface" />
-    <xacro:gazebo-joint joint="${arm_id}_joint1" transmission="hardware_interface/VelocityJointInterface" />
-    <xacro:gazebo-joint joint="${arm_id}_joint2" transmission="hardware_interface/VelocityJointInterface" />
-    <xacro:gazebo-joint joint="${arm_id}_joint3" transmission="hardware_interface/VelocityJointInterface" />
-    <xacro:gazebo-joint joint="${arm_id}_joint4" transmission="hardware_interface/VelocityJointInterface" />
-    <xacro:gazebo-joint joint="${arm_id}_joint5" transmission="hardware_interface/VelocityJointInterface" />
-    <xacro:gazebo-joint joint="${arm_id}_joint6" transmission="hardware_interface/VelocityJointInterface" />
-    <xacro:gazebo-joint joint="${arm_id}_joint7" transmission="hardware_interface/VelocityJointInterface" />
-    <xacro:gazebo-joint joint="${arm_id}_joint1" transmission="hardware_interface/EffortJointInterface" />
-    <xacro:gazebo-joint joint="${arm_id}_joint2" transmission="hardware_interface/EffortJointInterface" />
-    <xacro:gazebo-joint joint="${arm_id}_joint3" transmission="hardware_interface/EffortJointInterface" />
-    <xacro:gazebo-joint joint="${arm_id}_joint4" transmission="hardware_interface/EffortJointInterface" />
-    <xacro:gazebo-joint joint="${arm_id}_joint5" transmission="hardware_interface/EffortJointInterface" />
-    <xacro:gazebo-joint joint="${arm_id}_joint6" transmission="hardware_interface/EffortJointInterface" />
-    <xacro:gazebo-joint joint="${arm_id}_joint7" transmission="hardware_interface/EffortJointInterface" />
-    <xacro:transmission-franka-state arm_id="${arm_id}" />
-    <xacro:transmission-franka-model arm_id="${arm_id}"
-       root="${arm_id}_joint1"
-       tip="${arm_id}_joint8"
-    />
-    <xacro:if value="${hand}">
-      <xacro:gazebo-joint joint="${arm_id}_finger_joint1" transmission="hardware_interface/EffortJointInterface" />
-      <xacro:gazebo-joint joint="${arm_id}_finger_joint2" transmission="hardware_interface/EffortJointInterface" />
-      <!-- Friction specific material for Rubber/Rubber contact -->
-      <xacro:gazebo-friction link="${arm_id}_leftfinger" mu="1.13" />
-      <xacro:gazebo-friction link="${arm_id}_rightfinger" mu="1.13" />
+    <!-- wrist realsense -->
+    <xacro:include filename="$(find realsense2_description)/urdf/_d435.urdf.xacro" />
+    <xacro:include filename="$(find moma_description)/urdf/realsense.gazebo.xacro" />
+    <xacro:if value="${use_wrist_camera}">
+      <xacro:realsense_gazebo_plugin camera_name="wrist_camera" />
+      <xacro:sensor_d435 parent="${wrist_camera_parent_link}" name="wrist_camera"
+        use_nominal_extrinsics="true">
+        <origin rpy="${wrist_calibration_rpy}"
+          xyz="${wrist_calibration_xyz}" />
+      </xacro:sensor_d435>
     </xacro:if>
-    <xacro:if value="${include_control_plugin}">
-      <gazebo>
-        <plugin name="gazebo_ros_control" filename="libgazebo_ros_control.so">
-          <controlPeriod>0.001</controlPeriod>
-          <robotSimType>franka_gazebo/FrankaHWSim</robotSimType>
-          <robotNamespace>/panda</robotNamespace>
-          <robotParam>robot_description_arm</robotParam>
-          <robotDescription>robot_description_arm</robotDescription>
-        </plugin>
-        <self_collide>true</self_collide>
-      </gazebo>
+    <!-- fixed realsense -->
+    <xacro:if value="${use_fixed_camera}">
+      <xacro:realsense_gazebo_plugin camera_name="fixed_camera" />
+      <xacro:sensor_d435 parent="${fixed_camera_parent_link}" name="fixed_camera"
+        use_nominal_extrinsics="true">
+        <origin rpy="${fixed_calibration_rpy}"
+          xyz="${fixed_calibration_xyz}" />
+      </xacro:sensor_d435>
     </xacro:if>
-  </xacro:if>
-  <!-- end effector frame for MoveIt -->
-  <link name="${arm_id}_default_ee"/>
-  <joint name="joint_link8_default_ee" type="fixed">
-    <parent link="${arm_id}_link8"/>
-    <child link="${arm_id}_default_ee"/>
-    <origin rpy="0.0 0.0 -0.785" xyz="0.0 0.0 0.103"/>
-  </joint>
-  <!-- wrist realsense -->
-  <xacro:include filename="$(find realsense2_description)/urdf/_d435.urdf.xacro" />
-  <xacro:include filename="$(find moma_description)/urdf/realsense.gazebo.xacro" />
-  <xacro:realsense_gazebo_plugin camera_name="wrist_camera"/>
-  <xacro:property name="panda_link7_camera_bottom_screw_frame_rpy" value="-0.891 -1.562 -3.040" />
-  <xacro:property name="panda_link7_camera_bottom_screw_frame_xyz" value="0.0306 -0.0267  0.1604" />
-  <xacro:sensor_d435 parent="${arm_id}_link7" name="wrist_camera" use_nominal_extrinsics="${use_nominal_extrinsics}">
-    <origin rpy="${panda_link7_camera_bottom_screw_frame_rpy}" xyz="${panda_link7_camera_bottom_screw_frame_xyz}" />
-  </xacro:sensor_d435>
-  <!-- fixed realsense -->
-  <xacro:if value="${use_fixed_realsense}">
-    <xacro:realsense_gazebo_plugin camera_name="fixed_camera"/>
-    <xacro:property name="base_link_camera_bottom_screw_frame_rpy" value="0 0.79 -0.79" />
-    <xacro:property name="base_link_camera_bottom_screw_frame_xyz" value="0.1 0.75 0.9" />
-    <xacro:sensor_d435 parent="base_link" name="fixed_camera" use_nominal_extrinsics="${use_nominal_extrinsics}">
-      <origin rpy="${base_link_camera_bottom_screw_frame_rpy}" xyz="${base_link_camera_bottom_screw_frame_xyz}" />
-    </xacro:sensor_d435>
-  </xacro:if>
-</xacro:macro>
+    <!-- Below here, gazebo stuff. -->
+    <!-- Define additional Gazebo tags -->
+    <xacro:if value="${gazebo}">
+      <xacro:if value="${parent != ''}">
+        <!-- Gazebo requires a joint to a link called "world" for statically mounted robots -->
+        <xacro:if value="${parent == 'world'}">
+          <link name="${parent}" />
+        </xacro:if>
+        <joint name="${parent}_joint" type="fixed">
+          <origin xyz="${xyz}" rpy="${rpy}" />
+          <parent link="${parent}" />
+          <child link="${arm_id}_link0" />
+        </joint>
+      </xacro:if>
+      <xacro:gazebo-joint joint="${arm_id}_joint1"
+        transmission="hardware_interface/PositionJointInterface" />
+      <xacro:gazebo-joint joint="${arm_id}_joint2"
+        transmission="hardware_interface/PositionJointInterface" />
+      <xacro:gazebo-joint joint="${arm_id}_joint3"
+        transmission="hardware_interface/PositionJointInterface" />
+      <xacro:gazebo-joint joint="${arm_id}_joint4"
+        transmission="hardware_interface/PositionJointInterface" />
+      <xacro:gazebo-joint joint="${arm_id}_joint5"
+        transmission="hardware_interface/PositionJointInterface" />
+      <xacro:gazebo-joint joint="${arm_id}_joint6"
+        transmission="hardware_interface/PositionJointInterface" />
+      <xacro:gazebo-joint joint="${arm_id}_joint7"
+        transmission="hardware_interface/PositionJointInterface" />
+      <xacro:gazebo-joint joint="${arm_id}_joint1"
+        transmission="hardware_interface/VelocityJointInterface" />
+      <xacro:gazebo-joint joint="${arm_id}_joint2"
+        transmission="hardware_interface/VelocityJointInterface" />
+      <xacro:gazebo-joint joint="${arm_id}_joint3"
+        transmission="hardware_interface/VelocityJointInterface" />
+      <xacro:gazebo-joint joint="${arm_id}_joint4"
+        transmission="hardware_interface/VelocityJointInterface" />
+      <xacro:gazebo-joint joint="${arm_id}_joint5"
+        transmission="hardware_interface/VelocityJointInterface" />
+      <xacro:gazebo-joint joint="${arm_id}_joint6"
+        transmission="hardware_interface/VelocityJointInterface" />
+      <xacro:gazebo-joint joint="${arm_id}_joint7"
+        transmission="hardware_interface/VelocityJointInterface" />
+      <xacro:gazebo-joint joint="${arm_id}_joint1"
+        transmission="hardware_interface/EffortJointInterface" />
+      <xacro:gazebo-joint joint="${arm_id}_joint2"
+        transmission="hardware_interface/EffortJointInterface" />
+      <xacro:gazebo-joint joint="${arm_id}_joint3"
+        transmission="hardware_interface/EffortJointInterface" />
+      <xacro:gazebo-joint joint="${arm_id}_joint4"
+        transmission="hardware_interface/EffortJointInterface" />
+      <xacro:gazebo-joint joint="${arm_id}_joint5"
+        transmission="hardware_interface/EffortJointInterface" />
+      <xacro:gazebo-joint joint="${arm_id}_joint6"
+        transmission="hardware_interface/EffortJointInterface" />
+      <xacro:gazebo-joint joint="${arm_id}_joint7"
+        transmission="hardware_interface/EffortJointInterface" />
+      <xacro:transmission-franka-state arm_id="${arm_id}" />
+      <xacro:transmission-franka-model arm_id="${arm_id}"
+        root="${arm_id}_joint1"
+        tip="${arm_id}_joint8"
+      />
+      <xacro:if value="${hand}">
+        <xacro:gazebo-joint joint="${arm_id}_finger_joint1"
+          transmission="hardware_interface/EffortJointInterface" />
+        <xacro:gazebo-joint joint="${arm_id}_finger_joint2"
+          transmission="hardware_interface/EffortJointInterface" />
+        <!-- Friction specific material for Rubber/Rubber contact -->
+        <xacro:gazebo-friction link="${arm_id}_leftfinger" mu="1.13" />
+        <xacro:gazebo-friction link="${arm_id}_rightfinger" mu="1.13" />
+      </xacro:if>
+      <xacro:if value="${include_control_plugin}">
+        <gazebo>
+          <plugin name="gazebo_ros_control" filename="libgazebo_ros_control.so">
+            <controlPeriod>0.001</controlPeriod>
+            <robotSimType>franka_gazebo/FrankaHWSim</robotSimType>
+            <robotNamespace>/panda</robotNamespace>
+            <robotParam>robot_description_arm</robotParam>
+            <robotDescription>robot_description_arm</robotDescription>
+          </plugin>
+          <self_collide>true</self_collide>
+        </gazebo>
+      </xacro:if>
+    </xacro:if>
+  </xacro:macro>
 </robot>
