Commit message: Modified the xacros.

File: moma_description/urdf/panda.urdf.xacro (robot description, xacro)
@@ -1,22 +1,24 @@
 <?xml version="1.0" encoding="utf-8"?>
 <robot xmlns:xacro="http://www.ros.org/wiki/xacro" name="panda">
-  <xacro:arg name="arm_id" default="panda"/>
-  <xacro:arg name="hand" default="true"/>
-  <xacro:arg name="gazebo" default="false"/>
-  <xacro:arg name="xyz" default="0 0 0"/>
-  <xacro:arg name="rpy" default="0 0 0"/>
-  <xacro:arg name="use_fixed_camera" default="true"/>
-  <xacro:arg name="use_wrist_camera" default="true"/>
-  <xacro:arg name="include_control_plugin" default="false"/>
-  <xacro:arg name="parent" default="world"/>
-  <xacro:include filename="$(find moma_description)/urdf/panda_arm.xacro"/>
+  <xacro:arg name="arm_id" default="panda" />
+  <xacro:arg name="hand" default="true" />
+  <xacro:arg name="gazebo" default="false" />
+  <xacro:arg name="xyz" default="0 0 0" />
+  <xacro:arg name="rpy" default="0 0 0" />
+  <xacro:arg name="use_fixed_camera" default="true" />
+  <xacro:arg name="use_wrist_camera" default="true" />
+  <xacro:arg name="use_bota" default="true" />
+  <xacro:arg name="include_control_plugin" default="true" />
+  <xacro:arg name="parent" default="world" />
+  <xacro:include filename="$(find moma_description)/urdf/panda_arm.xacro" />
   <xacro:moma_panda arm_id="$(arg arm_id)"
-                    hand="$(arg hand)"
-                    gazebo="$(arg gazebo)"
-                    parent="$(arg parent)"
-                    xyz="$(arg xyz)"
-                    rpy="$(arg rpy)"
-                    use_fixed_camera="$(arg use_fixed_camera)"
-                    use_wrist_camera="$(arg use_wrist_camera)"
-                    include_control_plugin="$(arg include_control_plugin)"/>
+    hand="$(arg hand)"
+    gazebo="$(arg gazebo)"
+    parent="$(arg parent)"
+    xyz="$(arg xyz)"
+    rpy="$(arg rpy)"
+    use_fixed_camera="$(arg use_fixed_camera)"
+    use_wrist_camera="$(arg use_wrist_camera)"
+    use_bota="$(arg use_bota)"
+    include_control_plugin="$(arg include_control_plugin)" />
 </robot>

File: moma_description/urdf/panda_arm.xacro (robot description, xacro)
@@ -20,4 +20,5 @@
         fixed_calibration_xyz:='1 0 1'
         fixed_camera_parent_link:='panda_link0'
+        use_bota:=false
         include_control_plugin:=false">
     <xacro:include filename="$(find franka_description)/robots/common/utils.xacro" />
@@ -26,4 +27,11 @@
     <xacro:franka_arm arm_id="${arm_id}" safety_distance="0.03" gazebo="${gazebo}"
       joint_limits="${xacro.load_yaml('$(find franka_description)/robots/panda/joint_limits.yaml')}" />
+    <!-- Offset the hand if we have a bota sensor. -->
+    <xacro:if value="${use_bota}">
+      <xacro:property name="hand_xyz" value="0 0 0.035"/>
+    </xacro:if>
+    <xacro:unless value="${use_bota}">
+      <xacro:property name="hand_xyz" value="0 0 0"/>
+    </xacro:unless>
     <!-- Put in a basic hand. -->
     <xacro:if value="${hand}">
@@ -32,4 +40,5 @@
         arm_id="${arm_id}"
         rpy="0 0 ${-pi/4}"
+        xyz="${hand_xyz}"
         tcp_xyz="${tcp_xyz}"
         tcp_rpy="${tcp_rpy}"

Commit message: changing default panda xacros

File: moma_description/urdf/panda.urdf.xacro (robot description, xacro)
@@ -8,5 +8,5 @@
   <xacro:arg name="use_fixed_camera" default="true" />
   <xacro:arg name="use_wrist_camera" default="true" />
-  <xacro:arg name="use_bota" default="true" />
+  <xacro:arg name="use_bota" default="false" />
   <xacro:arg name="include_control_plugin" default="true" />
   <xacro:arg name="parent" default="world" />

File: moma_description/urdf/panda_arm.xacro (robot description, xacro)
@@ -158,5 +158,5 @@
       <parent link="${arm_id}_link8"/>
       <child link="${arm_id}_default_ee"/>
-      <origin rpy="0.0 0.0 -0.785" xyz="0.0 0.0 0.103"/>
+      <origin rpy="0 0 ${-pi/4}" xyz="${tcp_xyz}"/>
     </joint>
   </xacro:macro>
