Commit message: first grasp goal reaching for object

File: moma_description/urdf/object.urdf.xacro (robot description, xacro)
@@ -1,8 +1,12 @@
 <?xml version="1.0" encoding="utf-8"?>
-<robot xmlns:xacro="http://www.ros.org/wiki/xacro" name="panda">
+<robot xmlns:xacro="http://www.ros.org/wiki/xacro" name="object">
   <xacro:arg name="side_length" default="0.04" />
-  <xacro:arg name="mass_1" default="0.05" />
+  <xacro:arg name="mass_m" default="0.05" />
+  <xacro:arg name="mass_l" default="0.05" />
+  <xacro:arg name="mass_r" default="0.05" />
   <xacro:include filename="$(find moma_description)/urdf/single_cube.xacro" />
   <xacro:i_object side_length="$(arg side_length)"
-    mass_1="$(arg mass_1)" />
+    mass_m="$(arg mass_m)"
+    mass_l="$(arg mass_l)"
+    mass_r="$(arg mass_r)" />
 </robot>

File: moma_description/urdf/panda_arm.xacro (robot description, xacro)
@@ -37,4 +37,5 @@
     </xacro:unless>
     <!-- Input a bota sensor geometry -->
+    <!-- Remove bota collision geometry as otherwise collision between bota and panda_link7-->
     <link name="bota">
       <visual>
@@ -43,10 +44,10 @@
         </geometry>
       </visual>
-      <collision>
+      <!-- <collision>
         <origin xyz="0 0 0" rpy="0 0 0" />
         <geometry>
           <box size="0.2 0.2 0.035" />
         </geometry>
-      </collision>
+      </collision> -->
     </link>
     <joint name="arm_to_bota" type="revolute">

File: moma_description/urdf/single_cube.xacro (robot description, xacro)
@@ -31,5 +31,4 @@
         <!-- The reference frame of the visual element with respect to the reference frame of the link. -->
         <origin rpy="0 0 0" xyz="0.0 0.0 0.0"/>
-        <material name="blue"/>
       </visual>
       <collision>
@@ -65,5 +64,5 @@
       <parent link="middle_cube"/>
       <child link="left_cube"/>
-      <origin xyz="0 -${side_length} 0"/>
+      <origin xyz="-${side_length} 0 0"/>
       <!-- <origin xyz="-1.0 0 0"/> -->
     </joint>
@@ -87,5 +86,5 @@
       <parent link="middle_cube"/>
       <child link="right_cube"/>
-      <origin xyz="0 ${side_length} 0"/>
+      <origin xyz="${side_length} 0 0"/>
       <!-- <origin xyz="1.0 0 0"/> -->
     </joint>

Commit message: ramp up friction values to succeed in grasping

File: moma_description/urdf/object.urdf.xacro (robot description, xacro)
@@ -10,3 +10,22 @@
     mass_l="$(arg mass_l)"
     mass_r="$(arg mass_r)" />
+  <!-- Apply gazebo fix to succesfully grasp objects -->
+  <!-- <gazebo>
+  <plugin name="gazebo_grasp_fix" filename="libgazebo_grasp_fix.so">
+        <arm>
+           <arm_name>panda_arm</arm_name>
+           <palm_link> hand_link_name  </palm_link>
+           <gripper_link> finger_index_link_1 </gripper_link>
+           <gripper_link> finger_index_link_2 </gripper_link>
+           <gripper_link> ... </gripper_link>
+        </arm>
+       <forces_angle_tolerance>100</forces_angle_tolerance>
+       <update_rate>4</update_rate>
+       <grip_count_threshold>4</grip_count_threshold>
+       <max_grip_count>8</max_grip_count>
+       <release_tolerance>0.005</release_tolerance>
+       <disable_collisions_on_attach>false</disable_collisions_on_attach>
+       <contact_topic>__default_topic__</contact_topic>
+    </plugin>
+  </gazebo> -->
 </robot>

File: moma_description/urdf/panda_arm.xacro (robot description, xacro)
@@ -183,6 +183,8 @@
           transmission="hardware_interface/EffortJointInterface" />
           <!-- Friction specific material for Rubber/Rubber contact -->
-        <xacro:gazebo-friction link="${arm_id}_leftfinger" mu="1.13" />
-        <xacro:gazebo-friction link="${arm_id}_rightfinger" mu="1.13" />
+        <!-- <xacro:gazebo-friction link="${arm_id}_leftfinger" mu="1.13" />
+        <xacro:gazebo-friction link="${arm_id}_rightfinger" mu="1.13" /> -->
+        <xacro:gazebo-friction link="${arm_id}_leftfinger" mu="100" />
+        <xacro:gazebo-friction link="${arm_id}_rightfinger" mu="100" />
       </xacro:if>
       <xacro:if value="${include_control_plugin}">

File: moma_description/urdf/single_cube.xacro (robot description, xacro)
@@ -17,4 +17,14 @@
       </geometry>
     </xacro:property>
+    <xacro:property name="friction_properties">
+      <surface>
+        <friction>
+          <ode>
+            <mu>100</mu>
+            <mu2>50</mu2>
+          </ode>
+        </friction>
+      </surface>
+    </xacro:property>
     <material name="blue">
       <color rgba="0 0 0.8 1"/>
@@ -34,4 +44,5 @@
       <collision>
         <xacro:insert_block name="box_geometry"/>
+        <xacro:insert_block name="friction_properties"/>
         <!-- The reference frame of the collision element, relative to the reference frame of the link.  -->
         <origin rpy="0 0 0" xyz="0.0 0.0 0.0"/>
@@ -53,4 +64,5 @@
       <collision>
         <xacro:insert_block name="box_geometry"/>
+        <xacro:insert_block name="friction_properties"/>
       </collision>
       <inertial>
@@ -75,4 +87,5 @@
       <collision>
         <xacro:insert_block name="box_geometry"/>
+        <xacro:insert_block name="friction_properties"/>
       </collision>
       <inertial>
@@ -99,4 +112,9 @@
       <material>Gazebo/White</material>
     </gazebo>
+    <!-- create gazebo friction properties -->
+    <xacro:include filename="$(find moma_description)/urdf/utils.urdf.xacro" />
+    <xacro:gazebo-friction link="middle_cube" mu="100" />
+    <xacro:gazebo-friction link="right_cube" mu="100" />
+    <xacro:gazebo-friction link="left_cube" mu="100" />
   </xacro:macro>
 </robot>
