Commit message: launch different number of cubes depending on configured object type

File: moma_description/urdf/double_cube.xacro (robot description, xacro)
@@ -56,11 +56,38 @@
       </inertial>
     </link>
+    <link name="left_cube">
+      <visual>
+        <xacro:insert_block name="box_geometry"/>
+        <origin rpy="0 0 0" xyz="0.0 0 0"/>
+        <material name="white"/>
+      </visual>
+      <collision>
+        <xacro:insert_block name="box_geometry"/>
+        <xacro:insert_block name="friction_properties"/>
+      </collision>
+      <inertial>
+        <mass value="${mass_l}"/>
+        <inertia ixx="${1/12 * mass_l * (side_length*side_length + side_length*side_length)}" ixy="0.0" ixz="0.0"
+                  iyy="0.0000416" iyz="0.0" izz="${1/12 * mass_l * (side_length*side_length + side_length*side_length)}"/>
+      </inertial>
+    </link>
+    <!-- Let’s start by examining the joint’s origin. It is defined in terms of the parent’s reference frame. -->
+    <joint name="left_to_middle" type="fixed">
+      <parent link="middle_cube"/>
+      <child link="left_cube"/>
+      <origin xyz="-${side_length} 0 0"/>
+      <!-- <origin xyz="-1.0 0 0"/> -->
+    </joint>
     <!-- create gazebo colors -->
     <gazebo reference="middle_cube">
       <material>Gazebo/Blue</material>
     </gazebo>
+     <gazebo reference="left_cube">
+      <material>Gazebo/White</material>
+    </gazebo>
     <!-- create gazebo friction properties -->
     <xacro:include filename="$(find moma_description)/urdf/utils.urdf.xacro" />
     <xacro:gazebo-friction link="middle_cube" mu="100" />
+    <xacro:gazebo-friction link="left_cube" mu="100" />
   </xacro:macro>
 </robot>

File: moma_description/urdf/object.urdf.xacro (robot description, xacro)
@@ -5,5 +5,6 @@
   <xacro:arg name="mass_l" default="0.05" />
   <xacro:arg name="mass_r" default="0.05" />
-  <xacro:include filename="$(find moma_description)/urdf/single_cube.xacro" />
+  <xacro:arg name="file_name" default="single_cube" />
+  <xacro:include filename="$(find moma_description)/urdf/$(arg file_name).xacro" />
   <xacro:i_object side_length="$(arg side_length)"
     mass_m="$(arg mass_m)"

File: moma_description/urdf/triple_cube.xacro (robot description, xacro)
@@ -56,11 +56,65 @@
       </inertial>
     </link>
+    <link name="left_cube">
+      <visual>
+        <xacro:insert_block name="box_geometry"/>
+        <origin rpy="0 0 0" xyz="0.0 0 0"/>
+        <material name="white"/>
+      </visual>
+      <collision>
+        <xacro:insert_block name="box_geometry"/>
+        <xacro:insert_block name="friction_properties"/>
+      </collision>
+      <inertial>
+        <mass value="${mass_l}"/>
+        <inertia ixx="${1/12 * mass_l * (side_length*side_length + side_length*side_length)}" ixy="0.0" ixz="0.0"
+                  iyy="0.0000416" iyz="0.0" izz="${1/12 * mass_l * (side_length*side_length + side_length*side_length)}"/>
+      </inertial>
+    </link>
+    <!-- Let’s start by examining the joint’s origin. It is defined in terms of the parent’s reference frame. -->
+    <joint name="left_to_middle" type="fixed">
+      <parent link="middle_cube"/>
+      <child link="left_cube"/>
+      <origin xyz="-${side_length} 0 0"/>
+      <!-- <origin xyz="-1.0 0 0"/> -->
+    </joint>
+    <link name="right_cube">
+      <visual>
+        <xacro:insert_block name="box_geometry"/>
+        <origin rpy="0 0 0" xyz="0.0 0 0"/>
+        <material name="black"/>
+      </visual>
+      <collision>
+        <xacro:insert_block name="box_geometry"/>
+        <xacro:insert_block name="friction_properties"/>
+      </collision>
+      <inertial>
+        <mass value="${mass_r}"/>
+        <inertia ixx="${1/12 * mass_r * (side_length*side_length + side_length*side_length)}" ixy="0.0" ixz="0.0"
+                  iyy="0.0000416" iyz="0.0" izz="${1/12 * mass_r * (side_length*side_length + side_length*side_length)}"/>
+      </inertial>
+    </link>
+    <!-- Let’s start by examining the joint’s origin. It is defined in terms of the parent’s reference frame. -->
+    <joint name="right_to_middle" type="fixed">
+      <parent link="middle_cube"/>
+      <child link="right_cube"/>
+      <origin xyz="${side_length} 0 0"/>
+      <!-- <origin xyz="1.0 0 0"/> -->
+    </joint>
     <!-- create gazebo colors -->
     <gazebo reference="middle_cube">
       <material>Gazebo/Blue</material>
     </gazebo>
+    <gazebo reference="right_cube">
+      <material>Gazebo/Black</material>
+    </gazebo>
+     <gazebo reference="left_cube">
+      <material>Gazebo/White</material>
+    </gazebo>
     <!-- create gazebo friction properties -->
     <xacro:include filename="$(find moma_description)/urdf/utils.urdf.xacro" />
     <xacro:gazebo-friction link="middle_cube" mu="100" />
+    <xacro:gazebo-friction link="right_cube" mu="100" />
+    <xacro:gazebo-friction link="left_cube" mu="100" />
   </xacro:macro>
 </robot>
