Commit message: Update hand-eye calibration

File: moma_description/urdf/panda_arm.xacro (robot description, xacro)
@@ -97,6 +97,6 @@
   <xacro:include filename="$(find moma_description)/urdf/realsense.gazebo.xacro" />
   <xacro:realsense_gazebo_plugin camera_name="wrist_camera"/>
-  <xacro:property name="panda_link7_camera_bottom_screw_frame_rpy" value="-0.5033 -1.566 2.865" />
-  <xacro:property name="panda_link7_camera_bottom_screw_frame_xyz" value="0.0256 -0.0246 0.1522" />
+  <xacro:property name="panda_link7_camera_bottom_screw_frame_rpy" value="-0.891 -1.562 -3.040" />
+  <xacro:property name="panda_link7_camera_bottom_screw_frame_xyz" value="0.0306 -0.0267  0.1604" />
   <xacro:sensor_d435 parent="panda_link7" name="wrist_camera" use_nominal_extrinsics="${use_nominal_extrinsics}">
     <origin rpy="${panda_link7_camera_bottom_screw_frame_rpy}" xyz="${panda_link7_camera_bottom_screw_frame_xyz}" />

Commit message: Update our franka description wrapper

File: moma_description/urdf/panda_arm.xacro (robot description, xacro)
@@ -1,5 +1,5 @@
 <?xml version='1.0' encoding='utf-8'?>
 <robot xmlns:xacro="http://www.ros.org/wiki/xacro" name="panda">
-<!-- Adapted from franka_description/robots/panda_arm.urdf.xacro -->
+<!-- Adapted from franka_description/robots/common/franka_robot.xacro -->
 <xacro:macro name="moma_panda" params="arm_id:='panda'
                                        hand:=true
@@ -12,30 +12,31 @@
                                        use_nominal_extrinsics:=false
                                        include_control_plugin:=false">
-  <xacro:unless value="${gazebo}">
-    <!-- Create a URDF for a real hardware -->
-    <xacro:include filename="$(find franka_description)/robots/panda_arm.xacro" />
-    <xacro:panda_arm arm_id="${arm_id}"
-                     connected_to="${connected_to}"
-                     xyz="${xyz}"
-                     rpy="${rpy}"
-                     safety_distance="0.03"/>
-    <xacro:if value="${hand}">
-      <xacro:include filename="$(find franka_description)/robots/hand.xacro"/>
-      <xacro:hand arm_id="${arm_id}" rpy="0 0 ${-pi/4}" connected_to="${arm_id}_link8" safety_distance="0.03"/>
-    </xacro:if>
-  </xacro:unless>
+  <xacro:include filename="$(find franka_description)/robots/common/utils.xacro" />
+  <xacro:include filename="$(find franka_description)/robots/common/franka_arm.xacro" />
+  <!-- Positional offset between $(arm_id)_hand -> $(arm_id)_hand_tcp [m]. Only used when hand:=true -->
+  <xacro:arg name="tcp_xyz" default="0 0 0.1034" />
+  <!-- Rotational offset between $(arm_id)_hand -> $(arm_id)_hand_tcp [rad]. Only used when hand:=true -->
+  <xacro:arg name="tcp_rpy" default="0 0 0" />
+  <xacro:franka_arm
+      arm_id="${arm_id}"
+      connected_to="${connected_to}"
+      xyz="${xyz}"
+      rpy="${rpy}"
+      safety_distance="0.03"
+      gazebo="${gazebo}"
+      joint_limits="${xacro.load_yaml('$(find franka_description)/robots/panda/joint_limits.yaml')}"/>
+  <xacro:if value="${hand}">
+    <xacro:include filename="$(find franka_description)/robots/common/franka_hand.xacro"/>
+    <xacro:franka_hand
+        arm_id="${arm_id}"
+        rpy="0 0 ${-pi/4}"
+        tcp_xyz="$(arg tcp_xyz)"
+        tcp_rpy="$(arg tcp_rpy)"
+        connected_to="${arm_id}_link8"
+        safety_distance="0.03"
+        gazebo="${gazebo}"
+     />
+  </xacro:if>
   <xacro:if value="${gazebo}">
-    <!-- Create a simulatable URDF -->
-    <xacro:include filename="$(find franka_description)/robots/utils.xacro" />
-    <xacro:include filename="$(find franka_description)/robots/panda_gazebo.xacro" />
-    <xacro:panda_arm arm_id="${arm_id}"
-                     connected_to="${connected_to}"
-                     xyz="${xyz}"
-                     rpy="${rpy}"/>
-    <xacro:if value="${hand}">
-      <xacro:hand arm_id="${arm_id}" rpy="0 0 ${-pi/4}" connected_to="${arm_id}_link8" />
-      <xacro:gazebo-joint joint="${arm_id}_finger_joint1" transmission="hardware_interface/EffortJointInterface" />
-      <xacro:gazebo-joint joint="${arm_id}_finger_joint2" transmission="hardware_interface/EffortJointInterface" />
-    </xacro:if>
     <!-- Gazebo requires a joint to a link called "world" for statically mounted robots -->
     <xacro:if value="${fixed_to_world}">
@@ -72,5 +73,12 @@
        root="${arm_id}_joint1"
        tip="${arm_id}_joint8"
-     />
+    />
+    <xacro:if value="${hand}">
+      <xacro:gazebo-joint joint="${arm_id}_finger_joint1" transmission="hardware_interface/EffortJointInterface" />
+      <xacro:gazebo-joint joint="${arm_id}_finger_joint2" transmission="hardware_interface/EffortJointInterface" />
+      <!-- Friction specific material for Rubber/Rubber contact -->
+      <xacro:gazebo-friction link="${arm_id}_leftfinger" mu="1.13" />
+      <xacro:gazebo-friction link="${arm_id}_rightfinger" mu="1.13" />
+    </xacro:if>
     <xacro:if value="${include_control_plugin}">
       <gazebo>
@@ -87,8 +95,8 @@
   </xacro:if>
   <!-- end effector frame for MoveIt -->
-  <link name="panda_default_ee"/>
+  <link name="${arm_id}_default_ee"/>
   <joint name="joint_link8_default_ee" type="fixed">
-    <parent link="panda_link8"/>
-    <child link="panda_default_ee"/>
+    <parent link="${arm_id}_link8"/>
+    <child link="${arm_id}_default_ee"/>
     <origin rpy="0.0 0.0 -0.785" xyz="0.0 0.0 0.103"/>
   </joint>
@@ -99,5 +107,5 @@
   <xacro:property name="panda_link7_camera_bottom_screw_frame_rpy" value="-0.891 -1.562 -3.040" />
   <xacro:property name="panda_link7_camera_bottom_screw_frame_xyz" value="0.0306 -0.0267  0.1604" />
-  <xacro:sensor_d435 parent="panda_link7" name="wrist_camera" use_nominal_extrinsics="${use_nominal_extrinsics}">
+  <xacro:sensor_d435 parent="${arm_id}_link7" name="wrist_camera" use_nominal_extrinsics="${use_nominal_extrinsics}">
     <origin rpy="${panda_link7_camera_bottom_screw_frame_rpy}" xyz="${panda_link7_camera_bottom_screw_frame_xyz}" />
   </xacro:sensor_d435>

Commit message: Re-calibration from SBB Demo 11.08.2023

File: moma_description/urdf/panda_arm.xacro (robot description, xacro)
@@ -31,4 +31,5 @@
         arm_id="${arm_id}"
         rpy="0 0 ${-pi/4}"
+        xyz="0 0 0.035"
         tcp_xyz="$(arg tcp_xyz)"
         tcp_rpy="$(arg tcp_rpy)"
@@ -105,8 +106,8 @@
   <xacro:include filename="$(find moma_description)/urdf/realsense.gazebo.xacro" />
   <xacro:realsense_gazebo_plugin camera_name="wrist_camera"/>
-  <xacro:property name="panda_link7_camera_bottom_screw_frame_rpy" value="-0.891 -1.562 -3.040" />
-  <xacro:property name="panda_link7_camera_bottom_screw_frame_xyz" value="0.0306 -0.0267  0.1604" />
-  <xacro:sensor_d435 parent="${arm_id}_link7" name="wrist_camera" use_nominal_extrinsics="${use_nominal_extrinsics}">
-    <origin rpy="${panda_link7_camera_bottom_screw_frame_rpy}" xyz="${panda_link7_camera_bottom_screw_frame_xyz}" />
+  <xacro:property name="panda_link8_camera_bottom_screw_frame_rpy" value="-1.8496651 -1.5663079 -2.0611032" />
+  <xacro:property name="panda_link8_camera_bottom_screw_frame_xyz" value="0.019939866636952783 -0.024666706576001673 0.08173953529353692" />
+  <xacro:sensor_d435 parent="${arm_id}_link8" name="wrist_camera" use_nominal_extrinsics="${use_nominal_extrinsics}">
+    <origin rpy="${panda_link8_camera_bottom_screw_frame_rpy}" xyz="${panda_link8_camera_bottom_screw_frame_xyz}" />
   </xacro:sensor_d435>
   <!-- fixed realsense -->

Commit message: changing default panda xacros

File: moma_description/urdf/panda_arm.xacro (robot description, xacro)
@@ -158,5 +158,5 @@
       <parent link="${arm_id}_link8"/>
       <child link="${arm_id}_default_ee"/>
-      <origin rpy="0.0 0.0 -0.785" xyz="0.0 0.0 0.103"/>
+      <origin rpy="0 0 ${-pi/4}" xyz="${tcp_xyz}"/>
     </joint>
   </xacro:macro>

Commit message: ft sensor publishing at approximate panda bota link

File: moma_description/urdf/panda_arm.xacro (robot description, xacro)
@@ -20,5 +20,5 @@
     fixed_calibration_xyz:='0.890 -0.162 1.293'
     fixed_camera_parent_link:='panda_link0'
-    use_bota:=false
+    use_bota:=true
     multiple_robots:=false
     include_control_plugin:=true,
@@ -36,4 +36,45 @@
       <xacro:property name="hand_xyz" value="0 0 0"/>
     </xacro:unless>
+    <!-- Input a bota sensor geometry -->
+    <link name="bota">
+      <visual>
+        <geometry>
+          <box size="0.2 0.2 0.035"/>
+        </geometry>
+      </visual>
+      <collision>
+        <origin xyz="0 0 0" rpy="0 0 0" />
+        <geometry>
+          <box size="0.2 0.2 0.035" />
+        </geometry>
+      </collision>
+    </link>
+    <joint name="arm_to_bota" type="revolute">
+      <parent link="${arm_id}_link8"/>
+      <child link="bota"/>
+      <limit velocity="6.5" effort="1000" lower="0" upper="0" />
+      <!-- Not needed but also doesn't throw an error -->
+      <!-- <sensor name="force_torque" type="force_torque">
+          <update_rate>30</update_rate>
+      </sensor> -->
+    </joint>
+    <!-- Enable the Joint Feedback -->
+    <gazebo reference="arm_to_bota">
+      <provideFeedback>true</provideFeedback>
+    </gazebo>
+    <!-- Do NOT include "reference="arm_to_bota"" as sometimes seen online, will cause failure without error message -->
+    <gazebo>
+        <always_on>true</always_on>
+        <update_rate>100</update_rate>
+        <visualize>true</visualize>
+        <!-- Do NOT include the plugin inside sensor tags, this will lead to failure as it's a ModelPlugin -->
+        <plugin filename="libgazebo_ros_ft_sensor.so" name="ft_sensor">
+          <topicName>/ft_sensor_topic</topicName>
+          <jointName>arm_to_bota</jointName>
+          <always_on>true</always_on>
+          <update_rate>100</update_rate>
+          <visualize>true</visualize>
+        </plugin>
+    </gazebo>
     <!-- Put in a basic hand. -->
     <xacro:if value="${hand}">
@@ -45,5 +86,5 @@
         tcp_xyz="${tcp_xyz}"
         tcp_rpy="${tcp_rpy}"
-        connected_to="${arm_id}_link8"
+        connected_to="bota"
         safety_distance="0.03"
         gazebo="${gazebo}" />
@@ -97,4 +138,6 @@
       <xacro:gazebo-joint joint="${arm_id}_joint7"
         transmission="hardware_interface/PositionJointInterface" />
+      <xacro:gazebo-joint joint="arm_to_bota"
+        transmission="hardware_interface/PositionJointInterface" />
       <xacro:gazebo-joint joint="${arm_id}_joint1"
         transmission="hardware_interface/VelocityJointInterface" />
@@ -111,4 +154,6 @@
       <xacro:gazebo-joint joint="${arm_id}_joint7"
         transmission="hardware_interface/VelocityJointInterface" />
+      <xacro:gazebo-joint joint="arm_to_bota"
+        transmission="hardware_interface/VelocityJointInterface" />
       <xacro:gazebo-joint joint="${arm_id}_joint1"
         transmission="hardware_interface/EffortJointInterface" />
@@ -124,4 +169,6 @@
         transmission="hardware_interface/EffortJointInterface" />
       <xacro:gazebo-joint joint="${arm_id}_joint7"
+        transmission="hardware_interface/EffortJointInterface" />
+      <xacro:gazebo-joint joint="arm_to_bota"
         transmission="hardware_interface/EffortJointInterface" />
       <xacro:transmission-franka-state arm_id="${arm_id}" />
@@ -148,4 +195,9 @@
               <robotDescription>robot_description_arm</robotDescription>
             </xacro:if>
+            <xacro:unless value="${multiple_robots}">
+              <robotNamespace>/</robotNamespace>
+              <robotParam>robot_description</robotParam>
+              <robotDescription>robot_description</robotDescription>
+            </xacro:unless>
           </plugin>
           <self_collide>true</self_collide>

Commit message: added rviz config, rotate bota joint to point in same direction as EE

File: moma_description/urdf/panda_arm.xacro (robot description, xacro)
@@ -39,4 +39,5 @@
     <!-- Remove bota collision geometry as otherwise collision between bota and panda_link7-->
     <link name="bota">
+      <!-- [ 0, 0, -0.4871745, -0.8733046 ] -->
       <visual>
         <geometry>
@@ -51,5 +52,10 @@
       </collision> -->
     </link>
+         <!-- rpy="0 0 ${-pi/4}"
+        xyz="${hand_xyz}" -->
     <joint name="arm_to_bota" type="revolute">
+      <!-- This is the transform from the parent link to the child link. The joint is located at the origin of the child link, as shown in the figure above.  -->
+      <!-- Rotate the bota joint the same way as the hand for easier interpretation with respect to the EE -->
+      <origin xyz="${hand_xyz}" rpy="0 0 ${-pi/4}" />
       <parent link="${arm_id}_link8"/>
       <child link="bota"/>

Commit message: Add new EE.

File: moma_description/urdf/panda_arm.xacro (robot description, xacro)
@@ -165,4 +165,24 @@
       <origin rpy="0 0 ${-pi/4}" xyz="${tcp_xyz}"/>
     </joint>
+<!-- Custom End Effector -->
+<link name="${arm_id}_custom_ee">
+  <visual>
+    <origin xyz="0 0 0" rpy="0 0 0"/>
+    <geometry>
+      <mesh filename="package://moma_description/meshes/attachment_v2.stl"/>
+    </geometry>
+  </visual>
+  <collision>
+    <origin xyz="0 0 0" rpy="0 0 0"/>
+    <geometry>
+      <mesh filename="package://moma_description/meshes/attachment_v2.stl"/>
+    </geometry>
+  </collision>
+</link>
+<joint name="joint_link8_custom_ee" type="fixed">
+  <parent link="${arm_id}_link8"/>  <!-- or ${arm_id}_hand if you keep the gripper -->
+  <child link="${arm_id}_custom_ee"/>
+  <origin xyz="0 0 0.04" rpy="0 0 0"/> <!-- adjust offset -->
+</joint>
   </xacro:macro>
 </robot>

Commit message: WIP: Add Morris' ee

File: moma_description/urdf/panda_arm.xacro (robot description, xacro)
@@ -174,5 +174,5 @@
   </visual>
   <collision>
-    <origin xyz="0 0 0" rpy="0 0 0"/>
+  <origin xyz="0 0 0.0" rpy="0 0 ${pi/4}"/> <!-- adjust offset -->
     <geometry>
       <mesh filename="package://moma_description/meshes/attachment_v2.stl"/>
@@ -183,5 +183,5 @@
   <parent link="${arm_id}_link8"/>  <!-- or ${arm_id}_hand if you keep the gripper -->
   <child link="${arm_id}_custom_ee"/>
-  <origin xyz="0 0 0.04" rpy="0 0 0"/> <!-- adjust offset -->
+  <origin xyz="0 0 0.0" rpy="0 0 ${pi/4}"/> <!-- adjust offset -->
 </joint>
   </xacro:macro>

Commit message: Breaking, remove panda hand for morris mount.

File: moma_description/urdf/panda_arm.xacro (robot description, xacro)
@@ -165,24 +165,18 @@
       <origin rpy="0 0 ${-pi/4}" xyz="${tcp_xyz}"/>
     </joint>
-<!-- Custom End Effector -->
-<link name="${arm_id}_custom_ee">
-  <visual>
-    <origin xyz="0 0 0" rpy="0 0 0"/>
-    <geometry>
-      <mesh filename="package://moma_description/meshes/attachment_v2.stl"/>
-    </geometry>
-  </visual>
-  <collision>
-  <origin xyz="0 0 0.0" rpy="0 0 ${pi/4}"/> <!-- adjust offset -->
-    <geometry>
-      <mesh filename="package://moma_description/meshes/attachment_v2.stl"/>
-    </geometry>
-  </collision>
-</link>
-<joint name="joint_link8_custom_ee" type="fixed">
-  <parent link="${arm_id}_link8"/>  <!-- or ${arm_id}_hand if you keep the gripper -->
-  <child link="${arm_id}_custom_ee"/>
-  <origin xyz="0 0 0.0" rpy="0 0 ${pi/4}"/> <!-- adjust offset -->
-</joint>
+    <!-- Custom End Effector -->
+    <link name="${arm_id}_morris_ee">
+      <visual>
+        <origin xyz="0 0 0" rpy="0 0 0"/>
+        <geometry>
+          <mesh filename="package://moma_description/meshes/attachment_v2.stl"/>
+        </geometry>
+      </visual>
+    </link>
+    <joint name="joint_link8_morris_ee" type="fixed">
+      <parent link="${arm_id}_link8"/>  <!-- or ${arm_id}_hand if you keep the gripper -->
+      <child link="${arm_id}_morris_ee"/>
+      <origin xyz="0 0 0.0" rpy="0 0 ${pi/4}"/> <!-- adjust offset -->
+    </joint>
   </xacro:macro>
 </robot>

Commit message: Revert offset

File: moma_description/urdf/panda_arm.xacro (robot description, xacro)
@@ -168,5 +168,5 @@
     <link name="${arm_id}_morris_ee">
       <visual>
-        <origin xyz="0 0 0" rpy="0 0 0"/>
+        <origin xyz="0 0 0.0" rpy="0 0 0"/>
         <geometry>
           <mesh filename="package://moma_description/meshes/attachment_v2.stl"/>

Commit message: Add locations for cone tip and slit head

File: moma_description/urdf/panda_arm.xacro (robot description, xacro)
@@ -179,4 +179,18 @@
       <origin xyz="0 0 0.0" rpy="0 0 ${pi/4}"/> <!-- adjust offset -->
     </joint>
+  <!-- Cone tip frame 45mm away along Z -->
+  <link name="${arm_id}_cone_tip"/>
+  <joint name="joint_morris_ee_cone_tip" type="fixed">
+    <parent link="${arm_id}_morris_ee"/>
+    <child link="${arm_id}_cone_tip"/>
+    <origin xyz="0 0 0.045" rpy="0 0 0"/> <!-- 45mm in Z -->
+  </joint>
+<!-- Slit head frame 43.1945mm in Y, 8.641mm in Z -->
+<link name="${arm_id}_slit_head"/>
+<joint name="joint_morris_ee_slit_head" type="fixed">
+  <parent link="${arm_id}_morris_ee"/>
+  <child link="${arm_id}_slit_head"/>
+  <origin xyz="0 0.0438 0.008641" rpy="0 0 0"/> <!-- Y and Z offsets -->
+</joint>
   </xacro:macro>
 </robot>

Commit message: Changsg

File: moma_description/urdf/panda_arm.xacro (robot description, xacro)
@@ -184,5 +184,5 @@
     <parent link="${arm_id}_morris_ee"/>
     <child link="${arm_id}_cone_tip"/>
-    <origin xyz="0 0 0.045" rpy="0 0 0"/> <!-- 45mm in Z -->
+    <origin xyz="0 0 0.045" rpy="${pi} 0 -${pi/2}"/> <!-- 45mm in Z -->
   </joint>
 <!-- Slit head frame 43.1945mm in Y, 8.641mm in Z -->
@@ -191,5 +191,5 @@
   <parent link="${arm_id}_morris_ee"/>
   <child link="${arm_id}_slit_head"/>
-  <origin xyz="0 0.0438 0.008641" rpy="0 0 0"/> <!-- Y and Z offsets -->
+  <origin xyz="0 0.0438 0.008641" rpy="${pi} 0 -${pi/2}"/> <!-- Y and Z offsets -->
 </joint>
   </xacro:macro>
