Commit message: Added new URDF models

File: moma_demos/articulated_demo/data/models/dishwasher/dishwasher_door.urdf (robot description, URDF)
Before this commit: robot dishwasher_door, 4 links, 3 joints
Links:
- removed link door_base_link
- removed link door_link
- removed link handle_link
- added link doorFrameLink; visual box size=0.1 0.1 2; visual box size=0.1 0.1 2
- added link doorLink, mass 1.0; collision box size=0.6 0.02 0.5; visual box size=0.6 0.02 0.5
- added link door_handle_dummy_link, mass 0.1
- added link handleLink, mass 0.1; collision cylinder length=0.010 radius=0.005; visual cylinder length=0.10 radius=0.005
Joints:
- removed joint door_joint
- added joint door_handle_dummy_joint: type fixed, parent handleLink, child door_handle_dummy_link, origin xyz=0 0 0 rpy=0 0 0
- added joint joint_doorFrameLink_doorLink: type continuous, parent doorFrameLink, child doorLink, origin xyz=0 0 0, axis 1 0 0
- joint fixed: child door_base_link -> doorFrameLink; origin xyz=0.65 0 0.01 rpy=0 0 3.14 -> xyz=0.65 0 0.01 rpy=0 0 0
- joint handle_joint: child handle_link -> handleLink; parent door_link -> doorLink
