Commit message: Created model_fitting and model_based_planning skills

File: moma_demos/articulated_demo/data/models/box_panda_hand_pb.urdf (robot description, URDF)
Before this commit: robot mopa, 15 links, 14 joints
Links:
- link panda_hand: geometry collision mesh filename=/home/marko/Master_thesis/catkin_ws/src/moma/submodules/fra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; visual mesh filename=/home/marko/Master_thesis/catkin_ws/src/moma/submodules/fra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
- link panda_leftfinger: geometry collision mesh filename=/home/marko/Master_thesis/catkin_ws/src/moma/submodules/fra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; visual mesh filename=/home/marko/Master_thesis/catkin_ws/src/moma/submodules/fra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
- link panda_link0: geometry collision mesh filename=/home/marko/Master_thesis/catkin_ws/src/moma/submodules/fra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; visual mesh filename=/home/marko/Master_thesis/catkin_ws/src/moma/submodules/fra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
- link panda_link1: geometry collision mesh filename=/home/marko/Master_thesis/catkin_ws/src/moma/submodules/fra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; visual mesh filename=/home/marko/Master_thesis/catkin_ws/src/moma/submodules/fra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
- link panda_link2: geometry collision mesh filename=/home/marko/Master_thesis/catkin_ws/src/moma/submodules/fra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; visual mesh filename=/home/marko/Master_thesis/catkin_ws/src/moma/submodules/fra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
- link panda_link3: geometry collision mesh filename=/home/marko/Master_thesis/catkin_ws/src/moma/submodules/fra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; visual mesh filename=/home/marko/Master_thesis/catkin_ws/src/moma/submodules/fra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
- link panda_link4: geometry collision mesh filename=/home/marko/Master_thesis/catkin_ws/src/moma/submodules/fra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; visual mesh filename=/home/marko/Master_thesis/catkin_ws/src/moma/submodules/fra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
- link panda_link5: geometry collision mesh filename=/home/marko/Master_thesis/catkin_ws/src/moma/submodules/fra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; visual mesh filename=/home/marko/Master_thesis/catkin_ws/src/moma/submodules/fra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
- link panda_link6: geometry collision mesh filename=/home/marko/Master_thesis/catkin_ws/src/moma/submodules/fra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; visual mesh filename=/home/marko/Master_thesis/catkin_ws/src/moma/submodules/fra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
- link panda_link7: geometry collision mesh filename=/home/marko/Master_thesis/catkin_ws/src/moma/submodules/fra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; visual mesh filename=/home/marko/Master_thesis/catkin_ws/src/moma/submodules/fra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
- link panda_rightfinger: geometry collision mesh filename=/home/marko/Master_thesis/catkin_ws/src/moma/submodules/fra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; visual mesh filename=/home/marko/Master_thesis/catkin_ws/src/moma/submodules/fra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

Commit message: Added dishwasher model and simulation

File: moma_demos/articulated_demo/data/models/box_panda_hand_pb.urdf (robot description, URDF)
Before this commit: robot mopa, 15 links, 14 joints
Links:
- link panda_hand: geometry collision mesh filename=/home/marko/MT/catkin_ws/src/moma/submodules/franka_ros/fra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; visual mesh filename=/home/marko/MT/catkin_ws/src/moma/submodules/franka_ros/fra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
- link panda_leftfinger: geometry collision mesh filename=/home/marko/MT/catkin_ws/src/moma/submodules/franka_ros/fra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; visual mesh filename=/home/marko/MT/catkin_ws/src/moma/submodules/franka_ros/fra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
- link panda_link0: geometry collision mesh filename=/home/marko/MT/catkin_ws/src/moma/submodules/franka_ros/fra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; visual mesh filename=/home/marko/MT/catkin_ws/src/moma/submodules/franka_ros/fra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
- link panda_link1: geometry collision mesh filename=/home/marko/MT/catkin_ws/src/moma/submodules/franka_ros/fra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; visual mesh filename=/home/marko/MT/catkin_ws/src/moma/submodules/franka_ros/fra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
- link panda_link2: geometry collision mesh filename=/home/marko/MT/catkin_ws/src/moma/submodules/franka_ros/fra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; visual mesh filename=/home/marko/MT/catkin_ws/src/moma/submodules/franka_ros/fra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
- link panda_link3: geometry collision mesh filename=/home/marko/MT/catkin_ws/src/moma/submodules/franka_ros/fra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; visual mesh filename=/home/marko/MT/catkin_ws/src/moma/submodules/franka_ros/fra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
- link panda_link4: geometry collision mesh filename=/home/marko/MT/catkin_ws/src/moma/submodules/franka_ros/fra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; visual mesh filename=/home/marko/MT/catkin_ws/src/moma/submodules/franka_ros/fra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
- link panda_link5: geometry collision mesh filename=/home/marko/MT/catkin_ws/src/moma/submodules/franka_ros/fra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; visual mesh filename=/home/marko/MT/catkin_ws/src/moma/submodules/franka_ros/fra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
- link panda_link6: geometry collision mesh filename=/home/marko/MT/catkin_ws/src/moma/submodules/franka_ros/fra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; visual mesh filename=/home/marko/MT/catkin_ws/src/moma/submodules/franka_ros/fra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
- link panda_link7: geometry collision mesh filename=/home/marko/MT/catkin_ws/src/moma/submodules/franka_ros/fra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; visual mesh filename=/home/marko/MT/catkin_ws/src/moma/submodules/franka_ros/fra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
- link panda_rightfinger: geometry collision mesh filename=/home/marko/MT/catkin_ws/src/moma/submodules/franka_ros/fra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; visual mesh filename=/home/marko/MT/catkin_ws/src/moma/submodules/franka_ros/fra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

File: moma_demos/articulated_demo/data/models/dishwasher/dishwasher_door.urdf (robot description, URDF)
Before this commit: robot dishwasher_door, 5 links, 4 joints
Links:
- link doorFrameLink: geometry visual box size=0.04 0.7 0.82; visual box size=0.04 0.7 0.82
- link doorLink: geometry collision box size=0.6 0.02 0.8; visual box size=0.6 0.02 0.8
- link handleLink: geometry collision box size=0.015 0.015 0.2; visual box size=0.015 0.015 0.2
Joints:
- joint fixed: origin xyz=0.65 0 0.01 rpy=0 0 0 -> xyz=0.0 0 0.01 rpy=0 0 0
- joint handle_joint: axis 0 1 0 -> 1 0 0; origin xyz=0.035 0 0.47 rpy=1.5708 0 0 -> xyz=0.0 -0.03 0.77 rpy=4.7124 0 -1.5708
- joint joint_doorFrameLink_doorLink: limit (none) -> lower=-0.01 upper=1.5708; type continuous -> revolute

File: moma_demos/articulated_demo/data/models/door/door.urdf (robot description, URDF)
Before this commit: robot urdf_door, 5 links, 4 joints
Joints:
- joint handle_joint: origin xyz=0.7 -0.05 -0.15 rpy=4.7124 0 -1.5708 -> xyz=0.7 -0.1 -0.15 rpy=4.7124 0 -1.5708
- joint joint_doorFrameLink_doorLink: limit lower=-1.5708 upper=-0.1 -> lower=-1.5708 upper=0.1
