Commit message: Added SOCP controller and Init direction estimation

File: moma_demos/articulated_demo/data/models/container/container_common.xacro (robot description, xacro)
@@ -31,5 +31,5 @@
     <inertial>
       <origin rpy="0 0 0" xyz="0 0 0"/>
-       <mass value="0.2"/>
+       <mass value="0.02"/>
        <inertia ixx="1" ixy="0" ixz="0" iyy="1" iyz="0" izz="1"/>
     </inertial>
@@ -74,5 +74,5 @@
   <inertial>
     <origin rpy="0 0 0" xyz="0 0 0"/>
-    <mass value="0.2"/>
+    <mass value="0.02"/>
     <inertia ixx="1" ixy="0" ixz="0" iyy="1" iyz="0" izz="1"/>
   </inertial>

File: moma_demos/articulated_demo/data/models/container/container_no_lid.urdf (robot description, URDF)
Before this commit: robot container_no_lid, 6 links, 5 joints
Links:
- link frame_back_plane: mass 0.2 -> 0.02
- link frame_bottom_plane: mass 0.2 -> 0.02
- link frame_front_plane: mass 0.2 -> 0.02
- link frame_left_plane: mass 0.2 -> 0.02
- link frame_right_plane: mass 0.2 -> 0.02

File: moma_demos/articulated_demo/data/models/container/container_removable_lid.urdf (robot description, URDF)
Before this commit: robot container_no_lid, 8 links, 7 joints
Links:
- link frame_back_plane: mass 0.2 -> 0.02
- link frame_bottom_plane: mass 0.2 -> 0.02
- link frame_front_plane: mass 0.2 -> 0.02
- link frame_left_plane: mass 0.2 -> 0.02
- link frame_right_plane: mass 0.2 -> 0.02
- link handle: mass 0.2 -> 0.02
- link lid_plane: mass 0.2 -> 0.02

File: moma_demos/articulated_demo/data/models/container/container_removable_lid_on_table.urdf (robot description, URDF)
Before this commit: robot container_no_lid, 10 links, 9 joints
Links:
- removed link door_handle_dummy_link
- removed link handle
- removed link lid_plane
- link frame_back_plane: mass 0.2 -> 0.02
- link frame_bottom_plane: mass 0.2 -> 0.02
- link frame_front_plane: mass 0.2 -> 0.02
- link frame_left_plane: mass 0.2 -> 0.02
- link frame_right_plane: mass 0.2 -> 0.02
Joints:
- removed joint door_handle_dummy_joint
- removed joint handle_joint
- removed joint lid_joint

File: moma_demos/articulated_demo/data/models/container/container_removable_lid_on_table.urdf.xacro (robot description, xacro)
@@ -72,31 +72,3 @@
   <child link="frame_bottom_plane"/>
 </joint>
-<xacro:plane prefix="lid" width="${total_width*1.05}" depth="${total_depth*1.05}" thickness="${wall_thickness}" color="white"/>
-<joint name="lid_joint" type="prismatic">
-  <origin xyz="0 0 ${total_height-wall_thickness}" rpy="0 0 0"/>
-  <parent link="frame_bottom_plane"/>
-  <child link="lid_plane"/>
-  <axis xyz="0 0 1"/>
-  <dynamics damping="8.0"/>
-  <limit lower="0.0" upper="${0.9*total_width}" effort="10.0" velocity="1.5"/>
-</joint>
-<xacro:handle length="${total_depth*0.8}"/>
-<joint name="handle_joint" type="fixed">
-  <origin xyz="0 0 ${wall_thickness/2+0.02}" rpy="${pi/2} ${3*pi/2} 0"/>
-  <parent link="lid_plane"/>
-  <child link="handle"/>
-</joint>
-<link name="door_handle_dummy_link">
-    <!-- This dummy link is added s.t. the handle is the parent of some link and we can find the handle's index. -->
-    <inertial>
-        <origin rpy="0 0 0" xyz="0 0 0"/>
-        <mass value="0.1"/>
-        <inertia ixx="1" ixy="0" ixz="0" iyy="1" iyz="0" izz="1"/>
-    </inertial>
-</link>
-<joint name="door_handle_dummy_joint" type="fixed">
-    <origin xyz="0 0 0" rpy="0 0 0"/>
-    <parent link="handle"/>
-    <child link="door_handle_dummy_link"/>
-</joint>
 </robot>

File: moma_demos/articulated_demo/data/models/container/container_sliding_lid.urdf (robot description, URDF)
Before this commit: robot container_no_lid, 8 links, 7 joints
Links:
- link frame_back_plane: mass 0.2 -> 0.02
- link frame_bottom_plane: mass 0.2 -> 0.02
- link frame_front_plane: mass 0.2 -> 0.02
- link frame_left_plane: mass 0.2 -> 0.02
- link frame_right_plane: mass 0.2 -> 0.02
- link handle: mass 0.2 -> 0.02
- link lid_plane: mass 0.2 -> 0.02

File: moma_demos/articulated_demo/data/models/container/container_sliding_lid_on_table.urdf (robot description, URDF)
Before this commit: robot container_no_lid, 10 links, 9 joints
Links:
- link frame_back_plane: mass 0.2 -> 0.02
- link frame_bottom_plane: mass 0.2 -> 0.02
- link frame_front_plane: mass 0.2 -> 0.02
- link frame_left_plane: mass 0.2 -> 0.02
- link frame_right_plane: mass 0.2 -> 0.02
- link handle: mass 0.2 -> 0.02
- link lid_plane: mass 0.2 -> 0.02

File: moma_demos/articulated_demo/data/models/container/lid_for_container_on_table.urdf (robot description, URDF)
Before this commit: robot lid, 7 links, 6 joints
Links:
- added link door_handle_dummy_link, mass 0.0
Joints:
- added joint door_handle_dummy_joint: type fixed, parent handle, child door_handle_dummy_link, origin xyz=0 0 0 rpy=0 0 0

File: moma_demos/articulated_demo/data/models/door/door.urdf (robot description, URDF)
Before this commit: robot urdf_door, 5 links, 4 joints
Joints:
- joint handle_joint: origin xyz=0.7 -0.1 -0.15 rpy=4.7124 0 -1.5708 -> xyz=0.7 -0.1 -0.1 rpy=4.7124 0 -1.5708
- joint joint_doorFrameLink_doorLink: limit lower=-1.5708 upper=0.1 -> lower=-1.5708 upper=0.0

File: moma_demos/articulated_demo/data/models/sliding_door/sliding_door.urdf (robot description, URDF)
Before this commit: robot urdf_sliding_door, 5 links, 4 joints
Links:
- link doorFrameLink: geometry collision box size=0.1 0.1 2; collision box size=0.1 0.1 2
Joints:
- joint joint_doorFrameLink_doorLink: origin xyz=0.05 0 0.95 -> xyz=0.05 0 1.0
