Commit message: cleanup, moving objects to moma_gazebo

File: moma_description/objects/urdf/valve.urdf.xacro (robot description, xacro)
@@ -50,5 +50,5 @@
       <origin xyz="0 0 0" rpy="0 0 0"/>
       <geometry>
-        <cylinder radius="0.07" length="0.02"/>
+        <cylinder radius="0.12" length="0.02"/>
       </geometry>
     </visual>
