Commit message: gripper calibration

File: moma_description/grippers/robotiq_2f_toolset/urdf/robotiq_2f_toolset.xacro (robot description, xacro)
@@ -9,5 +9,5 @@
     </xacro:bota_sensor>
     <xacro:zedm parent="ft_sensor0">
-      <origin xyz="0.0 0.0 0.0" rpy="0.0 0.0 3.14"/>
+      <origin xyz="0.0 0.0 0.0" rpy="0.0 0.0 0.0"/>
     </xacro:zedm>
     <xacro:robotiq_2f_85 parent="ft_sensor0" prefix="">

File: moma_description/urdf/panda.xacro (robot description, xacro)
@@ -23,5 +23,5 @@
       <xacro:include filename="$(find moma_description)/grippers/robotiq_2f_toolset/urdf/robotiq_2f_toolset.xacro"/>
       <xacro:robotiq_2f_toolset parent="panda_link8">
-        <origin xyz="0 0 0" rpy="0 0 0"/>
+        <origin xyz="0 0 0" rpy="0 0 ${-pi/2}"/>
       </xacro:robotiq_2f_toolset>
     </xacro:if>

Commit message: calibration urdf

File: moma_description/grippers/robotiq_2f_toolset/urdf/robotiq_2f_toolset.xacro (robot description, xacro)
@@ -9,5 +9,5 @@
     </xacro:bota_sensor>
     <xacro:zedm parent="ft_sensor0">
-      <origin xyz="0.0 0.0 0.0" rpy="0.0 0.0 0.0"/>
+      <origin xyz="0.0 0.0 0.0" rpy="0.0 0.0 3.14"/>
     </xacro:zedm>
     <xacro:robotiq_2f_85 parent="ft_sensor0" prefix="">

File: moma_description/sensors/bota/urdf/bota.urdf.xacro (robot description, xacro)
@@ -10,5 +10,5 @@
     <link name="ft_sensor0">
       <visual>
-        <origin xyz="0 0 0" rpy="0 0 3.14" />
+        <origin xyz="0 0 0" rpy="0 0 0" />
         <geometry>
           <mesh filename="package://moma_description/sensors/bota/meshes/bota_sensor.stl" scale="0.001 0.001 0.001"/>
@@ -19,5 +19,5 @@
       </visual>
       <collision>
-        <origin xyz="0 0 0" rpy="0 0 3.14" />
+        <origin xyz="0 0 0" rpy="0 0 0" />
         <geometry>
           <mesh filename="package://moma_description/sensors/bota/meshes/bota_sensor.stl" scale="0.001 0.001 0.001"/>

File: moma_description/urdf/panda.xacro (robot description, xacro)
@@ -23,5 +23,5 @@
       <xacro:include filename="$(find moma_description)/grippers/robotiq_2f_toolset/urdf/robotiq_2f_toolset.xacro"/>
       <xacro:robotiq_2f_toolset parent="panda_link8">
-        <origin xyz="0 0 0" rpy="0 0 ${-pi/2}"/>
+        <origin xyz="0 0 0" rpy="0 0 ${pi/2}"/>
       </xacro:robotiq_2f_toolset>
     </xacro:if>
