Commit message: tested mpc on the platform

File: moma_controllers/moma_ocs2/urdf/panda.urdf (robot description, URDF)
Before this commit: robot panda, 11 links, 10 joints
Links:
- link panda_hand: geometry collision box size=0.035 0.19 0.065; visual mesh filename=file:///home/franka/control_ws/src/moma/submodules/franka_r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
- link panda_link0: geometry collision mesh filename=file:///home/franka/control_ws/src/moma/submodules/franka_r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; visual mesh filename=file:///home/franka/control_ws/src/moma/submodules/franka_r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
- link panda_link1: geometry collision mesh filename=file:///home/franka/control_ws/src/moma/submodules/franka_r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; visual mesh filename=file:///home/franka/control_ws/src/moma/submodules/franka_r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
- link panda_link2: geometry collision mesh filename=file:///home/franka/control_ws/src/moma/submodules/franka_r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; visual mesh filename=file:///home/franka/control_ws/src/moma/submodules/franka_r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
- link panda_link3: geometry collision mesh filename=file:///home/franka/control_ws/src/moma/submodules/franka_r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; visual mesh filename=file:///home/franka/control_ws/src/moma/submodules/franka_r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
- link panda_link4: geometry collision mesh filename=file:///home/franka/control_ws/src/moma/submodules/franka_r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; visual mesh filename=file:///home/franka/control_ws/src/moma/submodules/franka_r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
- link panda_link5: geometry collision mesh filename=file:///home/franka/control_ws/src/moma/submodules/franka_r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; visual mesh filename=file:///home/franka/control_ws/src/moma/submodules/franka_r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
- link panda_link6: geometry collision mesh filename=file:///home/franka/control_ws/src/moma/submodules/franka_r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; visual mesh filename=file:///home/franka/control_ws/src/moma/submodules/franka_r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
- link panda_link7: geometry collision mesh filename=file:///home/franka/control_ws/src/moma/submodules/franka_r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; visual mesh filename=file:///home/franka/control_ws/src/moma/submodules/franka_r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

Commit message: using the right xml

File: moma_controllers/moma_ocs2/urdf/panda.urdf (robot description, URDF)
Before this commit: robot panda, 11 links, 10 joints
Links:
- link panda_hand: geometry collision box size=0.035 0.19 0.065; visual mesh filename=file:///home/giuseppe/kinova_ws/src/moma/submodules/franka_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
- link panda_link0: geometry collision mesh filename=file:///home/giuseppe/kinova_ws/src/moma/submodules/franka_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; visual mesh filename=file:///home/giuseppe/kinova_ws/src/moma/submodules/franka_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
- link panda_link1: geometry collision mesh filename=file:///home/giuseppe/kinova_ws/src/moma/submodules/franka_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; visual mesh filename=file:///home/giuseppe/kinova_ws/src/moma/submodules/franka_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
- link panda_link2: geometry collision mesh filename=file:///home/giuseppe/kinova_ws/src/moma/submodules/franka_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; visual mesh filename=file:///home/giuseppe/kinova_ws/src/moma/submodules/franka_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
- link panda_link3: geometry collision mesh filename=file:///home/giuseppe/kinova_ws/src/moma/submodules/franka_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; visual mesh filename=file:///home/giuseppe/kinova_ws/src/moma/submodules/franka_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
- link panda_link4: geometry collision mesh filename=file:///home/giuseppe/kinova_ws/src/moma/submodules/franka_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; visual mesh filename=file:///home/giuseppe/kinova_ws/src/moma/submodules/franka_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
- link panda_link5: geometry collision mesh filename=file:///home/giuseppe/kinova_ws/src/moma/submodules/franka_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; visual mesh filename=file:///home/giuseppe/kinova_ws/src/moma/submodules/franka_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
- link panda_link6: geometry collision mesh filename=file:///home/giuseppe/kinova_ws/src/moma/submodules/franka_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; visual mesh filename=file:///home/giuseppe/kinova_ws/src/moma/submodules/franka_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
- link panda_link7: geometry collision mesh filename=file:///home/giuseppe/kinova_ws/src/moma/submodules/franka_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; visual mesh filename=file:///home/giuseppe/kinova_ws/src/moma/submodules/franka_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
