Commit message: integration new grippers and removing old paths

File: moma_description/grippers/robotiq_2f_85/urdf/robotiq_2f_85.xacro (robot description, xacro)
@@ -3,5 +3,5 @@
   <xacro:include filename="$(find moma_description)/grippers/robotiq_2f_85/urdf/robotiq_arg2f_85_model.xacro" />
   <xacro:include filename="$(find moma_description)/grippers/robotiq_2f_85/urdf/robotiq_2f_85_transmission.xacro" />
-  <xacro:macro name="robotiq_arg2f_85" params="parent prefix *origin">
+  <xacro:macro name="robotiq_2f_85" params="parent prefix *origin">
     <joint name="${prefix}gripper_base_joint" type="fixed">
 	    <parent link="${parent}"/>

File: moma_description/grippers/robotiq_2f_toolset/urdf/robotiq_2f_toolset.xacro (robot description, xacro)
@@ -4,14 +4,14 @@
   <xacro:include filename="$(find moma_description)/sensors/bota/urdf/bota.urdf.xacro"/>
   <xacro:include filename="$(find moma_description)/sensors/zedm/urdf/zedm.urdf.xacro"/>
-  <xacro:macro name="robotiq_2f_toolset" params="parent">
+  <xacro:macro name="robotiq_2f_toolset" params="parent *origin">
     <xacro:bota_sensor parent="${parent}">
-      <origin xyz="0 0 0.0" rpy="0 0 0.0" />
+      <xacro:insert_block name='origin'/>
     </xacro:bota_sensor>
     <xacro:zedm parent="ft_sensor0">
       <origin xyz="0.0 0.0 0.0" rpy="0.0 0.0 3.14"/>
     </xacro:zedm>
-    <xacro:robotiq_arg2f_85 parent="ft_sensor0" prefix="">
+    <xacro:robotiq_2f_85 parent="ft_sensor0" prefix="">
       <origin xyz="0.0 0.0 0.046" rpy="0.0 0.0 0.0"/>
-    </xacro:robotiq_arg2f_85>
+    </xacro:robotiq_2f_85>
   </xacro:macro>
 </robot>

File: moma_description/sensors/bota/urdf/bota.urdf.xacro (robot description, xacro)
@@ -3,9 +3,14 @@
   <xacro:property name="bota_interface_height" default="0.06"/>
   <xacro:macro name="bota_sensor" params="parent *origin">
-    <link name="bota_interface">
+    <joint name="bota_joint" type="fixed">
+      <parent link="${parent}"/>
+      <child link="ft_sensor0"/>
+      <xacro:insert_block name="origin"/>
+    </joint>
+    <link name="ft_sensor0">
       <visual>
         <origin xyz="0 0 0" rpy="0 0 3.14" />
         <geometry>
-          <cylinder radius="0.035" length="${bota_interface_height}"/>
+          <mesh filename="package://moma_description/sensors/bota/meshes/bota_sensor.stl" scale="0.001 0.001 0.001"/>
         </geometry>
         <material name="">
@@ -16,5 +21,5 @@
         <origin xyz="0 0 0" rpy="0 0 3.14" />
         <geometry>
-          <cylinder radius="0.035" length="${bota_interface_height}"/>
+          <mesh filename="package://moma_description/sensors/bota/meshes/bota_sensor.stl" scale="0.001 0.001 0.001"/>
         </geometry>
         <material name="">
@@ -23,34 +28,4 @@
       </collision>
     </link>
-    <joint name="bota_interface_joint" type="fixed">
-      <parent link="${parent}"/>
-      <child link="bota_interface"/>
-      <xacro:insert_block name="origin"/>
-    </joint>
-    <link name="ft_sensor0">
-      <visual>
-        <origin xyz="0 0 0" rpy="0 0 3.14" />
-        <geometry>
-          <mesh filename="package://kinova_description/sensors/bota/meshes/bota_sensor.stl" scale="0.001 0.001 0.001"/>
-        </geometry>
-        <material name="">
-          <color rgba="0.75294 0.75294 0.75294 1" />
-        </material>
-      </visual>
-      <collision>
-        <origin xyz="0 0 0" rpy="0 0 3.14" />
-        <geometry>
-          <mesh filename="package://kinova_description/sensors/bota/meshes/bota_sensor.stl" scale="0.001 0.001 0.001"/>
-        </geometry>
-        <material name="">
-          <color rgba="0.75294 0.75294 0.75294 1" />
-        </material>
-      </collision>
-    </link>
-    <joint name="bota_sensor_joint" type="fixed">
-      <parent link="bota_interface"/>
-      <child link="ft_sensor0"/>
-      <origin xyz="0 0 ${bota_interface_height/2.0}" rpy="0 0 -1.57079" />
-    </joint>
   </xacro:macro>
 </robot>

File: moma_description/sensors/zedm/urdf/zedm.urdf.xacro (robot description, xacro)
@@ -1,5 +1,5 @@
 <?xml version="1.0"?>
 <robot name="stereolabs_camera" xmlns:xacro="http://ros.org/wiki/xacro">
-  <xacro:include filename="$(find kinova_description)/sensors/zedm/urdf/materials.urdf.xacro" />
+  <xacro:include filename="$(find moma_description)/sensors/zedm/urdf/materials.urdf.xacro" />
   <xacro:property name="M_PI"     value="3.1415926535897931" />
   <xacro:property name="baseline" value="0.063" />
@@ -9,5 +9,5 @@
         <origin xyz="0 0 0" rpy="0 0 0" />
         <geometry>
-          <mesh filename="package://kinova_description/sensors/zedm/meshes/zed_mount.stl" scale="0.001 0.001 0.001"/>
+          <mesh filename="package://moma_description/sensors/zedm/meshes/zed_mount.stl" scale="0.001 0.001 0.001"/>
         </geometry>
         <material name="">
@@ -18,5 +18,5 @@
         <origin xyz="0 0 0" rpy="0 0 0" />
         <geometry>
-          <mesh filename="package://kinova_description/sensors/zedm/meshes/zed_mount.stl" scale="0.001 0.001 0.001"/>
+          <mesh filename="package://moma_description/sensors/zedm/meshes/zed_mount.stl" scale="0.001 0.001 0.001"/>
         </geometry>
         <material name="">
@@ -46,5 +46,5 @@
             <origin xyz="0 0 0" rpy="0 0 0"/>
             <geometry>
-                <mesh filename="package://kinova_description/sensors/zedm/meshes/zedm.stl" />
+                <mesh filename="package://moma_description/sensors/zedm/meshes/zedm.stl" />
             </geometry>
             <material name="zedm_mat" />
@@ -53,5 +53,5 @@
             <origin xyz="0 0 0" rpy="0 0 0"/>
             <geometry>
-                <mesh filename="package://kinova_description/sensors/zedm/meshes/zedm.stl" />
+                <mesh filename="package://moma_description/sensors/zedm/meshes/zedm.stl" />
             </geometry>
             <material name="zedm_mat" />

File: moma_description/urdf/panda.xacro (robot description, xacro)
@@ -15,7 +15,14 @@
     <xacro:if value="${tool == 'robotiq_2f_85'}">
       <xacro:include filename="$(find moma_description)/grippers/robotiq_2f_85/urdf/robotiq_2f_85.xacro"/>
-      <xacro:robotiq_arg2f_85 parent="panda_link8" prefix="">
+      <xacro:robotiq_2f_85 parent="panda_link8" prefix="">
         <origin xyz="0 0 0" rpy="0 0 0"/>
-      </xacro:robotiq_arg2f_85>
+      </xacro:robotiq_2f_85>
+    </xacro:if>
+    <!-- robotiq 2f-85 toolset (plate + FT sensor + gripper + zedm camera) -->
+    <xacro:if value="${tool == 'robotiq_2f_toolset'}">
+      <xacro:include filename="$(find moma_description)/grippers/robotiq_2f_toolset/urdf/robotiq_2f_toolset.xacro"/>
+      <xacro:robotiq_2f_toolset parent="panda_link8">
+        <origin xyz="0 0 0" rpy="0 0 0"/>
+      </xacro:robotiq_2f_toolset>
     </xacro:if>
     <!-- end effector frame for MoveIt -->

Commit message: config changes

File: moma_description/grippers/robotiq_2f_85/urdf/robotiq_2f_85.xacro (robot description, xacro)
@@ -17,6 +17,6 @@
     <link name="${prefix}tool_frame"/>
     <joint name="${prefix}tool_frame_joint" type="fixed">
-        <origin xyz="0 0 0.120" rpy="0 0 0" />
-        <parent link="${parent}" />
+        <origin xyz="0 0 0.140" rpy="0 0 0" />
+        <parent link="robotiq_arg2f_base_link" />
         <child link="${prefix}tool_frame" />
         <axis xyz="0 0 0" />

Commit message: fixed description

File: moma_description/grippers/robotiq_2f_85/urdf/robotiq_2f_85.xacro (robot description, xacro)
@@ -3,9 +3,13 @@
   <xacro:include filename="$(find moma_description)/grippers/robotiq_2f_85/urdf/robotiq_arg2f_85_model.xacro" />
   <xacro:include filename="$(find moma_description)/grippers/robotiq_2f_85/urdf/robotiq_2f_85_transmission.xacro" />
+  <xacro:include filename="$(find moma_description)/grippers/robotiq_2f_85/urdf/robotiq_ur_coupler.urdf.xacro" />
   <xacro:macro name="robotiq_2f_85" params="parent prefix *origin">
+    <xacro:robotiq_ur_coupler parent="${parent}">
+      <xacro:insert_block name='origin'/>
+    </xacro:robotiq_ur_coupler>
     <joint name="${prefix}gripper_base_joint" type="fixed">
-	    <parent link="${parent}"/>
+	    <parent link="robotiq_coupler"/>
       <child link="${prefix}robotiq_arg2f_base_link"/>
-      <xacro:insert_block name='origin'/>
+      <!--xacro:insert_block name='origin'/-->
     </joint>
     <xacro:robotiq_arg2f_base_link prefix="${prefix}"/>

File: moma_description/grippers/robotiq_2f_toolset/urdf/robotiq_2f_toolset.xacro (robot description, xacro)
@@ -8,9 +8,9 @@
       <xacro:insert_block name='origin'/>
     </xacro:BFT_SENS_SER_M8>
-    <xacro:zedm parent="ft_sensor0">
+    <xacro:zedm parent="ft_sensor0_mounting">
       <origin xyz="0.0 0.0 0.0" rpy="0.0 0.0 3.14"/>
     </xacro:zedm>
-    <xacro:robotiq_2f_85 parent="ft_sensor0" prefix="">
-      <origin xyz="0.0 0.0 0.046" rpy="0.0 0.0 0.0"/>
+    <xacro:robotiq_2f_85 parent="ft_sensor0_wrench" prefix="">
+      <origin xyz="0.0 0.0 0.0" rpy="0.0 0.0 0.0"/>
     </xacro:robotiq_2f_85>
   </xacro:macro>

File: moma_description/sensors/bota/urdf/BFT_SENS_SER_M8.urdf.xacro (robot description, xacro)
@@ -51,5 +51,5 @@
     </link>
     <link
-      name="${prefix}">
+      name="${prefix}_wrench">
       <inertial>
         <origin
@@ -99,5 +99,5 @@
         link="${prefix}_mounting" />
       <child
-        link="${prefix}" />
+        link="${prefix}_wrench" />
       <axis
         xyz="0 0 0" />

Commit message: working state machine

File: moma_description/grippers/robotiq_2f_85/urdf/robotiq_2f_85.xacro (robot description, xacro)
@@ -21,5 +21,5 @@
     <link name="${prefix}tool_frame"/>
     <joint name="${prefix}tool_frame_joint" type="fixed">
-        <origin xyz="0 0 0.140" rpy="0 0 0" />
+        <origin xyz="0 0 0.140" rpy="0 0 -1.5708" />
         <parent link="robotiq_arg2f_base_link" />
         <child link="${prefix}tool_frame" />

Commit message: successful state machine test (with interaction)

File: moma_description/grippers/robotiq_2f_85/urdf/robotiq_2f_85.xacro (robot description, xacro)
@@ -21,5 +21,5 @@
     <link name="${prefix}tool_frame"/>
     <joint name="${prefix}tool_frame_joint" type="fixed">
-        <origin xyz="0 0 0.140" rpy="0 0 -1.5708" />
+        <origin xyz="0 0 0.135" rpy="0 0 -1.5708" />
         <parent link="robotiq_arg2f_base_link" />
         <child link="${prefix}tool_frame" />

Commit message: hardware tuning

File: moma_description/grippers/robotiq_2f_85/urdf/robotiq_2f_85.xacro (robot description, xacro)
@@ -21,5 +21,5 @@
     <link name="${prefix}tool_frame"/>
     <joint name="${prefix}tool_frame_joint" type="fixed">
-        <origin xyz="0 0 0.135" rpy="0 0 -1.5708" />
+        <origin xyz="0 0 0.125" rpy="0 0 -1.5708" />
         <parent link="robotiq_arg2f_base_link" />
         <child link="${prefix}tool_frame" />
