Commit message: Add static valve base (not working yet)

File: moma_demos/piloting_demo/urdf/valve.urdf (robot description, URDF)
Before this commit: robot valve_model, 3 links, 2 joints
Links:
- removed link world
- added link valve_base
- link wheel: geometry collision mesh filename=package://piloting_demo/models/valve/meshes/valve.dae scale=1.0 1.0 1.0; visual mesh filename=package://piloting_demo/models/valve/meshes/valve.stl scale=1.0 1.0 1.0
Joints:
- removed joint valve_base_joint

File: moma_demos/piloting_demo/urdf/valve.urdf.xacro (robot description, xacro)
@@ -1,15 +1,8 @@
 <?xml version="1.0" encoding="utf-8"?>
 <robot name="valve_model" xmlns:xacro="http://www.ros.org/wiki/xacro">
-   <xacro:arg name="x"      default="1.2"/>
-   <xacro:arg name="y"      default="0.0"/>
-   <xacro:arg name="z"      default="0.5"/>
-   <xacro:arg name="roll"   default="0.0"/>
-   <xacro:arg name="pitch"  default="0.0"/>
-   <xacro:arg name="yaw"    default="0.0"/>
-   <link name="world">
-   </link>
+    <link name="valve_base"/>
     <joint name="valve_base_joint" type="fixed">
-      <origin xyz="$(arg x) $(arg y) $(arg z)" rpy="0 $(arg pitch) $(arg yaw)"/>
-      <parent link="world"/>
+      <origin xyz="1.0 0.0 0.0" rpy="0.0 0.0 0.0"/>
+      <parent link="valve_base"/>
       <child link="valve_gt"/>
     </joint>
