Commit message: integrating perception in sim with no sim2real gap in state machine

File: moma_demos/piloting_demo/urdf/valve.urdf.xacro (robot description, xacro)
@@ -10,5 +10,5 @@
    </link>
     <joint name="valve_base_joint" type="fixed">
-      <origin xyz="$(arg x) $(arg y) $(arg z)" rpy="3.14 $(arg pitch) $(arg yaw)"/>
+      <origin xyz="$(arg x) $(arg y) $(arg z)" rpy="0 $(arg pitch) $(arg yaw)"/>
       <parent link="world"/>
       <child link="valve_gt"/>
@@ -42,5 +42,5 @@
     </inertial>
     <collision>
-      <origin xyz="0 0 0" rpy="0 0 0"/>
+      <origin xyz="0 0 0" rpy="3.14 0 0"/>
         <geometry>
           <mesh filename="package://piloting_demo/models/valve/meshes/valve.dae" scale="1.0 1.0 1.0"/>
@@ -48,5 +48,5 @@
     </collision>
     <visual>
-      <origin xyz="0 0 0" rpy="0 0 0"/>
+      <origin xyz="0 0 0" rpy="3.14 0 0"/>
         <geometry>
           <mesh filename="package://piloting_demo/models/valve/meshes/valve.stl" scale="1.0 1.0 1.0"/>

Commit message: Add valve turning simulatability

File: moma_demos/piloting_demo/urdf/valve.urdf.xacro (robot description, xacro)
@@ -46,4 +46,14 @@
           <mesh filename="package://piloting_demo/models/valve/meshes/valve.dae" scale="1.0 1.0 1.0"/>
         </geometry>
+      <surface>
+        <friction>
+          <ode>
+            <mu>1</mu>
+            <mu2>1</mu2>
+            <slip1>0</slip1>
+            <slip2>0</slip2>
+          </ode>
+        </friction>
+      </surface>
     </collision>
     <visual>
@@ -54,5 +64,6 @@
     </visual>
   </link>
-  <joint name="wheel_joint" type="continuous">
+  <link name="grasp_point" />
+  <joint name="wheel_joint" type="revolute">
     <origin xyz="0 0 0" rpy="0.0 0 0"/>
     <axis xyz="0 0 1" rpy="0 0 0"/>
@@ -61,4 +72,10 @@
     <dynamics damping="10.0" friction="10.0"/>
     <limit effort="30" velocity="1.0" lower="-3.14" upper="3.14"/>
+  </joint>
+  <joint name="grasp_point_joint" type="fixed">
+    <origin xyz="0 0.1 0" rpy="0 0 -1.57"/>
+    <axis xyz="0 0 1" rpy="0 0 0"/>
+    <parent link="wheel"/>
+    <child link="grasp_point"/>
   </joint>
   <!-- Gazebo simulation -->

Commit message: Add working real demo config and adjustment

File: moma_demos/piloting_demo/urdf/valve.urdf.xacro (robot description, xacro)
@@ -7,9 +7,9 @@
    <xacro:arg name="pitch"  default="0.0"/>
    <xacro:arg name="yaw"    default="0.0"/>
-   <link name="world">
+   <link name="map">
    </link>
     <joint name="valve_base_joint" type="fixed">
       <origin xyz="$(arg x) $(arg y) $(arg z)" rpy="0 $(arg pitch) $(arg yaw)"/>
-      <parent link="world"/>
+      <parent link="map"/>
       <child link="valve_gt"/>
     </joint>

Commit message: Fix valve in sim by using sim param and world anchoring

File: moma_demos/piloting_demo/urdf/valve.urdf.xacro (robot description, xacro)
@@ -1,15 +1,23 @@
 <?xml version="1.0" encoding="utf-8"?>
 <robot name="valve_model" xmlns:xacro="http://www.ros.org/wiki/xacro">
-   <xacro:arg name="x"      default="1.2"/>
-   <xacro:arg name="y"      default="0.0"/>
-   <xacro:arg name="z"      default="0.5"/>
-   <xacro:arg name="roll"   default="0.0"/>
-   <xacro:arg name="pitch"  default="0.0"/>
-   <xacro:arg name="yaw"    default="0.0"/>
-   <link name="map">
-   </link>
+    <xacro:arg name="sim"    default="false"/>
+    <xacro:arg name="x"      default="1.2"/>
+    <xacro:arg name="y"      default="0.0"/>
+    <xacro:arg name="z"      default="0.5"/>
+    <xacro:arg name="roll"   default="0.0"/>
+    <xacro:arg name="pitch"  default="0.0"/>
+    <xacro:arg name="yaw"    default="0.0"/>
+    <xacro:if value="$(arg sim)">
+        <!-- In sim, any static object needs to be anchored at world. Luckily, world and map align in sim -->
+        <xacro:property name="root_frame" value="world"/>
+    </xacro:if>
+    <xacro:unless value="$(arg sim)">
+        <xacro:property name="root_frame" value="map"/>
+    </xacro:unless>
+    <link name="${root_frame}">
+    </link>
     <joint name="valve_base_joint" type="fixed">
       <origin xyz="$(arg x) $(arg y) $(arg z)" rpy="0 $(arg pitch) $(arg yaw)"/>
-      <parent link="map"/>
+      <parent link="${root_frame}"/>
       <child link="valve_gt"/>
     </joint>
